File: launchpad.brd (EAGLE design)
At the start: 66 x 50.8 mm, 3 parts

Commit message: fix distance for display
Parts:
- moved JP2 1.27 mm to (39.4, 10.2)
- moved JP1 1.27 mm to (39.4, 40.6)
Routing:
- net N$1: track 48.4 -> 46.3 mm
- net +3V3: track 40.4 -> 39.2 mm
- net N$2: track 25.2 -> 26.5 mm
- net N$4: track 45.7 -> 44.4 mm
- net N$3: track 45.7 -> 44.4 mm
- net GND: track 23.7 -> 25.0 mm
- net N$5: track 43.6 -> 42.3 mm
Changed lines of the file:
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@@
 <elements>
 <element name="U$1" library="StellarisLaunchPad_Fred" package="LAUNCHPAD-COMPATIBLE" value="STELLARIS-LAUNCHPAD-COMPATIBLESTELLARIS-LAUNCHPAD-COMPATIBLE" x="0" y="0"/>
-<element name="JP1" library="pinhead" package="1X08" value="" x="39.37" y="41.91"/>
-<element name="JP2" library="pinhead" package="1X08" value="" x="39.37" y="8.89"/>
+<element name="JP1" library="pinhead" package="1X08" value="" x="39.37" y="40.64"/>
+<element name="JP2" library="pinhead" package="1X08" value="" x="39.37" y="10.16"/>
 </elements>
 <signals>
@@
 <contactref element="U$1" pad="3.3V"/>
 <contactref element="JP1" pad="1"/>
-<wire x1="30.48" y1="11.43" x2="30.48" y2="41.91" width="0.254" layer="1"/>
-<wire x1="31.75" y1="10.16" x2="30.48" y2="11.43" width="0.254" layer="1"/>
-<wire x1="31.75" y1="3.81" x2="31.75" y2="10.16" width="0.254" layer="1"/>
+<wire x1="30.48" y1="12.7" x2="30.48" y2="40.64" width="0.254" layer="1"/>
+<wire x1="31.75" y1="11.43" x2="30.48" y2="12.7" width="0.254" layer="1"/>
+<wire x1="31.75" y1="3.81" x2="31.75" y2="11.43" width="0.254" layer="1"/>
 <wire x1="30.48" y1="2.54" x2="31.75" y2="3.81" width="0.254" layer="1"/>
 </signal>
@@
 <contactref element="U$1" pad="GND2"/>
 <contactref element="JP1" pad="8"/>
-<wire x1="44.45" y1="45.72" x2="48.26" y2="41.91" width="0.254" layer="1"/>
-<wire x1="44.45" y1="49.53" x2="44.45" y2="45.72" width="0.254" layer="1"/>
+<wire x1="48.26" y1="43.18" x2="48.26" y2="40.64" width="0.254" layer="1"/>
+<wire x1="44.45" y1="46.99" x2="48.26" y2="43.18" width="0.254" layer="1"/>
+<wire x1="44.45" y1="49.53" x2="44.45" y2="46.99" width="0.254" layer="1"/>
 <wire x1="31.75" y1="49.53" x2="44.45" y2="49.53" width="0.254" layer="1"/>
 <wire x1="30.48" y1="48.26" x2="31.75" y2="49.53" width="0.254" layer="1"/>
@@
 <contactref element="U$1" pad="PB4"/>
 <contactref element="JP2" pad="1"/>
-<wire x1="30.48" y1="5.08" x2="30.48" y2="8.89" width="0.254" layer="1"/>
+<wire x1="30.48" y1="5.08" x2="30.48" y2="10.16" width="0.254" layer="1"/>
 <wire x1="29.21" y1="3.81" x2="30.48" y2="5.08" width="0.254" layer="1"/>
 <wire x1="29.21" y1="1.27" x2="29.21" y2="3.81" width="0.254" layer="1"/>
@@
 <contactref element="U$1" pad="PB7"/>
 <contactref element="JP2" pad="2"/>
-<wire x1="33.02" y1="22.86" x2="33.02" y2="8.89" width="0.254" layer="1"/>
-<wire x1="31.75" y1="24.13" x2="33.02" y2="22.86" width="0.254" layer="1"/>
-<wire x1="31.75" y1="43.18" x2="31.75" y2="24.13" width="0.254" layer="1"/>
-<wire x1="35.56" y1="46.99" x2="31.75" y2="43.18" width="0.254" layer="1"/>
-<wire x1="41.91" y1="46.99" x2="35.56" y2="46.99" width="0.254" layer="1"/>
+<wire x1="33.02" y1="24.13" x2="33.02" y2="10.16" width="0.254" layer="1"/>
+<wire x1="31.75" y1="25.4" x2="33.02" y2="24.13" width="0.254" layer="1"/>
+<wire x1="31.75" y1="41.91" x2="31.75" y2="25.4" width="0.254" layer="1"/>
+<wire x1="36.83" y1="46.99" x2="31.75" y2="41.91" width="0.254" layer="1"/>
+<wire x1="41.91" y1="46.99" x2="36.83" y2="46.99" width="0.254" layer="1"/>
 <wire x1="43.18" y1="48.26" x2="41.91" y2="46.99" width="0.254" layer="1"/>
 </signal>
@@
 <contactref element="U$1" pad="PA5"/>
 <contactref element="JP1" pad="2"/>
-<wire x1="33.02" y1="24.13" x2="33.02" y2="41.91" width="0.254" layer="1"/>
-<wire x1="46.99" y1="10.16" x2="33.02" y2="24.13" width="0.254" layer="1"/>
-<wire x1="46.99" y1="3.81" x2="46.99" y2="10.16" width="0.254" layer="1"/>
+<wire x1="33.02" y1="25.4" x2="33.02" y2="40.64" width="0.254" layer="1"/>
+<wire x1="46.99" y1="11.43" x2="33.02" y2="25.4" width="0.254" layer="1"/>
+<wire x1="46.99" y1="3.81" x2="46.99" y2="11.43" width="0.254" layer="1"/>
 <wire x1="48.26" y1="2.54" x2="46.99" y2="3.81" width="0.254" layer="1"/>
 </signal>
@@
 <contactref element="U$1" pad="PA6"/>
 <contactref element="JP1" pad="3"/>
-<wire x1="35.56" y1="24.13" x2="35.56" y2="41.91" width="0.254" layer="1"/>
-<wire x1="50.8" y1="8.89" x2="35.56" y2="24.13" width="0.254" layer="1"/>
-<wire x1="50.8" y1="2.54" x2="50.8" y2="8.89" width="0.254" layer="1"/>
+<wire x1="35.56" y1="25.4" x2="35.56" y2="40.64" width="0.254" layer="1"/>
+<wire x1="50.8" y1="10.16" x2="35.56" y2="25.4" width="0.254" layer="1"/>
+<wire x1="50.8" y1="2.54" x2="50.8" y2="10.16" width="0.254" layer="1"/>
 </signal>
 <signal name="N$5">
 <contactref element="U$1" pad="PA7"/>
 <contactref element="JP1" pad="6"/>
-<wire x1="43.18" y1="17.78" x2="43.18" y2="41.91" width="0.254" layer="1"/>
-<wire x1="53.34" y1="7.62" x2="43.18" y2="17.78" width="0.254" layer="1"/>
-<wire x1="53.34" y1="2.54" x2="53.34" y2="7.62" width="0.254" layer="1"/>
+<wire x1="43.18" y1="19.05" x2="43.18" y2="40.64" width="0.254" layer="1"/>
+<wire x1="53.34" y1="8.89" x2="43.18" y2="19.05" width="0.254" layer="1"/>
+<wire x1="53.34" y1="2.54" x2="53.34" y2="8.89" width="0.254" layer="1"/>
 </signal>
 </signals>

Commit message: add gnd polygons
Routing:
- added copper zone on layer 1, net GND
Changed lines of the file:
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@@
 </class>
 </classes>
-<designrules name="default">
+<designrules name="default *">
 <description language="de">&lt;b&gt;EAGLE Design Rules&lt;/b&gt;
 &lt;p&gt;
@@
 <param name="mtCopper" value="0.035mm 0.035mm 0.035mm 0.035mm 0.035mm 0.035mm 0.035mm 0.035mm 0.035mm 0.035mm 0.035mm 0.035mm 0.035mm 0.035mm 0.035mm 0.035mm"/>
 <param name="mtIsolate" value="1.5mm 0.15mm 0.2mm 0.15mm 0.2mm 0.15mm 0.2mm 0.15mm 0.2mm 0.15mm 0.2mm 0.15mm 0.2mm 0.15mm 0.2mm"/>
-<param name="mdWireWire" value="8mil"/>
-<param name="mdWirePad" value="8mil"/>
-<param name="mdWireVia" value="8mil"/>
-<param name="mdPadPad" value="8mil"/>
-<param name="mdPadVia" value="8mil"/>
-<param name="mdViaVia" value="8mil"/>
-<param name="mdSmdPad" value="8mil"/>
-<param name="mdSmdVia" value="8mil"/>
-<param name="mdSmdSmd" value="8mil"/>
+<param name="mdWireWire" value="12mil"/>
+<param name="mdWirePad" value="12mil"/>
+<param name="mdWireVia" value="12mil"/>
+<param name="mdPadPad" value="12mil"/>
+<param name="mdPadVia" value="12mil"/>
+<param name="mdViaVia" value="12mil"/>
+<param name="mdSmdPad" value="12mil"/>
+<param name="mdSmdVia" value="12mil"/>
+<param name="mdSmdSmd" value="12mil"/>
 <param name="mdViaViaSameLayer" value="8mil"/>
 <param name="mnLayersViaInSmd" value="2"/>
@@
 <wire x1="31.75" y1="49.53" x2="44.45" y2="49.53" width="0.254" layer="1"/>
 <wire x1="30.48" y1="48.26" x2="31.75" y2="49.53" width="0.254" layer="1"/>
+<polygon width="0.4064" layer="1">
+<vertex x="27.94" y="50.8"/>
+<vertex x="27.94" y="0"/>
+<vertex x="55.88" y="0"/>
+<vertex x="55.88" y="50.8"/>
+</polygon>
 </signal>
 <signal name="N$2">
