File: raspi.brd (EAGLE design)
At the start: 74.6 x 55.9 mm, 5 parts

Commit message: fix distance for display
Parts:
- moved JP1 2.54 mm to (49.5, 41.9)
- moved JP2 1.27 mm to (49.5, 11.4)
Connections:
- new net N$1: U$1.8
- new net N$2: U$1.10
Routing:
- net N$5: track 63.7 -> 141.8 mm
- net GND: track 107.1 -> 39.2 mm
- net N$8: track 67.1 -> 111.0 mm
- net +3V3: track 141.7 -> 98.0 mm
- net N$9: track 71.4 -> 95.5 mm
- net N$4: track 40.0 -> 61.1 mm
- net N$7: track 29.7 -> 39.2 mm
- net N$3: track 106.5 -> 108.0 mm

Commit message: rework raspi board
Parts:
- removed SW1, SW2: (no value), microbuilder:PUSHBUTTON_SMD_SJ
- added S1, S2: (no value), SparkFun:TACTILE-PTH
- moved JP1 30.6 mm to (47.0, 11.4)
- moved JP2 30.6 mm to (47.0, 41.9)
Connections:
- removed net N$1: U$1.8
- removed net N$4: SW2.P$1, U$1.26
- net +3V3: now also S1.3, S2.3; no longer SW1.P$2, SW2.P$2
- net N$2: now also S2.1, U$1.26; no longer U$1.10
- net N$3: now also S1.1; no longer SW1.P$1
Routing:
- net N$5: track 141.8 -> 29.1 mm
- net N$2: track 0.00 -> 109.0 mm
- net N$3: track 108.0 -> 29.6 mm
- net N$4: track 61.1 -> 0.00 mm
- net N$8: track 111.0 -> 61.5 mm
- net N$6: track 0.00 -> 33.7 mm
- net N$7: track 39.2 -> 71.0 mm
- net N$9: track 95.5 -> 67.7 mm
- net GND: track 39.2 -> 55.3 mm
- net +3V3: track 98.0 -> 98.6 mm

Commit message: add gnd polygons
Routing:
- added copper zone on layer 1, net GND
Other:
- board size 74.6 x 55.9 mm -> 60.6 x 53.3 mm
Changed lines of the file:
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@@
 <board>
 <plain>
-<wire x1="0" y1="0" x2="74.6" y2="0" width="0" layer="20"/>
-<wire x1="74.6" y1="0" x2="74.6" y2="55.87" width="0" layer="20"/>
-<wire x1="74.6" y1="55.87" x2="0" y2="55.87" width="0" layer="20"/>
-<wire x1="0" y1="55.87" x2="0" y2="0" width="0" layer="20"/>
+<wire x1="0" y1="2.54" x2="60.63" y2="2.54" width="0" layer="20"/>
+<wire x1="60.63" y1="2.54" x2="60.63" y2="55.87" width="0" layer="20"/>
+<wire x1="60.63" y1="55.87" x2="0" y2="55.87" width="0" layer="20"/>
+<wire x1="0" y1="55.87" x2="0" y2="2.54" width="0" layer="20"/>
 </plain>
 <attributes>
@@
 <wire x1="8.89" y1="52.07" x2="8.89" y2="46.99" width="0.254" layer="1"/>
 <wire x1="7.62" y1="53.34" x2="8.89" y2="52.07" width="0.254" layer="1"/>
+<polygon width="0.4064" layer="1">
+<vertex x="0" y="55.88"/>
+<vertex x="0" y="2.54"/>
+<vertex x="60.96" y="2.54"/>
+<vertex x="60.96" y="55.88"/>
+</polygon>
 </signal>
 <signal name="N$3">
