File: raspi.brd (EAGLE design)
At the start: 60.6 x 53.3 mm, 5 parts

Commit message: work on shield
Parts:
- removed JP1, JP2: (no value), pinhead:1X08
- added C1, C2, C4, C5: 1uF, SparkFun-Capacitors:0805
- added C3: 104, SparkFun-Capacitors:0805
- added R1: 390k/560k, SparkFun-Resistors:0805
- added U$2: USB_AB, SparkFun-Connectors:USB-AB-MICRO-SMD
- added U1: (no value), microbuilder:UG-2864HSWEG01_0.96IN_WRAPAROUND
- S1, S2: value (none) -> SWITCH-MOMENTARY-2PTH; device SparkFun:TACTILE-PTH -> SparkFun-Electromechanical:TACTILE-PTH
- moved S1 1.80 mm to (25.4, 34.3), turned to 270 degrees
- moved S2 1.80 mm to (25.4, 19.1), turned to 270 degrees
Connections:
- new net +5V: U$1.2, U$2.VBUS
- new net N$1: U$1.19, U1.19
- new net N$10: C1.1, U1.2
- new net N$11: C2.1, U1.4
- new net N$12: C1.2, U1.3
- new net N$13: C2.2, U1.5
- new net N$4: U$1.16, U1.15
- new net VCC: U1.28
- new net VSS: U1.8
- net +3V3: now also C3.1, C4.1, U1.9; no longer JP1.1
- net GND: now also C3.2, C4.2, C5.2, R1.2, U$1.25, U$1.9, U$2.GND, U1.1, U1.10, U1.11, U1.12, U1.29, U1.30; no longer JP1.8
- net N$5: now also U1.18; no longer JP2.1
- net N$6: now also C5.1, U1.27; no longer JP2.2, U$1.19
- net N$7: now also U1.13; no longer JP1.6
- net N$8: now also U1.14; no longer JP1.3
- net N$9: now also R1.1, U1.26; no longer JP1.2, U$1.16
Routing:
- net N$9: track 67.7 -> 7.90 mm
- net GND: track 55.3 -> 0.00 mm
- net +5V: track 0.00 -> 50.9 mm
- net N$4: track 0.00 -> 47.9 mm
- net N$2: track 109.0 -> 71.4 mm
- net N$1: track 0.00 -> 37.6 mm
- net N$6: track 33.7 -> 6.30 mm
- net N$3: track 29.6 -> 50.9 mm
- net N$7: track 71.0 -> 50.4 mm
- net N$13: track 0.00 -> 9.45 mm
- net N$5: track 29.1 -> 38.5 mm, vias 0 -> 2
- net N$11: track 0.00 -> 8.88 mm
- net N$12: track 0.00 -> 7.04 mm
- net N$8: track 61.5 -> 54.6 mm
- net N$10: track 0.00 -> 6.62 mm
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- added copper zone on layer 16, net GND
- removed copper zone on layer 1, net GND
Other:
- board size 60.6 x 53.3 mm -> 53.3 x 55.2 mm

Commit message: work in progress
Parts:
- removed U$1: RASPBERRY-PI, RaspberryPi:RASPBERRY-PI
- added U$3: RASPBERRY-PI_REV1, RaspberryPi:RASPBERRY-PI_REV1
- added U2: CP2110-F01-GM, bxl_import:CP2110-F01-GM
Connections:
- new net N$14: U$2.D-, U2.4
- new net N$15: U$2.D+, U2.3
- new net N$16: U$3.8, U2.21
- new net N$17: U$3.10, U2.20
- net +3V3: now also U$3.1; no longer U$1.1
- net +5V: now also U$3.2; no longer U$1.2
- net GND: now also U$3.25, U$3.6, U$3.9, U2.2, U2.25; no longer U$1.25, U$1.6, U$1.9
- net N$1: now also U$3.19; no longer U$1.19
- net N$2: now also U$3.26; no longer U$1.26
- net N$3: now also U$3.24; no longer U$1.24
- net N$4: now also U$3.16; no longer U$1.16
- net N$5: now also U$3.23; no longer U$1.23
- net N$7: now also U$3.22; no longer U$1.22
- net N$8: now also U$3.18; no longer U$1.18
Routing:
- net N$17: track 0.00 -> 49.9 mm, vias 0 -> 2
- net N$16: track 0.00 -> 49.8 mm, vias 0 -> 2
- net N$15: track 0.00 -> 23.9 mm
- net N$14: track 0.00 -> 19.4 mm
- net +3V3: track 101.0 -> 108.1 mm

Commit message: work on product scheme
Changed lines of the file:
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@@
 <wire x1="34.66" y1="19.95" x2="34.66" y2="18.415" width="0.4064" layer="16"/>
 <wire x1="34.66" y1="18.415" x2="34.66" y2="16.51" width="0.4064" layer="16"/>
-<wire x1="34.66" y1="18.415" x2="23.1775" y2="18.415" width="0.4064" layer="16"/>
 <wire x1="45.085" y1="22.12" x2="46.92" y2="22.12" width="0.3048" layer="16"/>
 <wire x1="23.1394" y1="22.3012" x2="20.955" y2="22.3012" width="0.4064" layer="16"/>
@@
 <wire x1="18.415" y1="15.875" x2="20.955" y2="18.415" width="0.4064" layer="16"/>
 <wire x1="20.955" y1="18.415" x2="23.1775" y2="18.415" width="0.4064" layer="16"/>
+<wire x1="23.1775" y1="18.415" x2="34.66" y2="18.415" width="0.4064" layer="16"/>
 </signal>
 <signal name="GND">

Commit message: work in progress
Parts:
- added C6, C7: 1uF, SparkFun-Capacitors:0805
- added C8: 0.1uF, SparkFun-Capacitors:0805
- added R2: 4k7, SparkFun-Resistors:0805
- moved U2 9.55 mm to (23.5, 8.26)
Connections:
- new net N$18: C6.2, U2.7
- new net N$20: R2.2, U2.9
- net +3V3: now also C7.2, C8.2, R2.1, U2.5, U2.6
- net +5V: now also U2.8
- net GND: now also C6.1, C7.1, C8.1
Routing:
- net +3V3: track 108.1 -> 135.6 mm
- net +5V: track 50.7 -> 74.3 mm
- net GND: track 0.00 -> 17.6 mm
- net N$14: track 19.4 -> 35.3 mm, vias 0 -> 2
- net N$20: track 0.00 -> 7.99 mm
- net N$15: track 23.9 -> 31.6 mm, vias 0 -> 2
- net N$18: track 0.00 -> 7.02 mm
- net N$16: track 49.8 -> 55.0 mm
- net N$17: track 49.9 -> 52.5 mm

Commit message: work on pcbs
Other:
- board text added: "trezor"
Changed lines of the file:
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@@
 <wire x1="39.37" y1="56.505" x2="0" y2="56.505" width="0" layer="20"/>
 <wire x1="0" y1="56.505" x2="0" y2="1.27" width="0" layer="20"/>
+<text x="15.24" y="11.43" size="1.778" layer="16" font="vector" rot="MR0">trezor</text>
 </plain>
 <attributes>

Commit message: work in progress
Routing:
- net N$14: track 35.3 -> 33.7 mm
- net N$16: track 55.0 -> 56.3 mm
- net N$1: track 37.6 -> 38.7 mm
- net N$15: track 31.6 -> 32.6 mm
Changed lines of the file:
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@@
 <setting verticaltext="up"/>
 </settings>
-<grid distance="25" unitdist="mil" unit="mil" style="lines" multiple="1" display="no" altdistance="12.5" altunitdist="mil" altunit="mil"/>
+<grid distance="0.635" unitdist="mm" unit="mm" style="lines" multiple="1" display="no" altdistance="0.3175" altunitdist="mm" altunit="mm"/>
 <layers>
 <layer number="1" name="Top" color="4" fill="1" visible="yes" active="yes"/>
@@
 </class>
 </classes>
-<designrules name="default *">
+<designrules name="default">
 <description language="de">&lt;b&gt;EAGLE Design Rules&lt;/b&gt;
 &lt;p&gt;
@@
 <wire x1="36.195" y1="30.48" x2="36.195" y2="40.005" width="0.4064" layer="16"/>
 <contactref element="U$3" pad="19"/>
-<wire x1="36.195" y1="40.005" x2="25.4" y2="50.8" width="0.4064" layer="16"/>
+<wire x1="25.4" y1="50.8" x2="25.4" y2="48.895" width="0.4064" layer="16"/>
+<wire x1="25.4" y1="48.895" x2="27.305" y2="48.895" width="0.4064" layer="16"/>
+<wire x1="27.305" y1="48.895" x2="36.195" y2="40.005" width="0.4064" layer="16"/>
 </signal>
 <signal name="N$5">
@@
 <contactref element="U$3" pad="23"/>
 <wire x1="34.925" y1="39.6875" x2="30.48" y2="44.1325" width="0.4064" layer="16"/>
-<via x="30.48" y="44.1325" extent="1-16" drill="0.6" shape="square"/>
+<via x="30.48" y="44.1325" extent="1-16" drill="0.8" diameter="1.27"/>
 <wire x1="30.48" y1="44.1325" x2="30.48" y2="48.26" width="0.4064" layer="1"/>
-<via x="30.48" y="48.26" extent="1-16" drill="0.6" shape="square"/>
+<via x="30.48" y="48.26" extent="1-16" drill="0.8" diameter="1.27"/>
 <wire x1="30.48" y1="48.26" x2="30.48" y2="50.8" width="0.4064" layer="16"/>
 </signal>
@@
 <contactref element="U2" pad="4"/>
 <wire x1="25.654" y1="8.001" x2="29.845" y2="8.001" width="0.3048" layer="16"/>
-<wire x1="29.845" y1="8.001" x2="29.845" y2="12.7" width="0.3048" layer="16"/>
-<via x="29.845" y="12.7" extent="1-16" drill="0.6" shape="square"/>
-<wire x1="29.845" y1="12.7" x2="15.875" y2="8.255" width="0.3048" layer="1"/>
-<via x="15.875" y="8.255" extent="1-16" drill="0.6" shape="square"/>
+<wire x1="29.845" y1="8.001" x2="29.845" y2="11.43" width="0.3048" layer="16"/>
+<via x="29.845" y="11.43" extent="1-16" drill="0.8" diameter="1.27"/>
+<wire x1="29.845" y1="11.43" x2="15.875" y2="8.255" width="0.3048" layer="1"/>
+<via x="15.875" y="8.255" extent="1-16" drill="0.8" diameter="1.27"/>
 <wire x1="15.875" y1="8.255" x2="15.875" y2="6.985" width="0.3048" layer="16"/>
 <wire x1="15.875" y1="6.985" x2="5.39" y2="6.985" width="0.3048" layer="16"/>
@@
 <wire x1="25.654" y1="8.509" x2="28.575" y2="8.509" width="0.3048" layer="16"/>
 <wire x1="28.575" y1="8.509" x2="28.575" y2="12.7" width="0.3048" layer="16"/>
-<via x="28.575" y="12.7" extent="1-16" drill="0.6" shape="square"/>
-<wire x1="28.575" y1="12.7" x2="14.605" y2="8.255" width="0.3048" layer="1"/>
-<via x="14.605" y="8.255" extent="1-16" drill="0.6" shape="square"/>
-<wire x1="14.605" y1="8.255" x2="14.605" y2="7.62" width="0.3048" layer="16"/>
+<via x="28.575" y="12.7" extent="1-16" drill="0.8" diameter="1.27"/>
+<wire x1="28.575" y1="12.7" x2="14.605" y2="9.525" width="0.3048" layer="1"/>
+<via x="14.605" y="9.525" extent="1-16" drill="0.8" diameter="1.27"/>
+<wire x1="14.605" y1="9.525" x2="14.605" y2="7.62" width="0.3048" layer="16"/>
 <wire x1="14.605" y1="7.62" x2="5.39" y2="7.62" width="0.3048" layer="16"/>
 </signal>
@@
 <contactref element="U2" pad="21"/>
 <contactref element="U$3" pad="8"/>
-<via x="23.8125" y="12.3825" extent="1-16" drill="0.6" shape="square"/>
-<via x="13.335" y="18.7325" extent="1-16" drill="0.6" shape="square"/>
+<via x="24.4475" y="12.3825" extent="1-16" drill="0.8" diameter="1.27"/>
+<via x="12.7" y="18.7325" extent="1-16" drill="0.8" diameter="1.27"/>
 <wire x1="10.16" y1="53.34" x2="9.525" y2="53.34" width="0.4064" layer="16"/>
 <wire x1="9.525" y1="53.34" x2="8.255" y2="52.07" width="0.4064" layer="16"/>
@@
 <wire x1="6.35" y1="50.165" x2="6.985" y2="49.53" width="0.4064" layer="16"/>
 <wire x1="6.985" y1="49.53" x2="6.985" y2="25.0825" width="0.4064" layer="16"/>
-<wire x1="6.985" y1="25.0825" x2="13.335" y2="18.7325" width="0.4064" layer="16"/>
-<wire x1="23.8125" y1="12.3825" x2="23.241" y2="12.3825" width="0.3048" layer="16"/>
+<wire x1="6.985" y1="25.0825" x2="12.7" y2="18.7325" width="0.4064" layer="16"/>
+<wire x1="24.4475" y1="12.3825" x2="23.241" y2="12.3825" width="0.3048" layer="16"/>
 <wire x1="23.241" y1="12.3825" x2="23.241" y2="10.414" width="0.3048" layer="16"/>
-<wire x1="13.335" y1="18.7325" x2="23.8125" y2="12.3825" width="0.3048" layer="1"/>
+<wire x1="12.7" y1="18.7325" x2="24.4475" y2="12.3825" width="0.3048" layer="1"/>
 </signal>
 <signal name="N$17">
 <contactref element="U2" pad="20"/>
 <contactref element="U$3" pad="10"/>
-<via x="22.225" y="12.3825" extent="1-16" drill="0.6" shape="square"/>
-<via x="14.9225" y="18.7325" extent="1-16" drill="0.6" shape="square"/>
+<via x="21.59" y="12.3825" extent="1-16" drill="0.8" diameter="1.27"/>
+<via x="14.9225" y="18.7325" extent="1-16" drill="0.8" diameter="1.27"/>
 <wire x1="12.7" y1="53.34" x2="12.065" y2="53.34" width="0.4064" layer="16"/>
 <wire x1="12.065" y1="53.34" x2="10.795" y2="52.07" width="0.4064" layer="16"/>
@@
 <wire x1="8.255" y1="49.53" x2="8.255" y2="25.4" width="0.4064" layer="16"/>
 <wire x1="8.255" y1="25.4" x2="14.9225" y2="18.7325" width="0.4064" layer="16"/>
-<wire x1="22.225" y1="12.3825" x2="22.733" y2="12.3825" width="0.3048" layer="16"/>
+<wire x1="21.59" y1="12.3825" x2="22.733" y2="12.3825" width="0.3048" layer="16"/>
 <wire x1="22.733" y1="12.3825" x2="22.733" y2="10.414" width="0.3048" layer="16"/>
-<wire x1="14.9225" y1="18.7325" x2="22.225" y2="12.3825" width="0.3048" layer="1"/>
+<wire x1="14.9225" y1="18.7325" x2="21.59" y2="12.3825" width="0.3048" layer="1"/>
 </signal>
 <signal name="N$18">

Commit message: raspi shield
Parts:
- moved U2 9.99 mm to (13.5, 7.44)
- moved C8 9.26 mm to (22.6, 8.26)
- moved C7 7.37 mm to (26.4, 8.26)
- moved C6 6.23 mm to (24.5, 8.26)
- moved R2 4.03 mm to (21.5, 3.81), turned to 0 degrees
Connections:
- net N$14 renamed USB_D_N
- net N$15 renamed USB_D_P
Routing:
- net N$2: track 71.4 -> 33.3 mm
- net +3V3: track 135.6 -> 99.6 mm
- net N$3: track 50.9 -> 17.0 mm
- net USB_D_N: track 33.7 -> 17.9 mm
- net USB_D_P: track 32.6 -> 18.1 mm
- net GND: track 17.6 -> 3.90 mm, vias 0 -> 9
- net N$16: track 56.3 -> 45.0 mm, vias 2 -> 0
- net +5V: track 74.3 -> 65.8 mm, vias 0 -> 3
- net N$7: track 50.4 -> 42.0 mm
- net N$18: track 7.02 -> 13.6 mm, vias 0 -> 2
- net N$4: track 47.9 -> 41.4 mm
- net N$8: track 54.6 -> 49.4 mm
- net N$5: track 38.5 -> 33.7 mm, vias 2 -> 0
- net N$1: track 38.7 -> 34.6 mm
- net N$17: track 52.6 -> 50.2 mm, vias 2 -> 0
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- added copper zone on layer 1, net GND
Other:
- board text added: "RASOR"
- board text removed: "trezor"

Commit message: raspi work rename product to trezor
Routing:
- net GND: track 3.90 -> 6.62 mm, vias 9 -> 11
- net N$5: track 33.7 -> 35.2 mm
- net N$7: track 42.0 -> 43.3 mm
Changed lines of the file:
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@@
 <param name="mtCopper" value="0.035mm 0.035mm 0.035mm 0.035mm 0.035mm 0.035mm 0.035mm 0.035mm 0.035mm 0.035mm 0.035mm 0.035mm 0.035mm 0.035mm 0.035mm 0.035mm"/>
 <param name="mtIsolate" value="1.5mm 0.15mm 0.2mm 0.15mm 0.2mm 0.15mm 0.2mm 0.15mm 0.2mm 0.15mm 0.2mm 0.15mm 0.2mm 0.15mm 0.2mm"/>
-<param name="mdWireWire" value="7mil"/>
-<param name="mdWirePad" value="7mil"/>
-<param name="mdWireVia" value="7mil"/>
-<param name="mdPadPad" value="7mil"/>
-<param name="mdPadVia" value="7mil"/>
-<param name="mdViaVia" value="7mil"/>
-<param name="mdSmdPad" value="7mil"/>
-<param name="mdSmdVia" value="7mil"/>
-<param name="mdSmdSmd" value="7mil"/>
+<param name="mdWireWire" value="12mil"/>
+<param name="mdWirePad" value="12mil"/>
+<param name="mdWireVia" value="12mil"/>
+<param name="mdPadPad" value="12mil"/>
+<param name="mdPadVia" value="12mil"/>
+<param name="mdViaVia" value="12mil"/>
+<param name="mdSmdPad" value="8mil"/>
+<param name="mdSmdVia" value="8mil"/>
+<param name="mdSmdSmd" value="8mil"/>
 <param name="mdViaViaSameLayer" value="8mil"/>
 <param name="mnLayersViaInSmd" value="2"/>
@@
 <vertex x="-1.2192" y="57.5056"/>
 </polygon>
-<via x="2.8448" y="15.0368" extent="1-16" drill="0.6" shape="square"/>
-<via x="20.5232" y="10.5664" extent="1-16" drill="0.6" shape="square"/>
+<via x="2.4384" y="14.8336" extent="1-16" drill="0.6" shape="square"/>
+<via x="24.384" y="4.064" extent="1-16" drill="0.6" shape="square"/>
 <via x="43.0784" y="27.8384" extent="1-16" drill="0.6" shape="square"/>
 <via x="44.0944" y="24.384" extent="1-16" drill="0.6" shape="square"/>
@@
 <via x="38.2016" y="35.56" extent="1-16" drill="0.6" shape="square"/>
 <via x="38.608" y="15.6464" extent="1-16" drill="0.6" shape="square"/>
-<via x="27.0256" y="10.7696" extent="1-16" drill="0.6" shape="square"/>
+<via x="24.5872" y="10.9728" extent="1-16" drill="0.6" shape="square"/>
 <via x="5.8928" y="46.1264" extent="1-16" drill="0.6" shape="square"/>
-<wire x1="15.6972" y1="8.2042" x2="16.9418" y2="8.2042" width="0.3048" layer="16"/>
-<wire x1="16.9418" y1="8.2042" x2="17.0688" y2="8.3312" width="0.3048" layer="16"/>
 <wire x1="15.6972" y1="8.2042" x2="14.3002" y2="8.2042" width="0.3048" layer="16"/>
 <wire x1="14.3002" y1="8.2042" x2="13.5382" y2="7.4422" width="0.3048" layer="16"/>
+<via x="17.0688" y="11.176" extent="1-16" drill="0.6" shape="square"/>
+<wire x1="15.6972" y1="8.2042" x2="16.7386" y2="8.2042" width="0.3048" layer="16"/>
+<wire x1="16.7386" y1="8.2042" x2="17.0688" y2="8.5344" width="0.3048" layer="16"/>
+<wire x1="17.0688" y1="8.5344" x2="17.0688" y2="11.176" width="0.3048" layer="16"/>
+<via x="46.9392" y="14.6304" extent="1-16" drill="0.6" shape="square"/>
 </signal>
 <signal name="N$3">
@@
 <wire x1="48.3503" y1="24.92" x2="48.8351" y2="25.4048" width="0.3048" layer="16"/>
 <wire x1="48.8351" y1="25.4048" x2="48.8351" y2="37.3438" width="0.3048" layer="16"/>
-<wire x1="48.8351" y1="37.3438" x2="44.0536" y2="42.1253" width="0.3048" layer="16"/>
-<wire x1="44.0536" y1="42.1253" x2="39.9434" y2="42.1253" width="0.3048" layer="16"/>
-<wire x1="39.9434" y1="42.1253" x2="31.5644" y2="50.5043" width="0.3048" layer="16"/>
+<wire x1="48.8351" y1="37.3438" x2="44.2568" y2="41.9221" width="0.3048" layer="16"/>
 <wire x1="31.5644" y1="50.5043" x2="31.5644" y2="51.2872" width="0.3048" layer="16"/>
 <wire x1="31.5644" y1="51.2872" x2="30.7816" y2="52.07" width="0.3048" layer="16"/>
 <wire x1="30.7816" y1="52.07" x2="29.21" y2="52.07" width="0.3048" layer="16"/>
 <wire x1="29.21" y1="52.07" x2="27.94" y2="53.34" width="0.3048" layer="16"/>
+<wire x1="37.7323" y1="42.1253" x2="33.7312" y2="46.1264" width="0.3048" layer="16"/>
+<wire x1="31.5644" y1="50.5043" x2="31.5644" y2="48.2932" width="0.3048" layer="16"/>
+<wire x1="31.5644" y1="48.2932" x2="33.7312" y2="46.1264" width="0.3048" layer="16"/>
+<wire x1="44.2568" y1="41.9221" x2="37.9355" y2="41.9221" width="0.3048" layer="16"/>
+<wire x1="37.9355" y1="41.9221" x2="37.7323" y2="42.1253" width="0.3048" layer="16"/>
 </signal>
 <signal name="N$8">
@@
 <wire x1="48.3503" y1="37.1458" x2="44.2265" y2="41.2696" width="0.3048" layer="16"/>
 <wire x1="44.2265" y1="41.2696" x2="40.0104" y2="41.2696" width="0.3048" layer="16"/>
-<wire x1="40.0104" y1="41.2696" x2="30.48" y2="50.8" width="0.3048" layer="16"/>
+<wire x1="40.0104" y1="41.2696" x2="37.3688" y2="41.2696" width="0.3048" layer="16"/>
+<wire x1="37.3688" y1="41.2696" x2="30.48" y2="48.1584" width="0.3048" layer="16"/>
+<wire x1="30.48" y1="48.1584" x2="30.48" y2="50.8" width="0.3048" layer="16"/>
 </signal>
 <signal name="N$4">
