File: raspi.brd (EAGLE design)
At the start: 53.3 x 55.2 mm, 16 parts, among them U2 CP2110-F01-GM

Commit message: work snapshot
Parts:
- C3: value 104 -> 0.1uF
Changed lines of the file:
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@@
 <element name="C1" library="SparkFun-Capacitors" package="0805" value="1uF" x="40.64" y="17.78" rot="MR90"/>
 <element name="C2" library="SparkFun-Capacitors" package="0805" value="1uF" x="40.64" y="21.59" rot="MR90"/>
-<element name="C3" library="SparkFun-Capacitors" package="0805" value="104" x="38.1" y="19.05" rot="MR270"/>
+<element name="C3" library="SparkFun-Capacitors" package="0805" value="0.1uF" x="38.1" y="19.05" rot="MR270"/>
 <element name="C4" library="SparkFun-Capacitors" package="0805" value="1uF" x="35.56" y="16.51" rot="MR180"/>
 <element name="C5" library="SparkFun-Capacitors" package="0805" value="1uF" x="40.64" y="35.56" rot="MR90"/>

Commit message: wip
Routing:
- net +3V3: track 99.6 -> 106.9 mm
- net N$7: track 43.3 -> 44.3 mm
- net GND: vias 11 -> 12
Other:
- outline, holes or cut-outs redrawn
- board text added: "shield"
- board text removed: "RASOR"
Changed lines of the file:
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@@
 <plain>
 <wire x1="0" y1="1.27" x2="53.34" y2="1.27" width="0" layer="20"/>
-<wire x1="53.34" y1="1.27" x2="53.34" y2="43.18" width="0" layer="20"/>
-<wire x1="53.34" y1="43.18" x2="39.37" y2="43.18" width="0" layer="20"/>
-<wire x1="39.37" y1="43.18" x2="39.37" y2="56.505" width="0" layer="20"/>
+<wire x1="53.34" y1="1.27" x2="53.34" y2="42.5704" width="0" layer="20"/>
+<wire x1="53.34" y1="42.5704" x2="39.37" y2="42.5704" width="0" layer="20"/>
+<wire x1="39.37" y1="42.5704" x2="39.37" y2="56.505" width="0" layer="20"/>
 <wire x1="39.37" y1="56.505" x2="0" y2="56.505" width="0" layer="20"/>
 <wire x1="0" y1="56.505" x2="0" y2="1.27" width="0" layer="20"/>
-<text x="9.5504" y="37.9984" size="5.08" layer="1" font="vector" ratio="12" rot="SR270">RASOR</text>
+<text x="6.7056" y="26.8224" size="2.54" layer="1" font="vector" ratio="12" rot="SR270" align="center">shield</text>
 </plain>
 <attributes>
@@
 <wire x1="22.5806" y1="6.7454" x2="22.5806" y2="6.6247" width="0.3048" layer="16"/>
 <wire x1="22.5806" y1="7.355" x2="22.5806" y2="6.7454" width="0.3048" layer="16"/>
-<wire x1="21.8573" y1="37.5412" x2="23.1394" y2="37.5412" width="0.3048" layer="1"/>
-<wire x1="3.6243" y1="50.8" x2="3.6243" y2="50.6645" width="0.3048" layer="1"/>
-<wire x1="3.6243" y1="50.6645" x2="16.7476" y2="37.5412" width="0.3048" layer="1"/>
-<wire x1="16.7476" y1="37.5412" x2="21.8573" y2="37.5412" width="0.3048" layer="1"/>
-<wire x1="21.8573" y1="37.5412" x2="21.8573" y2="23.5833" width="0.3048" layer="1"/>
-<wire x1="21.8573" y1="23.5833" x2="23.1394" y2="22.3012" width="0.3048" layer="1"/>
-<wire x1="2.54" y1="50.8" x2="3.6243" y2="50.8" width="0.3048" layer="1"/>
 <wire x1="22.4392" y1="3.81" x2="21.7089" y2="3.81" width="0.3048" layer="16"/>
+<wire x1="23.1394" y1="22.3012" x2="23.1394" y2="27.4066" width="0.3048" layer="16"/>
+<wire x1="23.1394" y1="27.4066" x2="25.4" y2="29.6672" width="0.3048" layer="16"/>
+<wire x1="25.4" y1="29.6672" x2="25.4" y2="35.2806" width="0.3048" layer="16"/>
+<wire x1="25.4" y1="35.2806" x2="23.1394" y2="37.5412" width="0.3048" layer="16"/>
+<wire x1="23.1394" y1="37.5412" x2="23.1394" y2="42.0878" width="0.3048" layer="1"/>
+<wire x1="23.1394" y1="42.0878" x2="23.1394" y2="47.9806" width="0.3048" layer="1"/>
+<wire x1="23.1394" y1="47.9806" x2="21.9456" y2="49.1744" width="0.3048" layer="1"/>
+<wire x1="21.9456" y1="49.1744" x2="4.1656" y2="49.1744" width="0.3048" layer="1"/>
+<wire x1="4.1656" y1="49.1744" x2="2.54" y2="50.8" width="0.3048" layer="1"/>
 </signal>
 <signal name="GND">
@@
 <vertex x="-1.2192" y="57.5056"/>
 </polygon>
-<via x="2.4384" y="14.8336" extent="1-16" drill="0.6" shape="square"/>
+<via x="2.4384" y="15.4432" extent="1-16" drill="0.6" shape="square"/>
 <via x="24.384" y="4.064" extent="1-16" drill="0.6" shape="square"/>
 <via x="43.0784" y="27.8384" extent="1-16" drill="0.6" shape="square"/>
@@
 <via x="38.608" y="15.6464" extent="1-16" drill="0.6" shape="square"/>
 <via x="24.5872" y="10.9728" extent="1-16" drill="0.6" shape="square"/>
-<via x="5.8928" y="46.1264" extent="1-16" drill="0.6" shape="square"/>
+<via x="9.9568" y="11.176" extent="1-16" drill="0.6" shape="square"/>
 <wire x1="15.6972" y1="8.2042" x2="14.3002" y2="8.2042" width="0.3048" layer="16"/>
 <wire x1="14.3002" y1="8.2042" x2="13.5382" y2="7.4422" width="0.3048" layer="16"/>
@@
 <wire x1="17.0688" y1="8.5344" x2="17.0688" y2="11.176" width="0.3048" layer="16"/>
 <via x="46.9392" y="14.6304" extent="1-16" drill="0.6" shape="square"/>
+<via x="2.4384" y="47.752" extent="1-16" drill="0.6" shape="square"/>
 </signal>
 <signal name="N$3">
@@
 <contactref element="U1" pad="13"/>
 <contactref element="U$3" pad="22"/>
-<wire x1="46.92" y1="24.92" x2="48.3503" y2="24.92" width="0.3048" layer="16"/>
-<wire x1="48.3503" y1="24.92" x2="48.8351" y2="25.4048" width="0.3048" layer="16"/>
-<wire x1="48.8351" y1="25.4048" x2="48.8351" y2="37.3438" width="0.3048" layer="16"/>
-<wire x1="48.8351" y1="37.3438" x2="44.2568" y2="41.9221" width="0.3048" layer="16"/>
 <wire x1="31.5644" y1="50.5043" x2="31.5644" y2="51.2872" width="0.3048" layer="16"/>
 <wire x1="31.5644" y1="51.2872" x2="30.7816" y2="52.07" width="0.3048" layer="16"/>
 <wire x1="30.7816" y1="52.07" x2="29.21" y2="52.07" width="0.3048" layer="16"/>
 <wire x1="29.21" y1="52.07" x2="27.94" y2="53.34" width="0.3048" layer="16"/>
-<wire x1="37.7323" y1="42.1253" x2="33.7312" y2="46.1264" width="0.3048" layer="16"/>
+<wire x1="37.7323" y1="42.1253" x2="37.592" y2="42.2656" width="0.3048" layer="16"/>
+<wire x1="37.592" y1="42.2656" x2="33.7312" y2="46.1264" width="0.3048" layer="16"/>
 <wire x1="31.5644" y1="50.5043" x2="31.5644" y2="48.2932" width="0.3048" layer="16"/>
 <wire x1="31.5644" y1="48.2932" x2="33.7312" y2="46.1264" width="0.3048" layer="16"/>
-<wire x1="44.2568" y1="41.9221" x2="37.9355" y2="41.9221" width="0.3048" layer="16"/>
 <wire x1="37.9355" y1="41.9221" x2="37.7323" y2="42.1253" width="0.3048" layer="16"/>
+<wire x1="40.4368" y1="39.4208" x2="37.592" y2="42.2656" width="0.3048" layer="16"/>
+<wire x1="46.92" y1="24.92" x2="48.288" y2="24.92" width="0.3048" layer="16"/>
+<wire x1="48.288" y1="24.92" x2="49.1744" y2="25.8064" width="0.3048" layer="16"/>
+<wire x1="40.4368" y1="39.4208" x2="47.1424" y2="39.4208" width="0.3048" layer="16"/>
+<wire x1="47.1424" y1="39.4208" x2="49.1744" y2="37.3888" width="0.3048" layer="16"/>
+<wire x1="49.1744" y1="37.3888" x2="49.1744" y2="26.2128" width="0.3048" layer="16"/>
+<wire x1="49.1744" y1="26.2128" x2="49.1744" y2="25.8064" width="0.3048" layer="16"/>
 </signal>
 <signal name="N$8">
@@
 <contactref element="U1" pad="18"/>
 <contactref element="U$3" pad="23"/>
-<wire x1="46.92" y1="28.42" x2="48.3503" y2="28.42" width="0.3048" layer="16"/>
-<wire x1="48.3503" y1="28.42" x2="48.3503" y2="37.1458" width="0.3048" layer="16"/>
-<wire x1="48.3503" y1="37.1458" x2="44.2265" y2="41.2696" width="0.3048" layer="16"/>
-<wire x1="44.2265" y1="41.2696" x2="40.0104" y2="41.2696" width="0.3048" layer="16"/>
-<wire x1="40.0104" y1="41.2696" x2="37.3688" y2="41.2696" width="0.3048" layer="16"/>
 <wire x1="37.3688" y1="41.2696" x2="30.48" y2="48.1584" width="0.3048" layer="16"/>
 <wire x1="30.48" y1="48.1584" x2="30.48" y2="50.8" width="0.3048" layer="16"/>
+<wire x1="39.8072" y1="38.8312" x2="37.3688" y2="41.2696" width="0.3048" layer="16"/>
+<wire x1="46.92" y1="28.42" x2="48.3336" y2="28.42" width="0.3048" layer="16"/>
+<wire x1="48.3336" y1="28.42" x2="48.5648" y2="28.448" width="0.3048" layer="16"/>
+<wire x1="48.5648" y1="28.448" x2="48.5648" y2="37.1345" width="0.3048" layer="16"/>
+<wire x1="39.8072" y1="38.8312" x2="46.8681" y2="38.8312" width="0.3048" layer="16"/>
+<wire x1="46.8681" y1="38.8312" x2="48.5648" y2="37.1345" width="0.3048" layer="16"/>
 </signal>
 <signal name="N$4">
@@
 <wire x1="2.54" y1="53.34" x2="3.8204" y2="52.0596" width="0.3048" layer="16"/>
 <wire x1="3.8204" y1="52.0596" x2="3.8608" y2="52.0596" width="0.3048" layer="16"/>
-<wire x1="3.8608" y1="52.0596" x2="3.8608" y2="45.1104" width="0.3048" layer="16"/>
 <wire x1="5.39" y1="6.32" x2="7.112" y2="6.32" width="0.3048" layer="16"/>
 <wire x1="7.112" y1="6.32" x2="7.112" y2="4.064" width="0.3048" layer="16"/>
 <via x="7.112" y="4.064" extent="1-16" drill="0.6096"/>
-<wire x1="7.112" y1="4.064" x2="7.112" y2="42.2656" width="0.3048" layer="1"/>
-<via x="7.112" y="42.2656" extent="1-16" drill="0.6"/>
-<wire x1="7.112" y1="42.2656" x2="3.8608" y2="45.1104" width="0.3048" layer="16"/>
+<via x="7.112" y="10.7696" extent="1-16" drill="0.6"/>
 <wire x1="14.3002" y1="5.2832" x2="14.3002" y2="4.3942" width="0.3048" layer="16"/>
 <wire x1="14.3002" y1="4.3942" x2="15.0368" y2="3.6576" width="0.3048" layer="16"/>
@@
 <wire x1="15.0368" y1="3.6576" x2="7.5184" y2="3.6576" width="0.3048" layer="1"/>
 <wire x1="7.5184" y1="3.6576" x2="7.112" y2="4.064" width="0.3048" layer="1"/>
+<wire x1="3.8608" y1="52.0596" x2="3.8608" y2="45.5168" width="0.3048" layer="16"/>
+<wire x1="7.112" y1="10.7696" x2="7.112" y2="4.064" width="0.3048" layer="1"/>
+<wire x1="3.8608" y1="45.5168" x2="3.8608" y2="14.0208" width="0.3048" layer="16"/>
+<wire x1="3.8608" y1="14.0208" x2="7.112" y2="10.7696" width="0.3048" layer="16"/>
 </signal>
 <signal name="N$10">

Commit message: work on raspi
Routing:
- net GND: vias 12 -> 14
Other:
- board text added: "TREZOR"
Changed lines of the file:
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@@
 <wire x1="0" y1="56.505" x2="0" y2="1.27" width="0" layer="20"/>
 <text x="6.7056" y="26.8224" size="2.54" layer="1" font="vector" ratio="12" rot="SR270" align="center">shield</text>
+<text x="10.5664" y="27.0256" size="2.54" layer="1" font="vector" ratio="12" rot="SR270" align="center">TREZOR</text>
 </plain>
 <attributes>
@@
 <via x="46.9392" y="14.6304" extent="1-16" drill="0.6" shape="square"/>
 <via x="2.4384" y="47.752" extent="1-16" drill="0.6" shape="square"/>
+<via x="27.432" y="26.8224" extent="1-16" drill="0.6" shape="square"/>
+<via x="19.7104" y="28.6512" extent="1-16" drill="0.6" shape="square"/>
 </signal>
 <signal name="N$3">
@@
 <wire x1="30.7816" y1="52.07" x2="29.21" y2="52.07" width="0.3048" layer="16"/>
 <wire x1="29.21" y1="52.07" x2="27.94" y2="53.34" width="0.3048" layer="16"/>
-<wire x1="37.7323" y1="42.1253" x2="37.592" y2="42.2656" width="0.3048" layer="16"/>
-<wire x1="37.592" y1="42.2656" x2="33.7312" y2="46.1264" width="0.3048" layer="16"/>
-<wire x1="31.5644" y1="50.5043" x2="31.5644" y2="48.2932" width="0.3048" layer="16"/>
-<wire x1="31.5644" y1="48.2932" x2="33.7312" y2="46.1264" width="0.3048" layer="16"/>
-<wire x1="37.9355" y1="41.9221" x2="37.7323" y2="42.1253" width="0.3048" layer="16"/>
-<wire x1="40.4368" y1="39.4208" x2="37.592" y2="42.2656" width="0.3048" layer="16"/>
+<wire x1="31.5644" y1="50.5043" x2="31.5644" y2="47.6836" width="0.3048" layer="16"/>
 <wire x1="46.92" y1="24.92" x2="48.288" y2="24.92" width="0.3048" layer="16"/>
 <wire x1="48.288" y1="24.92" x2="49.1744" y2="25.8064" width="0.3048" layer="16"/>
-<wire x1="40.4368" y1="39.4208" x2="47.1424" y2="39.4208" width="0.3048" layer="16"/>
+<wire x1="39.8272" y1="39.4208" x2="47.1424" y2="39.4208" width="0.3048" layer="16"/>
 <wire x1="47.1424" y1="39.4208" x2="49.1744" y2="37.3888" width="0.3048" layer="16"/>
 <wire x1="49.1744" y1="37.3888" x2="49.1744" y2="26.2128" width="0.3048" layer="16"/>
 <wire x1="49.1744" y1="26.2128" x2="49.1744" y2="25.8064" width="0.3048" layer="16"/>
+<wire x1="39.8272" y1="39.4208" x2="31.5644" y2="47.6836" width="0.3048" layer="16"/>
 </signal>
 <signal name="N$8">
@@
 <contactref element="U1" pad="18"/>
 <contactref element="U$3" pad="23"/>
-<wire x1="37.3688" y1="41.2696" x2="30.48" y2="48.1584" width="0.3048" layer="16"/>
-<wire x1="30.48" y1="48.1584" x2="30.48" y2="50.8" width="0.3048" layer="16"/>
-<wire x1="39.8072" y1="38.8312" x2="37.3688" y2="41.2696" width="0.3048" layer="16"/>
+<wire x1="30.48" y1="47.752" x2="30.48" y2="50.8" width="0.3048" layer="16"/>
 <wire x1="46.92" y1="28.42" x2="48.3336" y2="28.42" width="0.3048" layer="16"/>
 <wire x1="48.3336" y1="28.42" x2="48.5648" y2="28.448" width="0.3048" layer="16"/>
 <wire x1="48.5648" y1="28.448" x2="48.5648" y2="37.1345" width="0.3048" layer="16"/>
-<wire x1="39.8072" y1="38.8312" x2="46.8681" y2="38.8312" width="0.3048" layer="16"/>
+<wire x1="39.4008" y1="38.8312" x2="46.8681" y2="38.8312" width="0.3048" layer="16"/>
 <wire x1="46.8681" y1="38.8312" x2="48.5648" y2="37.1345" width="0.3048" layer="16"/>
+<wire x1="30.48" y1="47.752" x2="39.4008" y2="38.8312" width="0.3048" layer="16"/>
 </signal>
 <signal name="N$4">

Commit message: work on rpi
Parts:
- added C9: 4.7uF, SparkFun-Capacitors:0805
- U1: value (none) -> DISPLAY
Connections:
- removed net N$18: C6.2, U2.7
- new net N$14: C9.2, U2.16
- net +5V: now also C6.2, U2.7
- net GND: now also C9.1
- net N$16: now also U$3.10; no longer U$3.8
- net N$17: now also U$3.8; no longer U$3.10
Routing:
- net +5V: track 65.7 -> 84.9 mm, vias 3 -> 5
- net N$18: track 13.6 -> 0.00 mm, vias 2 -> 0
- net N$14: track 0.00 -> 4.48 mm
- net N$17: track 50.2 -> 45.8 mm
- net N$20: track 9.93 -> 9.36 mm
Changed lines of the file:
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@@
 <elements>
 <element name="U$2" library="SparkFun-Connectors" package="USB-AB-MICRO-SMD" value="USB_AB" x="2.54" y="7.62" rot="MR180"/>
-<element name="U1" library="microbuilder" package="UG-2864HSWEG01_0.96IN_WRAPAROUND" value="" x="45.72" y="26.67" rot="R90"/>
+<element name="U1" library="microbuilder" package="UG-2864HSWEG01_0.96IN_WRAPAROUND" value="DISPLAY" x="45.72" y="26.67" rot="R90"/>
 <element name="S1" library="SparkFun-Electromechanical" package="TACTILE-PTH" value="SWITCH-MOMENTARY-2PTH" x="25.4" y="34.29" rot="R270"/>
 <element name="S2" library="SparkFun-Electromechanical" package="TACTILE-PTH" value="SWITCH-MOMENTARY-2PTH" x="25.4" y="19.05" rot="R270"/>
@@
 <element name="C7" library="SparkFun-Capacitors" package="0805" value="1uF" x="26.3906" y="8.255" rot="MR270"/>
 <element name="C8" library="SparkFun-Capacitors" package="0805" value="0.1uF" x="22.5806" y="8.255" rot="MR270"/>
+<element name="C9" library="SparkFun-Capacitors" package="0805" value="4.7uF" x="10.16" y="11.9888" rot="MR270"/>
 </elements>
 <signals>
@@
 <via x="38.608" y="15.6464" extent="1-16" drill="0.6" shape="square"/>
 <via x="24.5872" y="10.9728" extent="1-16" drill="0.6" shape="square"/>
-<via x="9.9568" y="11.176" extent="1-16" drill="0.6" shape="square"/>
+<via x="10.16" y="14.8336" extent="1-16" drill="0.6" shape="square"/>
 <wire x1="15.6972" y1="8.2042" x2="14.3002" y2="8.2042" width="0.3048" layer="16"/>
 <wire x1="14.3002" y1="8.2042" x2="13.5382" y2="7.4422" width="0.3048" layer="16"/>
@@
 <via x="27.432" y="26.8224" extent="1-16" drill="0.6" shape="square"/>
 <via x="19.7104" y="28.6512" extent="1-16" drill="0.6" shape="square"/>
+<contactref element="C9" pad="1"/>
 </signal>
 <signal name="N$3">
@@
 <contactref element="U$2" pad="VBUS"/>
 <contactref element="U$3" pad="2"/>
-<contactref element="U2" pad="8"/>
 <wire x1="4.8749" y1="6.32" x2="5.39" y2="6.32" width="0.3048" layer="16"/>
 <wire x1="2.54" y1="53.34" x2="3.8204" y2="52.0596" width="0.3048" layer="16"/>
@@
 <via x="7.112" y="4.064" extent="1-16" drill="0.6096"/>
 <via x="7.112" y="10.7696" extent="1-16" drill="0.6"/>
-<wire x1="14.3002" y1="5.2832" x2="14.3002" y2="4.3942" width="0.3048" layer="16"/>
-<wire x1="14.3002" y1="4.3942" x2="15.0368" y2="3.6576" width="0.3048" layer="16"/>
-<via x="15.0368" y="3.6576" extent="1-16" drill="0.6096"/>
-<wire x1="15.0368" y1="3.6576" x2="7.5184" y2="3.6576" width="0.3048" layer="1"/>
-<wire x1="7.5184" y1="3.6576" x2="7.112" y2="4.064" width="0.3048" layer="1"/>
+<via x="16.4592" y="4.064" extent="1-16" drill="0.6096"/>
 <wire x1="3.8608" y1="52.0596" x2="3.8608" y2="45.5168" width="0.3048" layer="16"/>
 <wire x1="7.112" y1="10.7696" x2="7.112" y2="4.064" width="0.3048" layer="1"/>
-<wire x1="3.8608" y1="45.5168" x2="3.8608" y2="14.0208" width="0.3048" layer="16"/>
+<wire x1="3.8608" y1="45.5168" x2="3.8608" y2="14.224" width="0.3048" layer="16"/>
+<wire x1="3.8608" y1="14.224" x2="3.8608" y2="14.0208" width="0.3048" layer="16"/>
 <wire x1="3.8608" y1="14.0208" x2="7.112" y2="10.7696" width="0.3048" layer="16"/>
+<wire x1="20.6749" y1="7.158" x2="21.6022" y2="8.0853" width="0.3048" layer="16"/>
+<wire x1="21.6022" y1="8.0853" x2="24.4856" y2="8.0853" width="0.3048" layer="16"/>
+<via x="20.6749" y="7.158" extent="1-16" drill="0.6096" diameter="1.016"/>
+<via x="7.1954" y="15.3653" extent="1-16" drill="0.6096" diameter="1.016"/>
+<wire x1="20.6749" y1="7.158" x2="20.6749" y2="5.8413" width="0.3048" layer="1"/>
+<wire x1="20.6749" y1="5.8413" x2="19.9136" y2="5.08" width="0.3048" layer="1"/>
+<wire x1="7.112" y1="4.064" x2="16.4592" y2="4.064" width="0.3048" layer="1"/>
+<wire x1="16.4592" y1="4.064" x2="18.8976" y2="4.064" width="0.3048" layer="1"/>
+<wire x1="18.8976" y1="4.064" x2="19.9136" y2="5.08" width="0.3048" layer="1"/>
+<wire x1="14.7828" y1="4.7244" x2="15.4432" y2="4.064" width="0.3048" layer="16"/>
+<wire x1="15.4432" y1="4.064" x2="16.4592" y2="4.064" width="0.3048" layer="16"/>
+<wire x1="14.3002" y1="4.5974" x2="14.8336" y2="4.064" width="0.3048" layer="16"/>
+<wire x1="14.8336" y1="4.064" x2="16.4592" y2="4.064" width="0.3048" layer="16"/>
+<contactref element="U2" pad="8"/>
+<contactref element="U2" pad="7"/>
+<contactref element="C6" pad="2"/>
+<wire x1="14.783" y1="5.2832" x2="14.7828" y2="5.2832" width="0.3046" layer="16"/>
+<wire x1="14.3002" y1="5.2832" x2="14.3002" y2="4.5974" width="0.3048" layer="16"/>
+<wire x1="14.7828" y1="5.2832" x2="14.7828" y2="4.7244" width="0.3048" layer="16"/>
+<wire x1="7.1954" y1="15.3653" x2="5.0021" y2="15.3653" width="0.3048" layer="16"/>
+<wire x1="5.0021" y1="15.3653" x2="3.8608" y2="14.224" width="0.3048" layer="16"/>
+<wire x1="24.4856" y1="8.0853" x2="24.4856" y2="7.355" width="0" layer="19" extent="16-16"/>
 </signal>
 <signal name="N$10">
@@
 <signal name="N$16">
 <contactref element="U2" pad="21"/>
-<contactref element="U$3" pad="8"/>
-<wire x1="13.2842" y1="9.6012" x2="13.2842" y2="28.571" width="0.3048" layer="16"/>
-<wire x1="13.2842" y1="28.571" x2="11.43" y2="30.4252" width="0.3048" layer="16"/>
-<wire x1="11.43" y1="30.4252" x2="11.43" y2="52.07" width="0.3048" layer="16"/>
-<wire x1="11.43" y1="52.07" x2="10.16" y2="53.34" width="0.3048" layer="16"/>
+<wire x1="13.2842" y1="9.6012" x2="13.2842" y2="48.2814" width="0.3048" layer="16"/>
+<wire x1="13.2842" y1="48.2814" x2="11.43" y2="50.1356" width="0.3048" layer="16"/>
+<contactref element="U$3" pad="10"/>
+<wire x1="11.43" y1="50.1356" x2="11.43" y2="52.07" width="0.3048" layer="16"/>
+<wire x1="11.43" y1="52.07" x2="12.7" y2="53.34" width="0.3048" layer="16"/>
 </signal>
 <signal name="N$17">
 <contactref element="U2" pad="20"/>
-<contactref element="U$3" pad="10"/>
-<wire x1="12.7764" y1="9.6012" x2="12.7764" y2="26.1503" width="0.3048" layer="16"/>
-<wire x1="12.7764" y1="26.1503" x2="9.0319" y2="29.8948" width="0.3048" layer="16"/>
-<wire x1="9.0319" y1="29.8948" x2="9.0319" y2="53.8392" width="0.3048" layer="16"/>
-<wire x1="9.0319" y1="53.8392" x2="9.6361" y2="54.4434" width="0.3048" layer="16"/>
-<wire x1="9.6361" y1="54.4434" x2="11.5966" y2="54.4434" width="0.3048" layer="16"/>
-<wire x1="11.5966" y1="54.4434" x2="12.7" y2="53.34" width="0.3048" layer="16"/>
+<wire x1="12.7764" y1="9.6012" x2="12.7764" y2="45.8607" width="0.3048" layer="16"/>
 <wire x1="12.7764" y1="9.6012" x2="12.7762" y2="9.6012" width="0.3046" layer="16"/>
-</signal>
-<signal name="N$18">
-<contactref element="U2" pad="7"/>
-<contactref element="C6" pad="2"/>
-<wire x1="24.4856" y1="7.355" x2="24.4856" y2="8.0853" width="0.3048" layer="16"/>
-<wire x1="20.6749" y1="7.158" x2="21.6022" y2="8.0853" width="0.3048" layer="16"/>
-<wire x1="21.6022" y1="8.0853" x2="24.4856" y2="8.0853" width="0.3048" layer="16"/>
-<via x="20.6749" y="7.158" extent="1-16" drill="0.6096" diameter="1.016"/>
-<via x="17.1522" y="3.7829" extent="1-16" drill="0.6096" diameter="1.016"/>
-<wire x1="14.783" y1="5.2832" x2="14.7828" y2="5.2832" width="0.3046" layer="16"/>
-<wire x1="17.1522" y1="3.7829" x2="18.6165" y2="3.7829" width="0.3048" layer="1"/>
-<wire x1="18.6165" y1="3.7829" x2="19.9136" y2="5.08" width="0.3048" layer="1"/>
-<wire x1="20.6749" y1="7.158" x2="20.6749" y2="5.8413" width="0.3048" layer="1"/>
-<wire x1="20.6749" y1="5.8413" x2="19.9136" y2="5.08" width="0.3048" layer="1"/>
-<wire x1="14.783" y1="5.2832" x2="15.6519" y2="5.2832" width="0.3048" layer="16"/>
-<wire x1="15.6519" y1="5.2832" x2="17.1522" y2="3.7829" width="0.3048" layer="16"/>
+<contactref element="U$3" pad="8"/>
+<wire x1="12.7764" y1="45.8607" x2="12.7764" y2="46.1516" width="0.3048" layer="16"/>
+<wire x1="12.7764" y1="46.1516" x2="8.9408" y2="49.9872" width="0.3048" layer="16"/>
+<wire x1="8.9408" y1="49.9872" x2="8.9408" y2="52.1208" width="0.3048" layer="16"/>
+<wire x1="8.9408" y1="52.1208" x2="10.16" y2="53.34" width="0.3048" layer="16"/>
 </signal>
 <signal name="N$20">
@@
 <contactref element="R2" pad="2"/>
 <wire x1="20.6392" y1="3.81" x2="19.9089" y2="3.81" width="0.3048" layer="16"/>
-<wire x1="18.6258" y1="2.5269" x2="19.9089" y2="3.81" width="0.3048" layer="16"/>
-<wire x1="13.7922" y1="5.2832" x2="13.7922" y2="2.8702" width="0.3048" layer="16"/>
-<wire x1="18.6258" y1="2.5269" x2="14.1355" y2="2.5269" width="0.3048" layer="16"/>
-<wire x1="14.1355" y1="2.5269" x2="13.7922" y2="2.8702" width="0.3048" layer="16"/>
+<wire x1="19.0322" y1="2.9333" x2="19.9089" y2="3.81" width="0.3048" layer="16"/>
+<wire x1="13.7922" y1="5.2832" x2="13.7922" y2="3.2766" width="0.3048" layer="16"/>
+<wire x1="19.0322" y1="2.9333" x2="14.1355" y2="2.9333" width="0.3048" layer="16"/>
+<wire x1="14.1355" y1="2.9333" x2="13.7922" y2="3.2766" width="0.3048" layer="16"/>
+</signal>
+<signal name="N$14">
+<contactref element="U2" pad="16"/>
+<contactref element="C9" pad="2"/>
+<wire x1="11.3792" y1="7.6962" x2="10.3886" y2="7.6962" width="0.3048" layer="16"/>
+<wire x1="10.3886" y1="7.6962" x2="10.16" y2="7.9248" width="0.3048" layer="16"/>
+<wire x1="10.16" y1="7.9248" x2="10.16" y2="11.0888" width="0.3048" layer="16"/>
 </signal>
 </signals>

Commit message: wip
Parts:
- C5: value 1uF -> 2.2uF
- R1: value 390k/560k -> 390k
- moved C4 8.75 mm to (42.4, 21.9), turned to 90 degrees
- moved C2 7.09 mm to (43.1, 14.9)
- moved C3 6.68 mm to (44.1, 22.0), turned to 90 degrees
- moved C1 2.44 mm to (43.1, 17.9)
Connections:
- net +3V3: now also U1.6
- net N$10: now also C2.1; no longer C1.1
- net N$11: now also C1.1; no longer C2.1
- net N$12: now also C2.2; no longer C1.2
- net N$13: now also C1.2; no longer C2.2
Routing:
- net N$13: track 7.59 -> 4.16 mm
- net N$11: track 7.57 -> 4.50 mm
- net N$12: track 7.02 -> 5.18 mm
- net +5V: track 84.9 -> 85.6 mm
