File: raspi.brd (EAGLE design)
At the start: 53.3 x 55.2 mm, 17 parts, among them U1 DISPLAY, U2 CP2110-F01-GM

Commit message: raspi work
Parts:
- S1, S2: value SWITCH-MOMENTARY-2PTH -> SWITCH-MOMENTARY-2; device SparkFun-Electromechanical:TACTILE-PTH -> SparkFun-Electromechanical:TACTILE_SWITCH_TALL
- moved S1 0.10 mm to (25.4, 34.2), turned to 90 degrees
- moved S2 0.10 mm to (25.4, 19.2), turned to 90 degrees
Connections:
- net +3V3: now also S1.B2, S2.B2; no longer S1.3, S2.3
- net N$2: now also S2.A2; no longer S2.1
- net N$3: now also S1.A2; no longer S1.1
Routing:
- net +3V3: track 107.1 -> 115.9 mm, vias 0 -> 1
- net N$2: track 33.3 -> 37.5 mm
- net N$3: track 17.0 -> 19.9 mm
- net +5V: track 85.6 -> 83.7 mm, vias 5 -> 4
- net GND: track 6.70 -> 6.29 mm, vias 14 -> 16
Other:
- board text removed: "TREZOR"
- board text removed: "shield"

Commit message: raspi work
Parts:
- moved R2 2.03 mm to (19.5, 3.81)
- moved C7 1.42 mm to (25.0, 8.26)
- moved C6 1.22 mm to (23.3, 8.26)
- moved C8 1.02 mm to (21.6, 8.26)
- moved R1 0.10 mm to (40.6, 29.1)
Routing:
- net +3V3: track 115.9 -> 119.4 mm
- net N$20: track 9.36 -> 7.33 mm
- net USB_D_P: track 18.1 -> 16.4 mm
- net USB_D_N: track 17.9 -> 16.2 mm
- net +5V: track 83.7 -> 82.1 mm
- net N$17: track 45.8 -> 44.8 mm
- net N$16: track 45.0 -> 44.5 mm
Other:
- board text added: "bitcointrezor.com"

Commit message: rework BOMs
Parts:
- removed U$2: USB_AB, SparkFun-Connectors:USB-AB-MICRO-SMD
- added USB: (no value), fabhack:MOLEX_47346-0001
Connections:
- net +5V: now also USB.1; no longer U$2.VBUS
- net GND: now also USB.5; no longer U$2.GND
- net USB_D_N: now also USB.2; no longer U$2.D-
- net USB_D_P: now also USB.3; no longer U$2.D+
Routing:
- net GND: track 5.87 -> 10.7 mm
- net +5V: track 82.1 -> 80.0 mm
- net USB_D_P: track 16.4 -> 17.4 mm
- net USB_D_N: track 16.2 -> 17.3 mm
Changed lines of the file:
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@@
 <layer number="54" name="bGND_GNDA" color="1" fill="9" visible="no" active="no"/>
 <layer number="56" name="wert" color="7" fill="1" visible="no" active="no"/>
+<layer number="59" name="tCarbon" color="7" fill="1" visible="yes" active="yes"/>
+<layer number="60" name="bCarbon" color="7" fill="1" visible="yes" active="yes"/>
 <layer number="91" name="Nets" color="2" fill="1" visible="no" active="no"/>
 <layer number="92" name="Busses" color="1" fill="1" visible="no" active="no"/>
@@
 <layer number="121" name="sName" color="7" fill="1" visible="yes" active="yes"/>
 <layer number="122" name="_bPlace" color="7" fill="1" visible="yes" active="yes"/>
+<layer number="123" name="tTestmark" color="7" fill="1" visible="yes" active="yes"/>
+<layer number="124" name="bTestmark" color="7" fill="1" visible="yes" active="yes"/>
 <layer number="125" name="_tNames" color="7" fill="1" visible="yes" active="yes"/>
 <layer number="126" name="_bNames" color="7" fill="1" visible="yes" active="yes"/>
 <layer number="127" name="_tValues" color="7" fill="1" visible="yes" active="yes"/>
 <layer number="128" name="_bValues" color="7" fill="1" visible="yes" active="yes"/>
+<layer number="129" name="Mask" color="7" fill="1" visible="yes" active="yes"/>
+<layer number="131" name="tAdjust" color="7" fill="1" visible="yes" active="yes"/>
+<layer number="132" name="bAdjust" color="7" fill="1" visible="yes" active="yes"/>
 <layer number="144" name="Drill_legend" color="7" fill="1" visible="yes" active="yes"/>
 <layer number="151" name="HeatSink" color="7" fill="1" visible="yes" active="yes"/>
@@
 </autorouter>
 <elements>
-<element name="U$2" library="SparkFun-Connectors" package="USB-AB-MICRO-SMD" value="USB_AB" x="2.54" y="7.62" rot="MR180"/>
+<element name="USB" library="fabhack" package="MOLEX_47346-0001" value="" x="4.3688" y="7.62" rot="MR90">
+<attribute name="PACKAGE" value="5 POS MICRO USB R/A" x="4.3688" y="7.62" size="1.778" layer="28" rot="MR90" display="off"/>
+<attribute name="OC_NEWARK" value="47M0505" x="4.3688" y="7.62" size="1.778" layer="28" rot="MR90" display="off"/>
+<attribute name="MPN" value="47346-0001" x="4.3688" y="7.62" size="1.778" layer="28" rot="MR90" display="off"/>
+<attribute name="SUPPLIER" value="MOLEX" x="4.3688" y="7.62" size="1.778" layer="28" rot="MR90" display="off"/>
+<attribute name="OC_FARNELL" value="1568026" x="4.3688" y="7.62" size="1.778" layer="28" rot="MR90" display="off"/>
+</element>
 <element name="U1" library="microbuilder" package="UG-2864HSWEG01_0.96IN_WRAPAROUND" value="DISPLAY" x="45.72" y="26.67" rot="R90"/>
 <element name="S1" library="SparkFun-Electromechanical" package="TACTILE_SWITCH_TALL" value="SWITCH-MOMENTARY-2" x="25.4" y="34.1884" rot="R90"/>
@@
 </signal>
 <signal name="GND">
-<contactref element="U$2" pad="GND"/>
+<contactref element="USB" pad="5"/>
 <contactref element="U1" pad="1"/>
 <contactref element="U2" pad="25"/>
@@
 <vertex x="-1.2192" y="57.5056"/>
 </polygon>
-<via x="2.2352" y="14.6304" extent="1-16" drill="0.6" shape="square"/>
+<via x="5.8928" y="12.192" extent="1-16" drill="0.6" shape="square"/>
 <via x="23.5712" y="4.2672" extent="1-16" drill="0.6" shape="square"/>
 <via x="43.2816" y="27.8384" extent="1-16" drill="0.6" shape="square"/>
@@
 <wire x1="15.6972" y1="8.2042" x2="16.6624" y2="8.2042" width="0.3048" layer="16"/>
 <wire x1="16.6624" y1="8.2042" x2="16.6624" y2="10.5664" width="0.3048" layer="16"/>
+<wire x1="4.3688" y1="8.92" x2="5.8928" y2="8.92" width="0.3048" layer="16"/>
+<wire x1="5.8928" y1="8.92" x2="5.8928" y2="12.192" width="0.3048" layer="16"/>
 </signal>
 <signal name="N$3">
@@
 </signal>
 <signal name="+5V">
-<contactref element="U$2" pad="VBUS"/>
+<contactref element="USB" pad="1"/>
 <contactref element="U$3" pad="2"/>
-<wire x1="4.8749" y1="6.32" x2="5.39" y2="6.32" width="0.3048" layer="16"/>
-<wire x1="2.54" y1="53.34" x2="3.8204" y2="52.0596" width="0.3048" layer="16"/>
-<wire x1="3.8204" y1="52.0596" x2="3.8608" y2="52.0596" width="0.3048" layer="16"/>
-<wire x1="5.39" y1="6.32" x2="7.112" y2="6.32" width="0.3048" layer="16"/>
-<wire x1="7.112" y1="6.32" x2="7.112" y2="4.064" width="0.3048" layer="16"/>
-<via x="7.112" y="4.064" extent="1-16" drill="0.6096"/>
-<via x="7.112" y="10.7696" extent="1-16" drill="0.6"/>
 <via x="16.4592" y="4.064" extent="1-16" drill="0.6096"/>
-<wire x1="3.8608" y1="52.0596" x2="3.8608" y2="45.5168" width="0.3048" layer="16"/>
-<wire x1="7.112" y1="10.7696" x2="7.112" y2="4.064" width="0.3048" layer="1"/>
 <via x="19.6589" y="7.3612" extent="1-16" drill="0.6096" diameter="1.016"/>
-<wire x1="7.112" y1="4.064" x2="16.4592" y2="4.064" width="0.3048" layer="1"/>
 <wire x1="14.7828" y1="4.7244" x2="15.4432" y2="4.064" width="0.3048" layer="16"/>
 <wire x1="15.4432" y1="4.064" x2="16.4592" y2="4.064" width="0.3048" layer="16"/>
@@
 <wire x1="16.4592" y1="4.064" x2="19.6589" y2="4.064" width="0.3048" layer="1"/>
 <wire x1="19.6589" y1="4.064" x2="19.6589" y2="7.3612" width="0.3048" layer="1"/>
-<wire x1="3.8608" y1="45.5168" x2="3.8608" y2="17.8816" width="0.3048" layer="16"/>
-<wire x1="3.8608" y1="17.8816" x2="7.112" y2="14.6304" width="0.3048" layer="16"/>
-<wire x1="7.112" y1="14.6304" x2="7.112" y2="10.7696" width="0.3048" layer="16"/>
 <wire x1="19.6589" y1="7.3612" x2="19.6589" y2="7.5685" width="0.3048" layer="16"/>
 <wire x1="19.6589" y1="7.5685" x2="20.32" y2="8.2296" width="0.3048" layer="16"/>
 <wire x1="20.32" y1="8.2296" x2="23.2664" y2="8.2296" width="0.3048" layer="16"/>
 <wire x1="23.2664" y1="8.2296" x2="23.2664" y2="7.355" width="0.3048" layer="16"/>
+<wire x1="2.54" y1="53.34" x2="3.8608" y2="52.0192" width="0.3048" layer="16"/>
+<wire x1="3.8608" y1="52.0192" x2="3.8608" y2="17.8816" width="0.3048" layer="16"/>
+<wire x1="3.8608" y1="17.8816" x2="7.112" y2="14.6304" width="0.3048" layer="16"/>
+<wire x1="7.112" y1="14.6304" x2="7.112" y2="9.5504" width="0.3048" layer="16"/>
+<via x="7.112" y="9.5504" extent="1-16" drill="0.6096"/>
+<wire x1="7.112" y1="9.5504" x2="7.112" y2="5.2832" width="0.3048" layer="1"/>
+<via x="7.112" y="5.2832" extent="1-16" drill="0.6096"/>
+<wire x1="7.112" y1="5.2832" x2="8.3312" y2="4.064" width="0.3048" layer="1"/>
+<wire x1="8.3312" y1="4.064" x2="16.4592" y2="4.064" width="0.3048" layer="1"/>
+<wire x1="4.3688" y1="6.32" x2="6.0752" y2="6.32" width="0.3048" layer="16"/>
+<wire x1="6.0752" y1="6.32" x2="7.112" y2="5.2832" width="0.3048" layer="16"/>
 </signal>
 <signal name="N$10">
@@
 </signal>
 <signal name="USB_D_N">
-<contactref element="U$2" pad="D-"/>
+<contactref element="USB" pad="2"/>
 <contactref element="U2" pad="4"/>
 <via x="17.6784" y="6.096" extent="1-16" drill="0.6096" diameter="1.016"/>
@@
 <wire x1="17.6784" y1="7.1882" x2="17.6784" y2="6.096" width="0.3048" layer="16"/>
 <wire x1="8.9408" y1="6.096" x2="17.6784" y2="6.096" width="0.3048" layer="1"/>
-<wire x1="5.39" y1="6.97" x2="8.9408" y2="6.97" width="0.3048" layer="16"/>
+<wire x1="4.3688" y1="6.97" x2="8.9408" y2="6.97" width="0.3048" layer="16"/>
 <wire x1="8.9408" y1="6.97" x2="8.9408" y2="6.096" width="0.3048" layer="16"/>
 </signal>
 <signal name="USB_D_P" airwireshidden="yes">
-<contactref element="U$2" pad="D+"/>
+<contactref element="USB" pad="3"/>
 <contactref element="U2" pad="3"/>
 <via x="17.6784" y="8.7376" extent="1-16" drill="0.6096" diameter="1.016"/>
@@
 <wire x1="17.6784" y1="7.6962" x2="17.6784" y2="8.7376" width="0.3048" layer="16"/>
 <wire x1="8.9408" y1="8.7376" x2="17.6784" y2="8.7376" width="0.3048" layer="1"/>
-<wire x1="5.39" y1="7.62" x2="8.9408" y2="7.62" width="0.3048" layer="16"/>
+<wire x1="4.3688" y1="7.62" x2="8.9408" y2="7.62" width="0.3048" layer="16"/>
 <wire x1="8.9408" y1="7.62" x2="8.9408" y2="8.7376" width="0.3048" layer="16"/>
 </signal>
