File: raspi.brd (EAGLE design)
At the start: 53.3 x 55.2 mm, 17 parts, among them U1 DISPLAY, U2 CP2110-F01-GM

Commit message: logo tDocu->tSilk
Other:
- board size 53.3 x 55.2 mm -> 53.3 x 54.8 mm
Changed lines of the file:
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@@
 <wire x1="53.34" y1="1.27" x2="53.34" y2="42.5704" width="0" layer="20"/>
 <wire x1="53.34" y1="42.5704" x2="39.37" y2="42.5704" width="0" layer="20"/>
-<wire x1="39.37" y1="42.5704" x2="39.37" y2="56.505" width="0" layer="20"/>
-<wire x1="39.37" y1="56.505" x2="0" y2="56.505" width="0" layer="20"/>
-<wire x1="0" y1="56.505" x2="0" y2="1.27" width="0" layer="20"/>
-<polygon width="0" layer="51">
+<wire x1="39.37" y1="42.5704" x2="39.37" y2="56.0986" width="0" layer="20"/>
+<wire x1="39.37" y1="56.0986" x2="0" y2="56.0986" width="0" layer="20"/>
+<wire x1="0" y1="56.0986" x2="0" y2="1.27" width="0" layer="20"/>
+<polygon width="0" layer="112">
 <vertex x="6.0325" y="20.10448125"/>
 <vertex x="5.2712625" y="20.10448125"/>
@@
 <vertex x="6.0325" y="19.593434375"/>
 </polygon>
-<polygon width="0" layer="51">
+<polygon width="0" layer="112">
 <vertex x="6.0325" y="20.10448125"/>
 <vertex x="6.0325" y="21.13241875"/>
@@
 <vertex x="5.2712625" y="20.10448125"/>
 </polygon>
-<polygon width="0" layer="51">
+<polygon width="0" layer="112">
 <vertex x="6.0825375" y="22.91041875"/>
 <vertex x="5.310378125" y="22.91041875"/>
@@
 <vertex x="6.054853125" y="22.588346875"/>
 </polygon>
-<polygon width="0" layer="51">
+<polygon width="0" layer="112">
 <vertex x="6.0825375" y="22.91041875"/>
 <vertex x="6.054853125" y="23.238334375"/>
@@
 <vertex x="5.310378125" y="22.91041875"/>
 </polygon>
-<polygon width="0" layer="51">
+<polygon width="0" layer="112">
 <vertex x="3.1518875" y="26.853515625"/>
 <vertex x="3.843275" y="26.853515625"/>
@@
 <vertex x="3.1518875" y="24.571834375"/>
 </polygon>
-<polygon width="0" layer="51">
+<polygon width="0" layer="112">
 <vertex x="3.1518875" y="29.2434"/>
 <vertex x="6.034278125" y="29.2434"/>
@@
 <vertex x="3.1518875" y="27.0564625"/>
 </polygon>
-<polygon width="0" layer="51">
+<polygon width="0" layer="112">
 <vertex x="6.0325" y="31.03918125"/>
 <vertex x="5.2712625" y="31.03918125"/>
@@
 <vertex x="6.0325" y="30.528134375"/>
 </polygon>
-<polygon width="0" layer="51">
+<polygon width="0" layer="112">
 <vertex x="6.0325" y="31.03918125"/>
 <vertex x="6.0325" y="32.06711875"/>
@@
 <vertex x="5.2712625" y="31.03918125"/>
 </polygon>
-<polygon width="0" layer="51">
+<polygon width="0" layer="112">
 <vertex x="3.1518875" y="33.910396875"/>
 <vertex x="5.273803125" y="33.910396875"/>
@@
 <vertex x="3.1518875" y="33.0374"/>
 </polygon>
-<polygon width="0" layer="51">
+<polygon width="0" layer="112">
 <vertex x="20.8732125" y="26.77756875"/>
 <vertex x="19.4564" y="26.77756875"/>
@@
 <vertex x="20.8788" y="26.72753125"/>
 </polygon>
-<polygon width="0" layer="51">
+<polygon width="0" layer="112">
 <vertex x="20.8732125" y="26.77756875"/>
 <vertex x="20.812253125" y="27.416634375"/>
@@
 <vertex x="19.4564" y="26.77756875"/>
 </polygon>
-<text x="28.6512" y="3.4544" size="1.6764" layer="51" font="vector" ratio="12">bitcointrezor.com</text>
+<text x="28.6512" y="3.4544" size="1.6764" layer="112" font="vector" ratio="12">bitcointrezor.com</text>
 </plain>
 <attributes>

Commit message: raspi
Parts:
- S1, S2: value SWITCH-MOMENTARY-2 -> SWITCH-MOMENTARY-2SMD; device SparkFun-Electromechanical:TACTILE_SWITCH_TALL -> SparkFun-Electromechanical:TACTILE_SWITCH_SMD
- turned S1 to 270 degrees
- turned S2 to 270 degrees
Connections:
- net +3V3: now also S1.3, S2.3; no longer S1.B2, S2.B2
- net N$2: now also S2.1; no longer S2.A2
- net N$3: now also S1.1; no longer S1.A2
Routing:
- net +3V3: track 119.4 -> 117.4 mm
- net N$3: track 19.9 -> 21.7 mm
- net N$2: track 37.5 -> 39.2 mm
Changed lines of the file:
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@@
 </element>
 <element name="U1" library="microbuilder" package="UG-2864HSWEG01_0.96IN_WRAPAROUND" value="DISPLAY" x="45.72" y="26.67" rot="R90"/>
-<element name="S1" library="SparkFun-Electromechanical" package="TACTILE_SWITCH_TALL" value="SWITCH-MOMENTARY-2" x="25.4" y="34.1884" rot="R90"/>
-<element name="S2" library="SparkFun-Electromechanical" package="TACTILE_SWITCH_TALL" value="SWITCH-MOMENTARY-2" x="25.4" y="19.1516" rot="R90"/>
+<element name="S1" library="SparkFun-Electromechanical" package="TACTILE_SWITCH_SMD" value="SWITCH-MOMENTARY-2SMD" x="25.4" y="34.1884" rot="R270"/>
+<element name="S2" library="SparkFun-Electromechanical" package="TACTILE_SWITCH_SMD" value="SWITCH-MOMENTARY-2SMD" x="25.4" y="19.1516" rot="R270"/>
 <element name="C2" library="SparkFun-Capacitors" package="0805" value="1uF" x="43.0784" y="14.9352" rot="MR90"/>
 <element name="C1" library="SparkFun-Capacitors" package="0805" value="1uF" x="43.0784" y="17.9324" rot="MR90"/>
@@
 <signal name="+3V3">
 <contactref element="U1" pad="9"/>
-<contactref element="S1" pad="B2"/>
-<contactref element="S2" pad="B2"/>
+<contactref element="S1" pad="3"/>
+<contactref element="S2" pad="3"/>
 <contactref element="C3" pad="1"/>
 <contactref element="C4" pad="1"/>
@@
 <wire x1="44.0944" y1="21.0964" x2="42.4688" y2="21.0964" width="0.3048" layer="16"/>
 <wire x1="42.4688" y1="21.0964" x2="42.418" y2="21.0456" width="0.3048" layer="16"/>
-<wire x1="23.1394" y1="47.9806" x2="23.1394" y2="38.174" width="0.3048" layer="1"/>
-<wire x1="23.1394" y1="38.174" x2="23.15" y2="38.1634" width="0.3048" layer="1"/>
-<wire x1="23.15" y1="38.1634" x2="23.203" y2="38.1634" width="0.3048" layer="1"/>
 <via x="33.528" y="19.1008" extent="1-16" drill="0.6" shape="square"/>
 <wire x1="33.528" y1="19.1008" x2="40.4732" y2="19.1008" width="0.3048" layer="16"/>
 <wire x1="40.4732" y1="19.1008" x2="42.418" y2="21.0456" width="0.3048" layer="16"/>
-<wire x1="23.15" y1="34.1376" x2="23.15" y2="38.1634" width="0.3048" layer="1"/>
 <wire x1="33.528" y1="19.1008" x2="25.4" y2="19.1008" width="0.3048" layer="1"/>
-<wire x1="25.4" y1="19.1008" x2="23.15" y2="19.1008" width="0.3048" layer="1"/>
-<wire x1="23.15" y1="19.1008" x2="23.15" y2="23.1266" width="0.3048" layer="1"/>
-<wire x1="23.15" y1="34.1376" x2="25.4" y2="34.1376" width="0.3048" layer="1"/>
 <wire x1="25.4" y1="34.1376" x2="25.4" y2="19.1008" width="0.3048" layer="1"/>
 <wire x1="15.6972" y1="6.6802" x2="16.4846" y2="6.6802" width="0.3048" layer="16"/>
@@
 <wire x1="45.1104" y1="21.1328" x2="45.1104" y2="21.9456" width="0.3048" layer="16"/>
 <wire x1="44.1308" y1="21.1328" x2="45.1104" y2="21.1328" width="0.3048" layer="16"/>
+<wire x1="25.4" y1="34.1376" x2="23.495" y2="34.1376" width="0.3048" layer="1"/>
+<wire x1="23.495" y1="34.1376" x2="23.495" y2="36.7284" width="0.3048" layer="1"/>
+<wire x1="23.1394" y1="47.9806" x2="23.495" y2="47.625" width="0.3048" layer="1"/>
+<wire x1="23.495" y1="47.625" x2="23.495" y2="36.7284" width="0.3048" layer="1"/>
+<wire x1="23.495" y1="21.6916" x2="23.495" y2="19.1008" width="0.3048" layer="1"/>
+<wire x1="23.495" y1="19.1008" x2="25.4" y2="19.1008" width="0.3048" layer="1"/>
 </signal>
 <signal name="GND">
@@
 </signal>
 <signal name="N$3">
-<contactref element="S1" pad="A2"/>
+<contactref element="S1" pad="1"/>
 <contactref element="U$3" pad="24"/>
 <wire x1="30.48" y1="53.34" x2="31.8008" y2="52.0192" width="0.3048" layer="1"/>
-<wire x1="31.8008" y1="52.0192" x2="31.8008" y2="42.3142" width="0.3048" layer="1"/>
-<wire x1="27.65" y1="38.1634" x2="31.8008" y2="38.1634" width="0.3048" layer="1"/>
-<wire x1="31.8008" y1="38.1634" x2="31.8008" y2="42.3142" width="0.3048" layer="1"/>
+<wire x1="27.305" y1="36.7284" x2="31.8008" y2="36.7284" width="0.3048" layer="1"/>
+<wire x1="31.8008" y1="36.7284" x2="31.8008" y2="52.0192" width="0.3048" layer="1"/>
 </signal>
 <signal name="N$7">
@@
 </signal>
 <signal name="N$2">
-<contactref element="S2" pad="A2"/>
+<contactref element="S2" pad="1"/>
 <contactref element="U$3" pad="26"/>
 <wire x1="33.02" y1="53.34" x2="34.3408" y2="52.0192" width="0.3048" layer="1"/>
 <wire x1="34.3408" y1="52.0192" x2="34.3408" y2="29.8174" width="0.3048" layer="1"/>
-<wire x1="27.65" y1="23.1266" x2="34.3408" y2="23.1266" width="0.3048" layer="1"/>
-<wire x1="34.3408" y1="23.1266" x2="34.3408" y2="29.8174" width="0.3048" layer="1"/>
+<wire x1="27.305" y1="21.6916" x2="34.3408" y2="21.6916" width="0.3048" layer="1"/>
+<wire x1="34.3408" y1="21.6916" x2="34.3408" y2="29.8174" width="0.3048" layer="1"/>
 </signal>
 <signal name="VSS">

Commit message: rework swd programmer
Connections:
- removed net VSS: U1.8
- net GND: now also U1.8
Changed lines of the file:
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@@
 <wire x1="21.9456" y1="49.1744" x2="4.1656" y2="49.1744" width="0.3048" layer="1"/>
 <wire x1="4.1656" y1="49.1744" x2="2.54" y2="50.8" width="0.3048" layer="1"/>
-<contactref element="U1" pad="6"/>
 <wire x1="44.1308" y1="21.1328" x2="44.0944" y2="21.0964" width="0.3048" layer="16"/>
 <wire x1="44.0944" y1="21.0964" x2="42.4688" y2="21.0964" width="0.3048" layer="16"/>
@@
 <wire x1="46.92" y1="22.12" x2="45.2848" y2="22.12" width="0.3048" layer="16"/>
 <wire x1="45.2848" y1="22.12" x2="45.1104" y2="21.9456" width="0.3048" layer="16"/>
-<wire x1="46.92" y1="20.02" x2="45.2072" y2="20.02" width="0.3048" layer="16"/>
 <wire x1="45.2072" y1="20.02" x2="45.1104" y2="20.1168" width="0.3048" layer="16"/>
 <wire x1="45.1104" y1="20.1168" x2="45.1104" y2="21.1328" width="0.3048" layer="16"/>
@@
 <wire x1="23.495" y1="21.6916" x2="23.495" y2="19.1008" width="0.3048" layer="1"/>
 <wire x1="23.495" y1="19.1008" x2="25.4" y2="19.1008" width="0.3048" layer="1"/>
+<contactref element="U1" pad="6"/>
+<wire x1="46.92" y1="20.02" x2="45.2072" y2="20.02" width="0.3048" layer="16"/>
 </signal>
 <signal name="GND">
@@
 <wire x1="4.3688" y1="8.92" x2="5.8928" y2="8.92" width="0.3048" layer="16"/>
 <wire x1="5.8928" y1="8.92" x2="5.8928" y2="12.192" width="0.3048" layer="16"/>
+<contactref element="U1" pad="8"/>
 </signal>
 <signal name="N$3">
@@
 <wire x1="34.3408" y1="21.6916" x2="34.3408" y2="29.8174" width="0.3048" layer="1"/>
 </signal>
-<signal name="VSS">
-<contactref element="U1" pad="8"/>
-</signal>
 <signal name="VCC">
