File: product.brd (EAGLE design)
At the start: 0 parts

Commit message: work in progress
Parts:
- added C1, C2, C4, C5: 1uF, SparkFun-Capacitors:0805
- added C3: 104, SparkFun-Capacitors:0805
- added C6: 0.1uF, SparkFun-Passives:0402-CAP
- added C7, C8: 16pF, SparkFun:0805
- added Q2: 16MHz, crystal:CTS406
- added R1: 390k/560k, SparkFun-Resistors:0805
- added R2: 100k, SparkFun-Passives:0402-RES
- added S1, S2: SWITCH-MOMENTARY-2SMD, SparkFun-Electromechanical:TACTILE_SWITCH_SMD
- added U$1: LM4F120H5QR, stellaris:LQFP64
- added U1: ATSHA204-TSU, SparkFun-DigitalIC:SOT23-3
- added U2: (no value), SparkFun-Connectors:USB-AB-MICRO-SMD
- added U3: (no value), microbuilder:UG-2864HSWEG01_0.96IN_WRAPAROUND
Connections:
- new net +3V3: C3.1, C4.1, C6.1, R2.2, S1.3, S2.3, U$1.11, U$1.26, U$1.42, U$1.54, U1.2, U3.9
- new net +5V: U2.VBUS
- new net GND: C3.2, C4.2, C5.2, C6.2, C7.2, C8.2, R1.2, U$1.12, U$1.27, U$1.39, U$1.55, U1.3, U2.GND, U3.1, U3.10, U3.11, U3.12, U3.29, U3.30
- new net GNDA: U$1.3
- new net GNDX: U$1.35
- new net N$1: U$1.22, U3.19
- new net N$10: C1.1, U3.2
- new net N$11: C2.1, U3.4
- new net N$12: C1.2, U3.3
- new net N$13: C2.2, U3.5
- new net N$14: S2.1, U$1.29
- new net N$15: S1.1, U$1.28
- new net N$2: U$1.9, U3.13
- new net N$3: U$1.43, U2.D-
- new net N$4: U$1.7, U3.15
- new net N$5: U$1.19, U3.18
- new net N$6: C5.1, U3.27
- new net N$7: U$1.44, U2.D+
- new net N$8: U$1.8, U3.14
- new net N$9: R1.1, U3.26
- new net SDA: R2.1, U$1.45, U1.1
- new net VBAT: U$1.37
- new net VCC: U3.28
- new net VDDA: U$1.2
- new net VDDC: U$1.25, U$1.56
- new net VSS: U3.8
- new net XTAL1: C7.1, Q2.1, U$1.40
- new net XTAL2: C8.1, Q2.3, U$1.41
Routing:
- net GND: track 0.00 -> 63.3 mm
- net +3V3: track 0.00 -> 37.9 mm
- net N$1: track 0.00 -> 23.0 mm
- net N$5: track 0.00 -> 21.6 mm
- net SDA: track 0.00 -> 17.1 mm
- net XTAL2: track 0.00 -> 15.1 mm
- net XTAL1: track 0.00 -> 12.2 mm
- net N$2: track 0.00 -> 10.3 mm
- net N$8: track 0.00 -> 10.1 mm
- net N$4: track 0.00 -> 9.94 mm
- net N$6: track 0.00 -> 8.49 mm
- net N$13: track 0.00 -> 6.28 mm
- net N$10: track 0.00 -> 5.99 mm
- net N$11: track 0.00 -> 5.18 mm
- net N$12: track 0.00 -> 4.89 mm
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Other:
- board outline added: 59.7 x 31.8 mm

Commit message: work on product scheme
Parts:
- added C10: 100nF, SparkFun-Capacitors:0805
- added C11: 10uF, SparkFun-Capacitors:0805
- added C12, C14, C19, C21: 0.1uF, SparkFun-Passives:0402-CAP
- added C13, C15, C16: 0.01uF, SparkFun-Passives:0402-CAP
- added C17, C18: 1uF, SparkFun-Passives:0402-CAP
- added C20: 2.2uF, SparkFun-Passives:0402-CAP
- added C9: 0.1uF, SparkFun:0805
- added R3, R4, R5: 10k, SparkFun-Passives:0402-RES
- added TP1, TP2, TP3, TP4: PTR1TP10R, testpad:TP10R
- added U4: (no value), microbuilder:SOT223-R
- C7, C8: value 16pF -> 10pF
- moved C4 22.9 mm to (31.8, 1.91), flipped to the top, turned to 180 degrees
- moved C5 21.9 mm to (34.9, 21.6), flipped to the top, turned to 270 degrees
- moved C7 17.8 mm to (10.2, 10.8), flipped to the top
- moved C3 17.1 mm to (34.9, 2.54), flipped to the top
- moved Q2 16.6 mm to (14.0, 7.62), flipped to the top, turned to 0 degrees
- moved U$1 15.9 mm to (23.5, 15.9), flipped to the top, turned to 225 degrees
- moved C1 14.6 mm to (34.9, 5.71), flipped to the top
- moved C2 14.6 mm to (34.9, 9.53), flipped to the top
- moved R1 14.6 mm to (34.9, 24.8), flipped to the top
- moved C8 10.3 mm to (14.0, 10.8), flipped to the top, turned to 180 degrees
- moved U1 8.98 mm to (14.0, 25.4), flipped to the top
- moved R2 7.85 mm to (14.0, 22.2), flipped to the top
- moved C6 2.29 mm to (17.1, 25.4), flipped to the top
Connections:
- removed net GNDA: U$1.3
- removed net GNDX: U$1.35
- removed net VBAT: U$1.37
- removed net VDDA: U$1.2
- removed net VDDC: U$1.25, U$1.56
- new net N$16: R4.1, TP2.TP, U$1.51
- new net N$17: R3.1, TP1.TP, U$1.52
- new net N$19: TP3.TP, U$1.50
- new net N$20: TP4.TP, U$1.49
- new net N$21: C9.2, R5.1, U$1.38
- new net N$23: C18.1, C19.1, C20.1, C21.1, U$1.25, U$1.56
- net +3V3: now also C11.2, C12.1, C13.1, C14.1, C15.1, C16.1, C17.1, R3.2, R4.2, R5.2, U$1.2, U$1.37, U4.2; no longer S1.3, S2.3
- net +5V: now also C10.2, U4.3
- net GND: now also C10.1, C11.1, C12.2, C13.2, C14.2, C15.2, C16.2, C17.2, C18.2, C19.2, C20.2, C21.2, C9.1, S1.3, S2.3, U$1.3, U$1.32, U$1.34, U$1.35, U4.1
- net SDA: now also U$1.48; no longer U$1.45
Routing:
- net GND: track 63.3 -> 33.2 mm
- net +3V3: track 37.9 -> 8.64 mm
- net N$1: track 23.0 -> 0.00 mm
- net N$5: track 21.6 -> 0.00 mm
- net XTAL2: track 15.1 -> 0.00 mm
- net SDA: track 17.1 -> 2.47 mm
- net XTAL1: track 12.2 -> 0.00 mm
- net N$2: track 10.3 -> 0.00 mm
- net N$8: track 10.1 -> 0.00 mm
- net N$4: track 9.94 -> 0.00 mm
- net N$6: track 8.49 -> 0.00 mm
- net N$13: track 6.28 -> 0.00 mm
- net N$10: track 5.99 -> 0.00 mm
- net N$11: track 5.18 -> 0.00 mm
- net N$12: track 4.89 -> 0.00 mm
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
Commit message: wip
Parts:
- removed U4: (no value), microbuilder:SOT223-R
- added IC1: MCP1703CB, linear:SOT23
- C1, C2, C3, C4, C5: device SparkFun-Capacitors:0805 -> SparkFun-Passives:0402-CAP
- C10: value 100nF -> 1uF; device SparkFun-Capacitors:0805 -> SparkFun-Passives:0402-CAP
- C11: value 10uF -> 1uF; device SparkFun-Capacitors:0805 -> SparkFun-Passives:0402-CAP
- C7, C8, C9: device SparkFun:0805 -> SparkFun-Passives:0402-CAP
- R1: device SparkFun-Resistors:0805 -> SparkFun-Passives:0402-RES
- moved C21 68.1 mm to (12.7, 24.4), turned to 270 degrees
- moved C20 65.8 mm to (13.7, 24.4), turned to 270 degrees
- moved R5 65.7 mm to (14.0, 17.8), turned to 270 degrees
- moved C19 64.9 mm to (31.1, 12.1), turned to 270 degrees
- moved C17 64.5 mm to (19.7, 28.6), turned to 270 degrees
- moved C18 62.1 mm to (30.2, 12.1), turned to 270 degrees
- moved C16 61.1 mm to (25.4, 28.6), turned to 270 degrees
- moved C15 56.1 mm to (21.6, 28.6), turned to 270 degrees
- moved C13 53.4 mm to (23.5, 28.6), turned to 270 degrees
- moved R4 52.8 mm to (26.0, 8.26)
- moved R3 50.6 mm to (26.0, 6.99)
- moved C12 47.9 mm to (27.9, 10.8), turned to 90 degrees
- moved C14 46.4 mm to (16.5, 22.9), turned to 270 degrees
- moved C11 35.2 mm to (10.2, 21.6), turned to 90 degrees
- moved C10 29.1 mm to (7.62, 19.1), turned to 180 degrees
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Connections:
- net +3V3: now also IC1.2; no longer U4.2
- net +5V: now also IC1.3; no longer U4.3
- net GND: now also IC1.1; no longer U4.1
Routing:
- net N$7: track 0.00 -> 29.7 mm
- net N$3: track 0.00 -> 28.9 mm
- net +3V3: track 8.64 -> 32.8 mm
- net N$23: track 0.00 -> 14.8 mm
- net XTAL1: track 0.00 -> 14.1 mm
- net N$21: track 0.00 -> 13.1 mm
- net GND: track 33.2 -> 45.7 mm
- net SDA: track 2.47 -> 12.1 mm
- net +5V: track 0.00 -> 6.45 mm
- net XTAL2: track 0.00 -> 5.48 mm

Commit message: work in progress
Parts:
- moved R5 4.84 mm to (9.53, 15.9), turned to 90 degrees
- moved C9 3.70 mm to (8.26, 15.9)
- moved C5 1.91 mm to (34.9, 23.5), turned to 90 degrees
- moved R1 1.91 mm to (34.9, 26.7)
- turned S1 to 270 degrees
Routing:
- net +3V3: track 32.8 -> 123.6 mm, vias 0 -> 1
- net N$1: track 0.00 -> 41.7 mm, vias 0 -> 1
- net GND: track 45.7 -> 87.0 mm, vias 0 -> 3
- net N$5: track 0.00 -> 38.6 mm, vias 0 -> 1
- net N$2: track 0.00 -> 38.0 mm, vias 0 -> 1
- net N$8: track 0.00 -> 36.5 mm, vias 0 -> 1
- net N$4: track 0.00 -> 35.2 mm, vias 0 -> 1
- net N$9: track 0.00 -> 21.1 mm, vias 0 -> 1
- net N$6: track 0.00 -> 21.1 mm, vias 0 -> 1
- net N$13: track 0.00 -> 20.0 mm, vias 0 -> 1
- net N$10: track 0.00 -> 19.7 mm, vias 0 -> 1
- net N$11: track 0.00 -> 19.4 mm, vias 0 -> 1
- net N$12: track 0.00 -> 19.1 mm, vias 0 -> 1
- net N$23: track 14.8 -> 26.2 mm, vias 0 -> 2
- net N$21: track 13.1 -> 10.5 mm
- added copper zone on layer 1, net GND

Commit message: work in progress
Parts:
- U2: value (none) -> USB
- U3: value (none) -> DISPLAY
- moved R4 2.84 mm to (24.8, 5.71)
- moved TP1 2.54 mm to (25.4, 8.26)
- moved TP2 2.54 mm to (24.1, 8.26)
- moved TP3 2.54 mm to (22.9, 8.26)
- moved TP4 2.54 mm to (21.6, 8.26)
- moved C9 0.63 mm to (8.89, 15.9)
- moved R5 0.63 mm to (10.2, 15.9)
- moved C19 0.33 mm to (31.4, 12.1)
- moved C20 0.30 mm to (14.0, 24.4)
- turned C13 to 90 degrees
- turned C15 to 90 degrees
- turned C16 to 90 degrees
- turned C17 to 90 degrees
Routing:
- net N$15: track 0.00 -> 25.1 mm, vias 0 -> 2
- net N$14: track 0.00 -> 21.5 mm, vias 0 -> 2
- net N$16: track 0.00 -> 7.36 mm
- net N$17: track 0.00 -> 6.28 mm
- net N$20: track 0.00 -> 5.12 mm
- net N$19: track 0.00 -> 4.95 mm
- net N$2: track 38.0 -> 41.2 mm
- net +3V3: track 123.6 -> 126.4 mm
- net N$8: track 36.5 -> 38.5 mm
- net GND: track 87.0 -> 88.0 mm, vias 3 -> 6
- net N$21: track 10.5 -> 11.4 mm
- net N$6: track 21.1 -> 22.0 mm
- net N$23: track 26.2 -> 27.1 mm
- net N$4: track 35.2 -> 35.9 mm

Commit message: work on pcbs
Parts:
- moved R5 5.82 mm to (14.1, 20.1)
- moved C9 5.65 mm to (11.8, 20.7), turned to 90 degrees
- moved C20 3.59 mm to (17.1, 26.2), turned to 90 degrees
- moved C21 3.48 mm to (15.7, 26.2), turned to 90 degrees
- moved C4 0.94 mm to (31.0, 2.49), turned to 90 degrees
- moved C10 0.86 mm to (7.01, 18.4)
- moved C11 0.86 mm to (9.55, 21.0)
- moved IC1 0.86 mm to (7.01, 21.0)
- moved C14 0.61 mm to (15.9, 22.9)
- moved U2 0.61 mm to (1.91, 15.9)
- moved C7 0.61 mm to (8.89, 10.8)
- moved Q2 0.61 mm to (13.3, 10.1)
- moved R4 0.61 mm to (25.4, 5.71)
- moved U1 0.61 mm to (22.9, 3.78)
- moved R2 0.61 mm to (22.9, 1.55)
Routing:
- net GND: track 88.0 -> 24.3 mm, vias 6 -> 13
- net +3V3: track 126.4 -> 113.1 mm
- net N$23: track 27.1 -> 23.7 mm
- net N$7: track 29.5 -> 27.2 mm
- net N$3: track 28.9 -> 26.9 mm
- net N$9: track 21.1 -> 19.5 mm
- net N$20: track 5.12 -> 3.94 mm
- net +5V: track 6.45 -> 5.48 mm
- net N$13: track 20.0 -> 19.2 mm
- net N$10: track 19.7 -> 18.9 mm
- net N$4: track 35.9 -> 36.7 mm
- net N$21: track 11.4 -> 12.1 mm
- net XTAL1: track 14.1 -> 13.5 mm
- net N$11: track 19.3 -> 18.8 mm
- net XTAL2: track 5.48 -> 6.01 mm
- added copper zone on layer 16, net GND
Other:
- board size 59.7 x 31.8 mm -> 59.8 x 31.6 mm
- board text added: "trezor"

Commit message: work in progress
Parts:
- moved C9 0.61 mm to (11.8, 21.3)
- moved R5 0.61 mm to (14.1, 20.8)
- moved Q2 0.30 mm to (13.3, 9.83)
Routing:
- net N$21: track 12.1 -> 14.8 mm, vias 0 -> 2
- net +3V3: track 113.1 -> 115.1 mm
- net N$3: track 26.9 -> 25.6 mm, vias 0 -> 2
- net N$7: track 27.2 -> 26.3 mm, vias 0 -> 2
- net GND: vias 13 -> 16

Commit message: try freerouting
Parts:
- added C22, C23: 10uF, SparkFun-Passives:0402-CAP
- added U4: TPD4S014_DSQ_10, imported:DSQ10_1P5X0P9
- moved C15 19.9 mm to (19.5, 8.76)
- moved C13 18.1 mm to (31.1, 12.1)
- moved C7 10.4 mm to (16.7, 3.86), turned to 270 degrees
- moved C8 5.89 mm to (12.1, 11.7), turned to 0 degrees
- moved C19 5.17 mm to (35.1, 15.7)
- moved C18 4.96 mm to (33.5, 15.7)
- moved C11 4.67 mm to (13.0, 24.1), turned to 270 degrees
- moved C17 4.23 mm to (23.3, 26.4)
- moved C10 3.48 mm to (4.88, 21.2), turned to 0 degrees
- moved R4 3.37 mm to (25.1, 2.36)
- moved C16 3.14 mm to (26.9, 25.8)
- moved U1 2.89 mm to (20.1, 4.70)
- moved R2 2.76 mm to (20.1, 1.85)
- moved IC1 2.60 mm to (9.45, 21.9)
- moved C6 2.46 mm to (22.7, 2.87)
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Connections:
- new net USB_D_N: U$1.43, U2.D-, U4.6
- new net USB_D_P: U$1.44, U2.D+, U4.7
- net +5V: now also C23.1, U4.1, U4.2; no longer U2.VBUS
- net GND: now also C22.2, C23.2, U4.8
- net N$3: now also U2.ID, U4.5; no longer U$1.43, U2.D-
- net N$7: now also C22.1, U2.VBUS, U4.10, U4.9; no longer U$1.44, U2.D+
Routing:
- net +3V3: track 115.1 -> 0.00 mm, vias 1 -> 0
- net N$1: track 41.7 -> 0.00 mm, vias 1 -> 0
- net N$2: track 41.2 -> 0.00 mm, vias 1 -> 0
- net N$8: track 38.9 -> 0.00 mm, vias 1 -> 0
- net N$5: track 38.6 -> 0.00 mm, vias 1 -> 0
- net N$4: track 36.7 -> 0.00 mm, vias 1 -> 0
- net N$7: track 26.3 -> 0.00 mm, vias 2 -> 0
- net N$3: track 25.6 -> 0.00 mm, vias 2 -> 0
- net N$15: track 25.1 -> 0.00 mm, vias 2 -> 0
- net GND: track 24.3 -> 0.00 mm, vias 16 -> 0
- net N$23: track 23.7 -> 0.00 mm, vias 2 -> 0
- net N$6: track 21.7 -> 0.00 mm, vias 1 -> 0
- net N$14: track 21.5 -> 0.00 mm, vias 2 -> 0
- net N$9: track 19.5 -> 0.00 mm, vias 1 -> 0
- net N$13: track 19.2 -> 0.00 mm, vias 1 -> 0
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Other:
- outline, holes or cut-outs redrawn
- board text removed: "trezor"
