File: product.brd (EAGLE design)
At the start: 59.8 x 31.6 mm, 41 parts, among them IC1 MCP1703CB, Q2 16MHz, U1 ATSHA204-TSU, U2 USB, U3 DISPLAY, U4 TPD4S014_DSQ_10

Commit message: routed
Parts:
- moved U4 1.10 mm to (8.53, 13.1)
Changed lines of the file:
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@@
 <?xml version="1.0" encoding="utf-8"?>
 <!DOCTYPE eagle SYSTEM "eagle.dtd">
-<eagle version="6.3">
+<eagle version="6.4">
 <drawing>
 <settings>
@@
 </element>
 <element name="IC1" library="linear" package="SOT23" value="MCP1703CB" x="9.4488" y="21.8948" rot="R90"/>
-<element name="U4" library="imported" package="DSQ10_1P5X0P9" value="TPD4S014_DSQ_10" x="7.9248" y="14.0208" rot="R90"/>
+<element name="U4" library="imported" package="DSQ10_1P5X0P9" value="TPD4S014_DSQ_10" x="8.5344" y="13.1064" rot="R90"/>
 <element name="C22" library="SparkFun-Passives" package="0402-CAP" value="10uF" x="8.2296" y="17.9832"/>
 <element name="C23" library="SparkFun-Passives" package="0402-CAP" value="10uF" x="4.572" y="10.668" rot="R180"/>
@@
 <contactref element="C22" pad="2"/>
 <contactref element="C23" pad="2"/>
-<wire x1="8.8796" y1="17.9832" x2="7.9248" y2="15.0368" width="0" layer="19" extent="1-1"/>
+<wire x1="8.8796" y1="17.9832" x2="8.5344" y2="14.1224" width="0" layer="19" extent="1-1"/>
 <wire x1="53.27" y1="13.425" x2="35.1028" y2="15.0726" width="0" layer="19" extent="1-16"/>
 </signal>
@@
 <contactref element="C23" pad="1"/>
 <wire x1="5.5268" y1="21.1836" x2="8.3488" y2="21.8948" width="0" layer="19" extent="1-1"/>
-<wire x1="7.1374" y1="13.0048" x2="5.5268" y2="21.1836" width="0" layer="19" extent="1-1"/>
-<wire x1="7.5184" y1="13.0048" x2="7.1374" y2="13.0048" width="0" layer="19" extent="1-1"/>
-<wire x1="5.222" y1="10.668" x2="7.1374" y2="13.0048" width="0" layer="19" extent="1-1"/>
+<wire x1="7.747" y1="12.0904" x2="5.5268" y2="21.1836" width="0" layer="19" extent="1-1"/>
+<wire x1="8.128" y1="12.0904" x2="7.747" y2="12.0904" width="0" layer="19" extent="1-1"/>
+<wire x1="5.222" y1="10.668" x2="7.747" y2="12.0904" width="0" layer="19" extent="1-1"/>
 </signal>
 <signal name="SDA">
@@
 <contactref element="U2" pad="ID"/>
 <contactref element="U4" pad="5"/>
-<wire x1="4.755" y1="15.2504" x2="8.7122" y2="13.0048" width="0" layer="19" extent="1-1"/>
+<wire x1="4.755" y1="15.2504" x2="9.3218" y2="12.0904" width="0" layer="19" extent="1-1"/>
 </signal>
 <signal name="N$7">
@@
 <contactref element="C22" pad="1"/>
 <wire x1="4.755" y1="17.2004" x2="7.5796" y2="17.9832" width="0" layer="19" extent="1-1"/>
-<wire x1="7.5184" y1="15.0368" x2="7.5796" y2="17.9832" width="0" layer="19" extent="1-1"/>
-<wire x1="7.1374" y1="15.0368" x2="7.5184" y2="15.0368" width="0" layer="19" extent="1-1"/>
+<wire x1="8.128" y1="14.1224" x2="7.5796" y2="17.9832" width="0" layer="19" extent="1-1"/>
+<wire x1="7.747" y1="14.1224" x2="8.128" y2="14.1224" width="0" layer="19" extent="1-1"/>
 </signal>
 <signal name="USB_D_N">
@@
 <contactref element="U4" pad="6"/>
 <contactref element="U$1" pad="43"/>
-<wire x1="8.7122" y1="15.0368" x2="20.018171875" y2="12.25600625" width="0" layer="19" extent="1-1"/>
-<wire x1="4.755" y1="16.5504" x2="8.7122" y2="15.0368" width="0" layer="19" extent="1-1"/>
+<wire x1="9.3218" y1="14.1224" x2="20.018171875" y2="12.25600625" width="0" layer="19" extent="1-1"/>
+<wire x1="4.755" y1="16.5504" x2="9.3218" y2="14.1224" width="0" layer="19" extent="1-1"/>
 </signal>
 <signal name="USB_D_P">
@@
 <contactref element="U4" pad="7"/>
 <contactref element="U$1" pad="44"/>
-<wire x1="8.3312" y1="15.0368" x2="20.371728125" y2="11.902453125" width="0" layer="19" extent="1-1"/>
-<wire x1="4.755" y1="15.9004" x2="8.3312" y2="15.0368" width="0" layer="19" extent="1-1"/>
+<wire x1="8.9408" y1="14.1224" x2="20.371728125" y2="11.902453125" width="0" layer="19" extent="1-1"/>
+<wire x1="4.755" y1="15.9004" x2="8.9408" y2="14.1224" width="0" layer="19" extent="1-1"/>
 </signal>
 </signals>

Commit message: new pcb size :-/
Parts:
- moved C10 37.0 mm to (14.2, 56.9)
- moved C15 37.0 mm to (28.8, 44.5)
- moved C2 37.0 mm to (44.2, 45.3)
- moved C4 37.0 mm to (40.3, 38.3)
- moved C6 37.0 mm to (32.0, 38.6)
- moved C7 37.0 mm to (26.0, 39.6)
- moved C8 37.0 mm to (21.4, 47.4)
- moved Q2 37.0 mm to (24.8, 44.5)
- moved R2 37.0 mm to (29.4, 37.6)
- moved R3 37.0 mm to (35.4, 41.2)
- moved U1 37.0 mm to (29.4, 40.5)
- moved U2 37.0 mm to (11.2, 51.7)
- moved C1 37.0 mm to (44.2, 41.5)
- moved C11 37.0 mm to (22.3, 59.9)
- moved C12 37.0 mm to (36.7, 45.3)
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Routing:
- removed copper zone on layer 1, net GND
- removed copper zone on layer 16, net GND
Other:
- board size 59.8 x 31.6 mm -> 50 x 26.7 mm

Commit message: work in progress
Parts:
- removed C22, C23: 10uF, SparkFun-Passives:0402-CAP
- removed U4: TPD4S014_DSQ_10, imported:DSQ10_1P5X0P9
- added U5: TPD4S012_DRY_6, imported:DRY6
- moved C9 41.5 mm to (12.2, 16.4)
- moved C10 40.4 mm to (7.49, 17.1)
- moved C11 40.3 mm to (13.8, 20.5)
- moved U$1 39.6 mm to (33.0, 13.3), flipped to the bottom, turned to 45 degrees
- moved U2 39.4 mm to (2.08, 13.4)
- moved IC1 38.5 mm to (10.2, 20.1)
- moved Q2 24.2 mm to (21.3, 20.5), flipped to the bottom
- moved C7 24.0 mm to (21.3, 16.1), flipped to the bottom, turned to 180 degrees
- moved C8 23.9 mm to (25.1, 23.9), flipped to the bottom, turned to 180 degrees
- moved U1 16.8 mm to (32.7, 24.0), flipped to the bottom
- moved R2 16.4 mm to (32.7, 21.6), flipped to the bottom
- moved C6 15.7 mm to (30.4, 23.0), flipped to the bottom
- moved R4 5.66 mm to (29.1, 40.2)
- moved R3 0.64 mm to (35.6, 40.6)
- moved C15 0.64 mm to (28.2, 44.3)
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Connections:
- removed net N$7: C22.1, U2.VBUS, U4.10, U4.9
- net +5V: now also U2.VBUS, U5.6; no longer C23.1, U4.1, U4.2
- net GND: now also U5.4; no longer C22.2, C23.2, U4.8
- net N$3: now also U5.3; no longer U4.5
- net USB_D_N: now also U5.2; no longer U4.6
- net USB_D_P: now also U5.1; no longer U4.7
Other:
- outline, holes or cut-outs redrawn

Commit message: work on product
Parts:
- moved C17 60.1 mm to (39.5, 2.53), flipped to the bottom, turned to 0 degrees
- moved C21 57.1 mm to (16.1, 6.83), turned to 270 degrees
- moved C20 57.0 mm to (14.3, 7.67), turned to 270 degrees
- moved C19 55.1 mm to (12.5, 6.58)
- moved C18 54.5 mm to (10.7, 7.39)
- moved C14 49.8 mm to (17.9, 10.9), flipped to the bottom
- moved R5 45.6 mm to (22.5, 12.6), flipped to the bottom, turned to 270 degrees
- moved C13 44.4 mm to (16.1, 10.7), flipped to the bottom
- moved R1 42.4 mm to (44.6, 20.1), flipped to the bottom, turned to 270 degrees
- moved C12 42.2 mm to (29.2, 3.91), flipped to the bottom, turned to 0 degrees
- moved C15 42.1 mm to (29.1, 2.23), flipped to the bottom, turned to 0 degrees
- moved C2 39.2 mm to (44.8, 6.12), flipped to the bottom
- moved C1 38.5 mm to (44.8, 2.97), flipped to the bottom
- moved C5 37.4 mm to (35.5, 22.9), flipped to the bottom
- moved C16 37.2 mm to (36.9, 24.4), flipped to the bottom, turned to 270 degrees
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Routing:
- net +3V3: track 0.00 -> 119.2 mm, vias 0 -> 1
- net USB_D_N: track 0.00 -> 37.6 mm, vias 0 -> 1
- net N$23: track 0.00 -> 34.2 mm, vias 0 -> 1
- net USB_D_P: track 0.00 -> 31.6 mm, vias 0 -> 1
- net SDA: track 0.00 -> 28.5 mm
- net N$5: track 0.00 -> 21.5 mm, vias 0 -> 2
- net N$1: track 0.00 -> 15.8 mm
- net N$16: track 0.00 -> 14.9 mm
- net +5V: track 0.00 -> 14.6 mm
- net N$15: track 0.00 -> 14.0 mm, vias 0 -> 1
- net N$2: track 0.00 -> 12.8 mm, vias 0 -> 2
- net XTAL1: track 0.00 -> 12.2 mm
- net XTAL2: track 0.00 -> 11.0 mm
- net N$3: track 0.00 -> 10.5 mm, vias 0 -> 2
- net N$14: track 0.00 -> 10.0 mm, vias 0 -> 1
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- added copper zone on layer 1, net GND
- added copper zone on layer 16, net GND
