File: raspi.sch (EAGLE design)
At the start: 5 parts

Commit message: fix distance for display
Other:
- moved on the sheet: JP1
Changed lines of the file:
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@@
 <instances>
 <instance part="U$1" gate="G$1" x="33.02" y="25.4"/>
-<instance part="JP1" gate="A" x="91.44" y="66.04"/>
+<instance part="JP1" gate="A" x="109.22" y="33.02"/>
 <instance part="JP2" gate="A" x="0" y="22.86" rot="MR0"/>
 <instance part="SW1" gate="G$1" x="81.28" y="20.32"/>
@@
 <instance part="+3V1" gate="G$1" x="7.62" y="81.28"/>
 <instance part="+3V2" gate="G$1" x="88.9" y="25.4"/>
-<instance part="GND1" gate="1" x="66.04" y="60.96"/>
-<instance part="GND2" gate="1" x="81.28" y="53.34"/>
-<instance part="+3V4" gate="G$1" x="81.28" y="81.28"/>
+<instance part="GND1" gate="1" x="66.04" y="66.04" rot="R90"/>
+<instance part="GND2" gate="1" x="99.06" y="20.32"/>
+<instance part="+3V4" gate="G$1" x="99.06" y="48.26"/>
 <instance part="+3V3" gate="G$1" x="93.98" y="25.4"/>
 </instances>
@@
 <segment>
 <pinref part="JP1" gate="A" pin="1"/>
-<wire x1="88.9" y1="76.2" x2="81.28" y2="76.2" width="0.1524" layer="91"/>
+<wire x1="106.68" y1="43.18" x2="99.06" y2="43.18" width="0.1524" layer="91"/>
 <pinref part="+3V4" gate="G$1" pin="+3V3"/>
-<wire x1="81.28" y1="76.2" x2="81.28" y2="78.74" width="0.1524" layer="91"/>
+<wire x1="99.06" y1="43.18" x2="99.06" y2="45.72" width="0.1524" layer="91"/>
 </segment>
 <segment>
@@
 <segment>
 <pinref part="JP1" gate="A" pin="8"/>
-<wire x1="88.9" y1="58.42" x2="81.28" y2="58.42" width="0.1524" layer="91"/>
+<wire x1="106.68" y1="25.4" x2="99.06" y2="25.4" width="0.1524" layer="91"/>
 <pinref part="GND2" gate="1" pin="GND"/>
-<wire x1="81.28" y1="58.42" x2="81.28" y2="55.88" width="0.1524" layer="91"/>
+<wire x1="99.06" y1="25.4" x2="99.06" y2="22.86" width="0.1524" layer="91"/>
 </segment>
 <segment>
 <pinref part="U$1" gate="G$1" pin="6-GND"/>
-<wire x1="60.96" y1="66.04" x2="66.04" y2="66.04" width="0.1524" layer="91"/>
+<wire x1="60.96" y1="66.04" x2="63.5" y2="66.04" width="0.1524" layer="91"/>
 <pinref part="GND1" gate="1" pin="GND"/>
-<wire x1="66.04" y1="66.04" x2="66.04" y2="63.5" width="0.1524" layer="91"/>
 </segment>
 </net>
@@
 <segment>
 <wire x1="60.96" y1="25.4" x2="76.2" y2="25.4" width="0.1524" layer="91"/>
-<wire x1="76.2" y1="25.4" x2="76.2" y2="63.5" width="0.1524" layer="91"/>
+<wire x1="76.2" y1="25.4" x2="76.2" y2="30.48" width="0.1524" layer="91"/>
 <pinref part="JP1" gate="A" pin="6"/>
-<wire x1="76.2" y1="63.5" x2="88.9" y2="63.5" width="0.1524" layer="91"/>
+<wire x1="76.2" y1="30.48" x2="106.68" y2="30.48" width="0.1524" layer="91"/>
 <pinref part="U$1" gate="G$1" pin="22-GPIO6"/>
 </segment>
@@
 <pinref part="U$1" gate="G$1" pin="18-GPIO5"/>
 <wire x1="60.96" y1="35.56" x2="73.66" y2="35.56" width="0.1524" layer="91"/>
-<wire x1="73.66" y1="35.56" x2="73.66" y2="71.12" width="0.1524" layer="91"/>
+<wire x1="73.66" y1="35.56" x2="73.66" y2="38.1" width="0.1524" layer="91"/>
 <pinref part="JP1" gate="A" pin="3"/>
-<wire x1="73.66" y1="71.12" x2="88.9" y2="71.12" width="0.1524" layer="91"/>
+<wire x1="73.66" y1="38.1" x2="106.68" y2="38.1" width="0.1524" layer="91"/>
 </segment>
 </net>
@@
 <segment>
 <pinref part="JP1" gate="A" pin="2"/>
-<wire x1="88.9" y1="73.66" x2="71.12" y2="73.66" width="0.1524" layer="91"/>
-<wire x1="71.12" y1="73.66" x2="71.12" y2="40.64" width="0.1524" layer="91"/>
+<wire x1="106.68" y1="40.64" x2="60.96" y2="40.64" width="0.1524" layer="91"/>
 <pinref part="U$1" gate="G$1" pin="16-GPIO4"/>
-<wire x1="71.12" y1="40.64" x2="60.96" y2="40.64" width="0.1524" layer="91"/>
 </segment>
 </net>

Commit message: rework raspi board
Parts:
- removed SW1, SW2: (no value), microbuilder:SWITCH_PUSHBUTTONSOFTTOUCHSMD_SJ
- added S1, S2: (no value), SparkFun:TAC_SWITCHPTH
Connections:
- removed net N$4: SW2.P$1, U$1.26-SPI-CE1-N
- new net N$2: S2.1, U$1.26-SPI-CE1-N
- net +3V3: now also S1.3, S2.3; no longer SW1.P$2, SW2.P$2
- net N$3: now also S1.1; no longer SW1.P$1
Changed lines of the file:
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@@
 <layer number="111" name="MPL" color="7" fill="1" visible="yes" active="yes"/>
 <layer number="112" name="tSilk" color="7" fill="1" visible="yes" active="yes"/>
+<layer number="116" name="Patch_BOT" color="9" fill="4" visible="no" active="yes"/>
 <layer number="121" name="sName" color="7" fill="1" visible="yes" active="yes"/>
 <layer number="122" name="_bPlace" color="7" fill="1" visible="yes" active="yes"/>
@@
 <layer number="204" name="204bmp" color="7" fill="1" visible="yes" active="yes"/>
 <layer number="205" name="205bmp" color="7" fill="1" visible="yes" active="yes"/>
+<layer number="206" name="206bmp" color="7" fill="10" visible="no" active="yes"/>
+<layer number="207" name="207bmp" color="8" fill="10" visible="no" active="yes"/>
+<layer number="208" name="208bmp" color="9" fill="10" visible="no" active="yes"/>
+<layer number="209" name="209bmp" color="7" fill="1" visible="no" active="yes"/>
+<layer number="210" name="210bmp" color="7" fill="1" visible="no" active="yes"/>
+<layer number="211" name="211bmp" color="7" fill="1" visible="no" active="yes"/>
+<layer number="212" name="212bmp" color="7" fill="1" visible="no" active="yes"/>
+<layer number="213" name="213bmp" color="7" fill="1" visible="no" active="yes"/>
+<layer number="214" name="214bmp" color="7" fill="1" visible="no" active="yes"/>
+<layer number="215" name="215bmp" color="7" fill="1" visible="no" active="yes"/>
+<layer number="216" name="216bmp" color="7" fill="1" visible="no" active="yes"/>
+<layer number="217" name="217bmp" color="18" fill="1" visible="no" active="no"/>
+<layer number="218" name="218bmp" color="19" fill="1" visible="no" active="no"/>
+<layer number="219" name="219bmp" color="20" fill="1" visible="no" active="no"/>
+<layer number="220" name="220bmp" color="21" fill="1" visible="no" active="no"/>
+<layer number="221" name="221bmp" color="22" fill="1" visible="no" active="no"/>
+<layer number="222" name="222bmp" color="23" fill="1" visible="no" active="no"/>
+<layer number="223" name="223bmp" color="24" fill="1" visible="no" active="no"/>
+<layer number="224" name="224bmp" color="25" fill="1" visible="no" active="no"/>
 <layer number="248" name="Housing" color="7" fill="1" visible="yes" active="yes"/>
 <layer number="249" name="Edge" color="7" fill="1" visible="yes" active="yes"/>
@@
 <part name="JP1" library="pinhead" deviceset="PINHD-1X8" device=""/>
 <part name="JP2" library="pinhead" deviceset="PINHD-1X8" device=""/>
-<part name="SW1" library="microbuilder" deviceset="SWITCH_PUSHBUTTON" device="SOFTTOUCHSMD_SJ"/>
-<part name="SW2" library="microbuilder" deviceset="SWITCH_PUSHBUTTON" device="SOFTTOUCHSMD_SJ"/>
 <part name="+3V1" library="supply1" deviceset="+3V3" device=""/>
 <part name="+3V2" library="supply1" deviceset="+3V3" device=""/>
@@
 <part name="+3V4" library="supply1" deviceset="+3V3" device=""/>
 <part name="+3V3" library="supply1" deviceset="+3V3" device=""/>
+<part name="S1" library="SparkFun" deviceset="TAC_SWITCH" device="PTH"/>
+<part name="S2" library="SparkFun" deviceset="TAC_SWITCH" device="PTH"/>
 </parts>
 <sheets>
@@
 <instance part="JP1" gate="A" x="109.22" y="33.02"/>
 <instance part="JP2" gate="A" x="0" y="22.86" rot="MR0"/>
-<instance part="SW1" gate="G$1" x="81.28" y="20.32"/>
-<instance part="SW2" gate="G$1" x="81.28" y="15.24"/>
 <instance part="+3V1" gate="G$1" x="7.62" y="81.28"/>
 <instance part="+3V2" gate="G$1" x="88.9" y="25.4"/>
@@
 <instance part="+3V4" gate="G$1" x="99.06" y="48.26"/>
 <instance part="+3V3" gate="G$1" x="93.98" y="25.4"/>
+<instance part="S1" gate="S" x="78.74" y="20.32"/>
+<instance part="S2" gate="S" x="78.74" y="7.62"/>
 </instances>
 <busses>
@@
 </segment>
 <segment>
-<pinref part="SW1" gate="G$1" pin="P$2"/>
-<wire x1="88.9" y1="20.32" x2="86.36" y2="20.32" width="0.1524" layer="91"/>
 <pinref part="+3V2" gate="G$1" pin="+3V3"/>
 <wire x1="88.9" y1="20.32" x2="88.9" y2="22.86" width="0.1524" layer="91"/>
+<wire x1="88.9" y1="20.32" x2="83.82" y2="20.32" width="0.1524" layer="91"/>
+<pinref part="S1" gate="S" pin="3"/>
+</segment>
+<segment>
 <pinref part="+3V3" gate="G$1" pin="+3V3"/>
-<pinref part="SW2" gate="G$1" pin="P$2"/>
-<wire x1="86.36" y1="15.24" x2="93.98" y2="15.24" width="0.1524" layer="91"/>
-<wire x1="93.98" y1="15.24" x2="93.98" y2="22.86" width="0.1524" layer="91"/>
+<pinref part="S2" gate="S" pin="3"/>
+<wire x1="83.82" y1="7.62" x2="93.98" y2="7.62" width="0.1524" layer="91"/>
+<wire x1="93.98" y1="7.62" x2="93.98" y2="22.86" width="0.1524" layer="91"/>
 </segment>
 </net>
@@
 <segment>
 <pinref part="U$1" gate="G$1" pin="24-SPI-CE0-N"/>
-<wire x1="60.96" y1="20.32" x2="76.2" y2="20.32" width="0.1524" layer="91"/>
-<pinref part="SW1" gate="G$1" pin="P$1"/>
-</segment>
-</net>
-<net name="N$4" class="0">
-<segment>
-<pinref part="U$1" gate="G$1" pin="26-SPI-CE1-N"/>
-<wire x1="60.96" y1="15.24" x2="76.2" y2="15.24" width="0.1524" layer="91"/>
-<pinref part="SW2" gate="G$1" pin="P$1"/>
+<wire x1="60.96" y1="20.32" x2="73.66" y2="20.32" width="0.1524" layer="91"/>
+<pinref part="S1" gate="S" pin="1"/>
 </segment>
 </net>
@@
 <net name="N$7" class="0">
 <segment>
-<wire x1="60.96" y1="25.4" x2="76.2" y2="25.4" width="0.1524" layer="91"/>
-<wire x1="76.2" y1="25.4" x2="76.2" y2="30.48" width="0.1524" layer="91"/>
+<wire x1="60.96" y1="25.4" x2="73.66" y2="25.4" width="0.1524" layer="91"/>
+<wire x1="73.66" y1="25.4" x2="73.66" y2="30.48" width="0.1524" layer="91"/>
 <pinref part="JP1" gate="A" pin="6"/>
-<wire x1="76.2" y1="30.48" x2="106.68" y2="30.48" width="0.1524" layer="91"/>
+<wire x1="73.66" y1="30.48" x2="106.68" y2="30.48" width="0.1524" layer="91"/>
 <pinref part="U$1" gate="G$1" pin="22-GPIO6"/>
 </segment>
@@
 </segment>
 </net>
+<net name="N$2" class="0">
+<segment>
+<pinref part="S2" gate="S" pin="1"/>
+<wire x1="73.66" y1="7.62" x2="68.58" y2="7.62" width="0.1524" layer="91"/>
+<wire x1="68.58" y1="7.62" x2="68.58" y2="15.24" width="0.1524" layer="91"/>
+<pinref part="U$1" gate="G$1" pin="26-SPI-CE1-N"/>
+<wire x1="68.58" y1="15.24" x2="60.96" y2="15.24" width="0.1524" layer="91"/>
+</segment>
+</net>

Commit message: work on shield
Parts:
- removed JP1, JP2: (no value), pinhead:PINHD-1X8
- added C1, C2, C4, C5: 1uF, SparkFun-Capacitors:CAP0805
- added C3: 104, SparkFun-Capacitors:CAP0805
- added R1: 390k/560k, SparkFun-Resistors:RESISTOR0805-RES
- added U$2: USB_AB, SparkFun-Connectors:USB_AB
- added U1: (no value), microbuilder:DISP_OLED_UG-2864HSWEG010.96"
- S1, S2: value (none) -> SWITCH-MOMENTARY-2PTH; device SparkFun:TAC_SWITCHPTH -> SparkFun-Electromechanical:SWITCH-MOMENTARY-2PTH
Connections:
- new net +5V: U$1.2-+5V, U$2.VBUS
- new net N$1: U$1.19-SPI-MOSI, U1.D1/SPI_SDIN/I2C_SDA
- new net N$10: C1.1, U1.C2P
- new net N$11: C2.1, U1.C1P
- new net N$12: C1.2, U1.C2N
- new net N$13: C2.2, U1.C1N
- new net N$4: U$1.16-GPIO4, U1.DC/I2C_SA0
- net +3V3: now also C3.1, C4.1, S1.2, S2.2, U1.VDD; no longer JP1.1, S1.3, S2.3
- net GND: now also C3.2, C4.2, C5.2, R1.2, U$1.25-DNC, U$1.9-DNC, U$2.GND, U1.BS0, U1.BS1, U1.BS2, U1.NC(GND)@1, U1.NC(GND)@2, U1.VLSS; no longer JP1.8
- net N$5: now also U1.D0/SPI_SCLK/I2C_SCK; no longer JP2.1
- net N$6: now also C5.1, U1.VCOMH; no longer JP2.2, U$1.19-SPI-MOSI
- net N$7: now also U1./CS; no longer JP1.6
- net N$8: now also U1./RES; no longer JP1.3
- net N$9: now also R1.1, U1.IREF; no longer JP1.2, U$1.16-GPIO4

Commit message: work in progress
Parts:
- removed U$1: RASPBERRY-PI, RaspberryPi:RASPBERRY-PI
- added U$3: RASPBERRY-PI_REV1, RaspberryPi:RASPBERRY-PI_REV1
- added U2: CP2110-F01-GM, bxl_import:CP2110-F01-GM
Connections:
- new net N$14: U$2.D-, U2.D-
- new net N$15: U$2.D+, U2.D+
- new net N$16: U$3.GPIO14,UART0_TXD, U2.TX
- new net N$17: U$3.GPIO15,UART0_RXD, U2.RX
- net +3V3: now also U$3.3V3@1; no longer U$1.1-+3V3
- net +5V: now also U$3.5V@2; no longer U$1.2-+5V
- net GND: now also U$3.GND@25, U$3.GND@6, U$3.GND@9, U2.GND, U2.GND_2; no longer U$1.25-DNC, U$1.6-GND, U$1.9-DNC
- net N$1: now also U$3.GPIO10_MOSI; no longer U$1.19-SPI-MOSI
- net N$2: now also U$3.GPIO7,SPI0_CE1; no longer U$1.26-SPI-CE1-N
- net N$3: now also U$3.GPIO8,SPI0_CE0; no longer U$1.24-SPI-CE0-N
- net N$4: now also U$3.GPIO23; no longer U$1.16-GPIO4
- net N$5: now also U$3.GPIO11_SCLK; no longer U$1.23-SPI-SCLK
- net N$7: now also U$3.GPIO25; no longer U$1.22-GPIO6
- net N$8: now also U$3.GPIO24; no longer U$1.18-GPIO5
Other:
- moved on the sheet: S1, S2

Commit message: work in progress
Parts:
- added C6, C7: 1uF, SparkFun-Capacitors:CAP0805
- added C8: 0.1uF, SparkFun-Capacitors:CAP0805
- added R2: 4k7, SparkFun-Resistors:RESISTOR0805-RES
Connections:
- new net N$18: C6.2, U2.REGIN
- new net N$20: R2.2, U2.RST
- net +3V3: now also C7.2, C8.2, R2.1, U2.VDD, U2.VIO
- net +5V: now also U2.VBUS
- net GND: now also C6.1, C7.1, C8.1
Changed lines of the file:
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@@
 <part name="GND10" library="supply1" deviceset="GND" device=""/>
 <part name="U$3" library="RaspberryPi" deviceset="RASPBERRY-PI_REV1" device=""/>
+<part name="P+3" library="supply1" deviceset="+5V" device=""/>
+<part name="C6" library="SparkFun-Capacitors" deviceset="CAP" device="0805" value="1uF"/>
+<part name="GND11" library="supply1" deviceset="GND" device=""/>
+<part name="R2" library="SparkFun-Resistors" deviceset="RESISTOR" device="0805-RES" value="4k7"/>
+<part name="+3V5" library="supply1" deviceset="+3V3" device=""/>
+<part name="C7" library="SparkFun-Capacitors" deviceset="CAP" device="0805" value="1uF"/>
+<part name="C8" library="SparkFun-Capacitors" deviceset="CAP" device="0805" value="0.1uF"/>
 </parts>
 <sheets>
@@
 <instance part="GND10" gate="1" x="187.96" y="73.66"/>
 <instance part="U$3" gate="G$1" x="33.02" y="50.8"/>
+<instance part="P+3" gate="1" x="185.42" y="71.12"/>
+<instance part="C6" gate="G$1" x="187.96" y="43.18" rot="R180"/>
+<instance part="GND11" gate="1" x="195.58" y="30.48"/>
+<instance part="R2" gate="G$1" x="198.12" y="55.88" rot="R180"/>
+<instance part="+3V5" gate="G$1" x="203.2" y="71.12"/>
+<instance part="C7" gate="G$1" x="195.58" y="43.18" rot="R180"/>
+<instance part="C8" gate="G$1" x="203.2" y="43.18" rot="R180"/>
 </instances>
 <busses>
@@
 <pinref part="C4" gate="G$1" pin="1"/>
 <junction x="15.24" y="-12.7"/>
+</segment>
+<segment>
+<pinref part="U2" gate="A" pin="VIO"/>
+<wire x1="177.8" y1="66.04" x2="203.2" y2="66.04" width="0.1524" layer="91"/>
+<wire x1="203.2" y1="66.04" x2="203.2" y2="63.5" width="0.1524" layer="91"/>
+<pinref part="U2" gate="A" pin="VDD"/>
+<wire x1="203.2" y1="63.5" x2="177.8" y2="63.5" width="0.1524" layer="91"/>
+<pinref part="R2" gate="G$1" pin="1"/>
+<wire x1="203.2" y1="55.88" x2="203.2" y2="63.5" width="0.1524" layer="91"/>
+<junction x="203.2" y="63.5"/>
+<pinref part="+3V5" gate="G$1" pin="+3V3"/>
+<wire x1="203.2" y1="68.58" x2="203.2" y2="66.04" width="0.1524" layer="91"/>
+<junction x="203.2" y="66.04"/>
+<pinref part="C8" gate="G$1" pin="2"/>
+<wire x1="203.2" y1="55.88" x2="203.2" y2="48.26" width="0.1524" layer="91"/>
+<junction x="203.2" y="55.88"/>
+<pinref part="C7" gate="G$1" pin="2"/>
+<wire x1="203.2" y1="48.26" x2="203.2" y2="45.72" width="0.1524" layer="91"/>
+<wire x1="195.58" y1="45.72" x2="195.58" y2="48.26" width="0.1524" layer="91"/>
+<wire x1="195.58" y1="48.26" x2="203.2" y2="48.26" width="0.1524" layer="91"/>
+<junction x="203.2" y="48.26"/>
 </segment>
 </net>
@@
 <wire x1="68.58" y1="66.04" x2="71.12" y2="66.04" width="0.1524" layer="91"/>
 </segment>
+<segment>
+<pinref part="C6" gate="G$1" pin="1"/>
+<wire x1="187.96" y1="38.1" x2="187.96" y2="35.56" width="0.1524" layer="91"/>
+<wire x1="187.96" y1="35.56" x2="195.58" y2="35.56" width="0.1524" layer="91"/>
+<wire x1="195.58" y1="35.56" x2="195.58" y2="33.02" width="0.1524" layer="91"/>
+<pinref part="GND11" gate="1" pin="GND"/>
+<pinref part="C8" gate="G$1" pin="1"/>
+<wire x1="203.2" y1="38.1" x2="203.2" y2="35.56" width="0.1524" layer="91"/>
+<wire x1="203.2" y1="35.56" x2="195.58" y2="35.56" width="0.1524" layer="91"/>
+<junction x="195.58" y="35.56"/>
+<pinref part="C7" gate="G$1" pin="1"/>
+<wire x1="195.58" y1="35.56" x2="195.58" y2="38.1" width="0.1524" layer="91"/>
+</segment>
 </net>
 <net name="N$3" class="0">
@@
 <wire x1="139.7" y1="27.94" x2="139.7" y2="30.48" width="0.1524" layer="91"/>
 </segment>
+<segment>
+<pinref part="U2" gate="A" pin="VBUS"/>
+<pinref part="P+3" gate="1" pin="+5V"/>
+<wire x1="177.8" y1="58.42" x2="185.42" y2="58.42" width="0.1524" layer="91"/>
+<wire x1="185.42" y1="58.42" x2="185.42" y2="68.58" width="0.1524" layer="91"/>
+</segment>
 </net>
 <net name="N$10" class="0">
@@
 <segment>
 <pinref part="U$2" gate="G$1" pin="D-"/>
-<wire x1="132.08" y1="25.4" x2="185.42" y2="25.4" width="0.1524" layer="91"/>
-<wire x1="185.42" y1="25.4" x2="185.42" y2="68.58" width="0.1524" layer="91"/>
+<wire x1="132.08" y1="25.4" x2="180.34" y2="25.4" width="0.1524" layer="91"/>
+<wire x1="180.34" y1="25.4" x2="180.34" y2="68.58" width="0.1524" layer="91"/>
 <pinref part="U2" gate="A" pin="D-"/>
-<wire x1="185.42" y1="68.58" x2="177.8" y2="68.58" width="0.1524" layer="91"/>
+<wire x1="180.34" y1="68.58" x2="177.8" y2="68.58" width="0.1524" layer="91"/>
 </segment>
 </net>
@@
 <segment>
 <pinref part="U$2" gate="G$1" pin="D+"/>
-<wire x1="132.08" y1="22.86" x2="187.96" y2="22.86" width="0.1524" layer="91"/>
-<wire x1="187.96" y1="22.86" x2="187.96" y2="71.12" width="0.1524" layer="91"/>
+<wire x1="132.08" y1="22.86" x2="182.88" y2="22.86" width="0.1524" layer="91"/>
+<wire x1="182.88" y1="22.86" x2="182.88" y2="71.12" width="0.1524" layer="91"/>
 <pinref part="U2" gate="A" pin="D+"/>
-<wire x1="187.96" y1="71.12" x2="177.8" y2="71.12" width="0.1524" layer="91"/>
+<wire x1="182.88" y1="71.12" x2="177.8" y2="71.12" width="0.1524" layer="91"/>
 </segment>
 </net>
@@
 </segment>
 </net>
+<net name="N$18" class="0">
+<segment>
+<pinref part="U2" gate="A" pin="REGIN"/>
+<pinref part="C6" gate="G$1" pin="2"/>
+<wire x1="177.8" y1="60.96" x2="187.96" y2="60.96" width="0.1524" layer="91"/>
+<wire x1="187.96" y1="60.96" x2="187.96" y2="45.72" width="0.1524" layer="91"/>
+</segment>
+</net>
+<net name="N$20" class="0">
+<segment>
+<pinref part="U2" gate="A" pin="RST"/>
+<wire x1="193.04" y1="55.88" x2="177.8" y2="55.88" width="0.1524" layer="91"/>
+<pinref part="R2" gate="G$1" pin="2"/>
+</segment>
+</net>

Commit message: raspi shield
Connections:
- net N$14 renamed USB_D_N
- net N$15 renamed USB_D_P
Changed lines of the file:
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@@
 </segment>
 </net>
-<net name="N$14" class="0">
+<net name="USB_D_N" class="0">
 <segment>
 <pinref part="U$2" gate="G$1" pin="D-"/>
@@
 </segment>
 </net>
-<net name="N$15" class="0">
+<net name="USB_D_P" class="0">
 <segment>
 <pinref part="U$2" gate="G$1" pin="D+"/>

Commit message: work snapshot
Parts:
- C3: value 104 -> 0.1uF
Changed lines of the file:
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@@
 <part name="C1" library="SparkFun-Capacitors" deviceset="CAP" device="0805" value="1uF"/>
 <part name="C2" library="SparkFun-Capacitors" deviceset="CAP" device="0805" value="1uF"/>
-<part name="C3" library="SparkFun-Capacitors" deviceset="CAP" device="0805" value="104"/>
+<part name="C3" library="SparkFun-Capacitors" deviceset="CAP" device="0805" value="0.1uF"/>
 <part name="C4" library="SparkFun-Capacitors" deviceset="CAP" device="0805" value="1uF"/>
 <part name="GND6" library="supply1" deviceset="GND" device=""/>
