File: raspi.sch (EAGLE design)
At the start: 16 parts, among them U2 CP2110-F01-GM

Commit message: work on rpi
Parts:
- added C9: 4.7uF, SparkFun-Capacitors:CAP0805
- U1: value (none) -> DISPLAY
Connections:
- removed net N$18: C6.2, U2.REGIN
- new net N$14: C9.2, U2.VPP
- net +5V: now also C6.2, U2.REGIN
- net GND: now also C9.1
- net N$16: now also U$3.GPIO15,UART0_RXD; no longer U$3.GPIO14,UART0_TXD
- net N$17: now also U$3.GPIO14,UART0_TXD; no longer U$3.GPIO15,UART0_RXD
Changed lines of the file:
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@@
 <part name="+3V3" library="supply1" deviceset="+3V3" device=""/>
 <part name="U$2" library="SparkFun-Connectors" deviceset="USB_AB" device=""/>
-<part name="U1" library="microbuilder" deviceset="DISP_OLED_UG-2864HSWEG01" device="0.96&quot;"/>
+<part name="U1" library="microbuilder" deviceset="DISP_OLED_UG-2864HSWEG01" device="0.96&quot;" value="DISPLAY"/>
 <part name="+3V4" library="supply1" deviceset="+3V3" device=""/>
 <part name="GND3" library="supply1" deviceset="GND" device=""/>
@@
 <part name="C7" library="SparkFun-Capacitors" deviceset="CAP" device="0805" value="1uF"/>
 <part name="C8" library="SparkFun-Capacitors" deviceset="CAP" device="0805" value="0.1uF"/>
+<part name="C9" library="SparkFun-Capacitors" deviceset="CAP" device="0805" value="4.7uF"/>
+<part name="GND12" library="supply1" deviceset="GND" device=""/>
 </parts>
 <sheets>
@@
 <instance part="GND10" gate="1" x="187.96" y="73.66"/>
 <instance part="U$3" gate="G$1" x="33.02" y="50.8"/>
-<instance part="P+3" gate="1" x="185.42" y="71.12"/>
+<instance part="P+3" gate="1" x="193.04" y="71.12"/>
 <instance part="C6" gate="G$1" x="187.96" y="43.18" rot="R180"/>
 <instance part="GND11" gate="1" x="195.58" y="30.48"/>
@@
 <instance part="C7" gate="G$1" x="195.58" y="43.18" rot="R180"/>
 <instance part="C8" gate="G$1" x="203.2" y="43.18" rot="R180"/>
+<instance part="C9" gate="G$1" x="83.82" y="40.64" rot="R180"/>
+<instance part="GND12" gate="1" x="83.82" y="30.48"/>
 </instances>
 <busses>
@@
 <wire x1="195.58" y1="35.56" x2="195.58" y2="38.1" width="0.1524" layer="91"/>
 </segment>
+<segment>
+<pinref part="C9" gate="G$1" pin="1"/>
+<wire x1="83.82" y1="35.56" x2="83.82" y2="33.02" width="0.1524" layer="91"/>
+<pinref part="GND12" gate="1" pin="GND"/>
+</segment>
 </net>
 <net name="N$3" class="0">
@@
 </segment>
 <segment>
+<pinref part="P+3" gate="1" pin="+5V"/>
+<wire x1="193.04" y1="60.96" x2="193.04" y2="68.58" width="0.1524" layer="91"/>
 <pinref part="U2" gate="A" pin="VBUS"/>
-<pinref part="P+3" gate="1" pin="+5V"/>
 <wire x1="177.8" y1="58.42" x2="185.42" y2="58.42" width="0.1524" layer="91"/>
-<wire x1="185.42" y1="58.42" x2="185.42" y2="68.58" width="0.1524" layer="91"/>
+<pinref part="U2" gate="A" pin="REGIN"/>
+<pinref part="C6" gate="G$1" pin="2"/>
+<wire x1="177.8" y1="60.96" x2="187.96" y2="60.96" width="0.1524" layer="91"/>
+<wire x1="187.96" y1="60.96" x2="187.96" y2="58.42" width="0.1524" layer="91"/>
+<wire x1="187.96" y1="58.42" x2="187.96" y2="45.72" width="0.1524" layer="91"/>
+<wire x1="185.42" y1="58.42" x2="187.96" y2="58.42" width="0.1524" layer="91"/>
+<junction x="187.96" y="58.42"/>
+<wire x1="187.96" y1="60.96" x2="193.04" y2="60.96" width="0.1524" layer="91"/>
+<junction x="187.96" y="60.96"/>
 </segment>
 </net>
@@
 <net name="N$16" class="0">
 <segment>
-<wire x1="60.96" y1="58.42" x2="76.2" y2="58.42" width="0.1524" layer="91"/>
-<wire x1="76.2" y1="58.42" x2="76.2" y2="66.04" width="0.1524" layer="91"/>
 <pinref part="U2" gate="A" pin="TX"/>
 <wire x1="76.2" y1="66.04" x2="86.36" y2="66.04" width="0.1524" layer="91"/>
-<pinref part="U$3" gate="G$1" pin="GPIO14,UART0_TXD"/>
+<pinref part="U$3" gate="G$1" pin="GPIO15,UART0_RXD"/>
+<wire x1="60.96" y1="55.88" x2="76.2" y2="55.88" width="0.1524" layer="91"/>
+<wire x1="76.2" y1="55.88" x2="76.2" y2="66.04" width="0.1524" layer="91"/>
 </segment>
 </net>
 <net name="N$17" class="0">
 <segment>
-<wire x1="60.96" y1="55.88" x2="78.74" y2="55.88" width="0.1524" layer="91"/>
-<wire x1="78.74" y1="55.88" x2="78.74" y2="63.5" width="0.1524" layer="91"/>
 <pinref part="U2" gate="A" pin="RX"/>
 <wire x1="78.74" y1="63.5" x2="86.36" y2="63.5" width="0.1524" layer="91"/>
-<pinref part="U$3" gate="G$1" pin="GPIO15,UART0_RXD"/>
-</segment>
-</net>
-<net name="N$18" class="0">
-<segment>
-<pinref part="U2" gate="A" pin="REGIN"/>
-<pinref part="C6" gate="G$1" pin="2"/>
-<wire x1="177.8" y1="60.96" x2="187.96" y2="60.96" width="0.1524" layer="91"/>
-<wire x1="187.96" y1="60.96" x2="187.96" y2="45.72" width="0.1524" layer="91"/>
+<wire x1="78.74" y1="63.5" x2="78.74" y2="58.42" width="0.1524" layer="91"/>
+<pinref part="U$3" gate="G$1" pin="GPIO14,UART0_TXD"/>
+<wire x1="78.74" y1="58.42" x2="60.96" y2="58.42" width="0.1524" layer="91"/>
 </segment>
 </net>
@@
 </segment>
 </net>
+<net name="N$14" class="0">
+<segment>
+<pinref part="U2" gate="A" pin="VPP"/>
+<pinref part="C9" gate="G$1" pin="2"/>
+<wire x1="86.36" y1="53.34" x2="83.82" y2="53.34" width="0.1524" layer="91"/>
+<wire x1="83.82" y1="53.34" x2="83.82" y2="43.18" width="0.1524" layer="91"/>
+</segment>
+</net>
