File: raspi.sch (EAGLE design)
At the start: 17 parts, among them U1 DISPLAY, U2 CP2110-F01-GM

Commit message: wip
Parts:
- C5: value 1uF -> 2.2uF
- R1: value 390k/560k -> 390k
Connections:
- net +3V3: now also U1.VBAT
- net N$10: now also C2.1; no longer C1.1
- net N$11: now also C1.1; no longer C2.1
- net N$12: now also C2.2; no longer C1.2
- net N$13: now also C1.2; no longer C2.2
Other:
- moved on the sheet: C1, C2, C3, C4, C5, R1

Commit message: raspi work
Parts:
- S1, S2: value SWITCH-MOMENTARY-2PTH -> SWITCH-MOMENTARY-2; device SparkFun-Electromechanical:SWITCH-MOMENTARY-2PTH -> SparkFun-Electromechanical:SWITCH-MOMENTARY-2
Changed lines of the file:
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@@
 <part name="U1" library="microbuilder" deviceset="DISP_OLED_UG-2864HSWEG01" device="0.96&quot;" value="DISPLAY"/>
 <part name="+3V4" library="supply1" deviceset="+3V3" device=""/>
-<part name="S1" library="SparkFun-Electromechanical" deviceset="SWITCH-MOMENTARY-2" device="PTH"/>
-<part name="S2" library="SparkFun-Electromechanical" deviceset="SWITCH-MOMENTARY-2" device="PTH"/>
+<part name="S1" library="SparkFun-Electromechanical" deviceset="SWITCH-MOMENTARY-2" device="" value="SWITCH-MOMENTARY-2"/>
+<part name="S2" library="SparkFun-Electromechanical" deviceset="SWITCH-MOMENTARY-2" device="" value="SWITCH-MOMENTARY-2"/>
 <part name="P+1" library="supply1" deviceset="+5V" device=""/>
 <part name="P+2" library="supply1" deviceset="+5V" device=""/>

Commit message: rework BOMs
Parts:
- removed U$2: USB_AB, SparkFun-Connectors:USB_AB
- added USB: (no value), fabhack:47346-0001
Connections:
- net +5V: now also USB.VBUS; no longer U$2.VBUS
- net GND: now also USB.GND; no longer U$2.GND
- net USB_D_N: now also USB.D-; no longer U$2.D-
- net USB_D_P: now also USB.D+; no longer U$2.D+
Changed lines of the file:
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@@
 <layer number="54" name="bGND_GNDA" color="1" fill="9" visible="no" active="no"/>
 <layer number="56" name="wert" color="7" fill="1" visible="no" active="no"/>
+<layer number="59" name="tCarbon" color="7" fill="1" visible="no" active="no"/>
+<layer number="60" name="bCarbon" color="7" fill="1" visible="no" active="no"/>
 <layer number="91" name="Nets" color="2" fill="1" visible="yes" active="yes"/>
 <layer number="92" name="Busses" color="1" fill="1" visible="yes" active="yes"/>
@@
 <layer number="121" name="sName" color="7" fill="1" visible="yes" active="yes"/>
 <layer number="122" name="_bPlace" color="7" fill="1" visible="yes" active="yes"/>
+<layer number="123" name="tTestmark" color="7" fill="1" visible="yes" active="yes"/>
+<layer number="124" name="bTestmark" color="7" fill="1" visible="yes" active="yes"/>
 <layer number="125" name="_tNames" color="7" fill="1" visible="yes" active="yes"/>
 <layer number="126" name="_bNames" color="7" fill="1" visible="yes" active="yes"/>
 <layer number="127" name="_tValues" color="7" fill="1" visible="yes" active="yes"/>
 <layer number="128" name="_bValues" color="7" fill="1" visible="yes" active="yes"/>
+<layer number="129" name="Mask" color="7" fill="1" visible="yes" active="yes"/>
+<layer number="131" name="tAdjust" color="7" fill="1" visible="yes" active="yes"/>
+<layer number="132" name="bAdjust" color="7" fill="1" visible="yes" active="yes"/>
 <layer number="144" name="Drill_legend" color="7" fill="1" visible="yes" active="yes"/>
 <layer number="151" name="HeatSink" color="7" fill="1" visible="yes" active="yes"/>
@@
 <part name="+3V2" library="supply1" deviceset="+3V3" device=""/>
 <part name="+3V3" library="supply1" deviceset="+3V3" device=""/>
-<part name="U$2" library="SparkFun-Connectors" deviceset="USB_AB" device=""/>
+<part name="USB" library="fabhack" deviceset="47346-0001" device=""/>
 <part name="U1" library="microbuilder" deviceset="DISP_OLED_UG-2864HSWEG01" device="0.96&quot;" value="DISPLAY"/>
 <part name="+3V4" library="supply1" deviceset="+3V3" device=""/>
@@
 <instance part="+3V2" gate="G$1" x="93.98" y="25.4"/>
 <instance part="+3V3" gate="G$1" x="99.06" y="25.4"/>
-<instance part="U$2" gate="G$1" x="127" y="22.86" rot="R180"/>
+<instance part="USB" gate="G$1" x="124.46" y="22.86" rot="MR0"/>
 <instance part="U1" gate="G$1" x="30.48" y="-53.34" rot="MR270"/>
 <instance part="+3V4" gate="G$1" x="15.24" y="-5.08"/>
@@
 <segment>
 <pinref part="GND4" gate="1" pin="GND"/>
-<wire x1="132.08" y1="17.78" x2="139.7" y2="17.78" width="0.1524" layer="91"/>
+<wire x1="134.62" y1="17.78" x2="139.7" y2="17.78" width="0.1524" layer="91"/>
 <wire x1="139.7" y1="17.78" x2="139.7" y2="15.24" width="0.1524" layer="91"/>
-<pinref part="U$2" gate="G$1" pin="GND"/>
+<pinref part="USB" gate="G$1" pin="GND"/>
 </segment>
 <segment>
@@
 </segment>
 <segment>
-<pinref part="U$2" gate="G$1" pin="VBUS"/>
+<pinref part="USB" gate="G$1" pin="VBUS"/>
 <pinref part="P+2" gate="1" pin="+5V"/>
-<wire x1="132.08" y1="27.94" x2="139.7" y2="27.94" width="0.1524" layer="91"/>
+<wire x1="134.62" y1="27.94" x2="139.7" y2="27.94" width="0.1524" layer="91"/>
 <wire x1="139.7" y1="27.94" x2="139.7" y2="30.48" width="0.1524" layer="91"/>
 </segment>
@@
 <net name="USB_D_N" class="0">
 <segment>
-<pinref part="U$2" gate="G$1" pin="D-"/>
-<wire x1="132.08" y1="25.4" x2="180.34" y2="25.4" width="0.1524" layer="91"/>
+<pinref part="USB" gate="G$1" pin="D-"/>
+<wire x1="134.62" y1="25.4" x2="180.34" y2="25.4" width="0.1524" layer="91"/>
 <wire x1="180.34" y1="25.4" x2="180.34" y2="68.58" width="0.1524" layer="91"/>
 <pinref part="U2" gate="A" pin="D-"/>
@@
 <net name="USB_D_P" class="0">
 <segment>
-<pinref part="U$2" gate="G$1" pin="D+"/>
-<wire x1="132.08" y1="22.86" x2="182.88" y2="22.86" width="0.1524" layer="91"/>
+<pinref part="USB" gate="G$1" pin="D+"/>
+<wire x1="134.62" y1="22.86" x2="182.88" y2="22.86" width="0.1524" layer="91"/>
 <wire x1="182.88" y1="22.86" x2="182.88" y2="71.12" width="0.1524" layer="91"/>
 <pinref part="U2" gate="A" pin="D+"/>

Commit message: raspi
Parts:
- S1, S2: value SWITCH-MOMENTARY-2 -> SWITCH-MOMENTARY-2SMD; device SparkFun-Electromechanical:SWITCH-MOMENTARY-2 -> SparkFun-Electromechanical:SWITCH-MOMENTARY-2SMD
Changed lines of the file:
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@@
 <part name="U1" library="microbuilder" deviceset="DISP_OLED_UG-2864HSWEG01" device="0.96&quot;" value="DISPLAY"/>
 <part name="+3V4" library="supply1" deviceset="+3V3" device=""/>
-<part name="S1" library="SparkFun-Electromechanical" deviceset="SWITCH-MOMENTARY-2" device="" value="SWITCH-MOMENTARY-2"/>
-<part name="S2" library="SparkFun-Electromechanical" deviceset="SWITCH-MOMENTARY-2" device="" value="SWITCH-MOMENTARY-2"/>
+<part name="S1" library="SparkFun-Electromechanical" deviceset="SWITCH-MOMENTARY-2" device="SMD" value="SWITCH-MOMENTARY-2SMD"/>
+<part name="S2" library="SparkFun-Electromechanical" deviceset="SWITCH-MOMENTARY-2" device="SMD" value="SWITCH-MOMENTARY-2SMD"/>
 <part name="P+1" library="supply1" deviceset="+5V" device=""/>
 <part name="P+2" library="supply1" deviceset="+5V" device=""/>

Commit message: rework swd programmer
Connections:
- net GND: now also U1.VSS
Changed lines of the file:
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@@
 <pinref part="U1" gate="G$1" pin="VBAT"/>
 <wire x1="7.62" y1="-27.94" x2="7.62" y2="-25.4" width="0.1524" layer="91"/>
-<wire x1="7.62" y1="-25.4" x2="15.24" y2="-25.4" width="0.1524" layer="91"/>
-<junction x="15.24" y="-25.4"/>
+<wire x1="15.24" y1="-20.32" x2="7.62" y2="-20.32" width="0.1524" layer="91"/>
+<wire x1="7.62" y1="-20.32" x2="7.62" y2="-25.4" width="0.1524" layer="91"/>
 </segment>
 <segment>
@@
 <junction x="22.86" y="-20.32"/>
 <wire x1="22.86" y1="-22.86" x2="22.86" y2="-25.4" width="0.1524" layer="91"/>
+<pinref part="U1" gate="G$1" pin="VSS"/>
+<wire x1="17.78" y1="-25.4" x2="12.7" y2="-25.4" width="0.1524" layer="91"/>
+<wire x1="12.7" y1="-25.4" x2="12.7" y2="-27.94" width="0.1524" layer="91"/>
+<junction x="17.78" y="-25.4"/>
 </segment>
 </net>
