File: trezor.brd (EAGLE design)
At the start: 50 x 26.7 mm, 39 parts, among them IC1 MCP1703CB, Q2 16MHz, U1 ATSHA204-TSU, U2 USB, U3 DISPLAY, U5 TPD4S012_DRY_6

Commit message: work snapshot
Parts:
- removed U5: TPD4S012_DRY_6, imported:DRY6
- C20: device SparkFun-Passives:0402-CAP -> SparkFun-Passives:0805
- C3: value 104 -> 0.1uF
- moved C20 2.03 mm to (14.3, 5.64)
Connections:
- removed net N$3: U2.ID, U5.3
- net +5V: no longer U2.VBUS, U5.6
- net GND: no longer U2.GND, U5.4
- net USB_D_N: no longer U5.2
- net USB_D_P: no longer U5.1
Routing:
- net +3V3: track 119.2 -> 0.00 mm, vias 1 -> 0
- net USB_D_N: track 37.6 -> 0.00 mm, vias 1 -> 0
- net N$23: track 34.2 -> 0.00 mm, vias 1 -> 0
- net USB_D_P: track 31.6 -> 0.00 mm, vias 1 -> 0
- net SDA: track 28.5 -> 0.00 mm
- net N$5: track 21.5 -> 0.00 mm, vias 2 -> 0
- net N$1: track 15.8 -> 0.00 mm
- net N$16: track 14.9 -> 0.00 mm
- net +5V: track 14.6 -> 0.00 mm
- net N$15: track 14.0 -> 0.00 mm, vias 1 -> 0
- net N$2: track 12.8 -> 0.00 mm, vias 2 -> 0
- net XTAL1: track 12.2 -> 0.00 mm
- net XTAL2: track 11.0 -> 0.00 mm
- net N$3: track 10.5 -> 0.00 mm, vias 2 -> 0
- net N$14: track 10.0 -> 0.00 mm, vias 1 -> 0
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
Commit message: forgot to connect usb gnd/vcc
Connections:
- net +5V: now also U2.VBUS
- net GND: now also U2.GND
Changed lines of the file:
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@@
 <vertex x="-1.016" y="-0.4064"/>
 </polygon>
-<wire x1="35.5092" y1="23.5354" x2="36.52018125" y2="17.8958375" width="0" layer="19" extent="16-16"/>
-<wire x1="28.105609375" y1="10.188371875" x2="26.33784375" y2="11.956140625" width="0" layer="19" extent="16-16"/>
+<contactref element="U2" pad="GND"/>
+<wire x1="42.4496" y1="22.785" x2="42.4496" y2="23.485" width="0" layer="19" extent="16-16"/>
+<wire x1="39.7256" y1="23.8864" x2="42.4496" y2="23.485" width="0" layer="19" extent="16-16"/>
+<wire x1="38.2524" y1="23.8356" x2="39.7256" y2="23.8864" width="0" layer="19" extent="16-16"/>
+<wire x1="36.8554" y1="23.7594" x2="38.2524" y2="23.8356" width="0" layer="19" extent="16-16"/>
+<wire x1="35.5092" y1="23.5354" x2="36.8554" y2="23.7594" width="0" layer="19" extent="16-16"/>
+<wire x1="44.5516" y1="19.416" x2="42.4496" y2="22.785" width="0" layer="19" extent="16-16"/>
+<wire x1="36.52018125" y1="17.8958375" x2="35.5092" y2="23.5354" width="0" layer="19" extent="16-16"/>
+<wire x1="38.995053125" y1="11.249034375" x2="36.52018125" y2="17.8958375" width="0" layer="19" extent="16-16"/>
+<wire x1="42.4496" y1="10.885" x2="38.995053125" y2="11.249034375" width="0" layer="19" extent="16-16"/>
+<wire x1="42.4496" y1="10.185" x2="42.4496" y2="10.885" width="0" layer="19" extent="16-16"/>
+<wire x1="42.4496" y1="9.485" x2="42.4496" y2="10.185" width="0" layer="19" extent="16-16"/>
+<wire x1="35.813071875" y1="8.067053125" x2="38.995053125" y2="11.249034375" width="0" layer="19" extent="16-16"/>
+<wire x1="35.4662" y1="2.667" x2="35.813071875" y2="8.067053125" width="0" layer="19" extent="16-16"/>
+<wire x1="36.9062" y1="1.9662" x2="35.4662" y2="2.667" width="0" layer="19" extent="16-16"/>
+<wire x1="38.8837" y1="2.5261" x2="36.9062" y2="1.9662" width="0" layer="19" extent="16-16"/>
+<wire x1="42.4496" y1="3.185" x2="38.8837" y2="2.5261" width="0" layer="19" extent="16-16"/>
+<wire x1="28.4816" y1="2.2283" x2="35.4662" y2="2.667" width="0" layer="19" extent="16-16"/>
+<wire x1="28.5075" y1="3.9069" x2="28.4816" y2="2.2283" width="0" layer="19" extent="16-16"/>
 <wire x1="25.8826" y1="3.6322" x2="28.5075" y2="3.9069" width="0" layer="19" extent="1-16"/>
+<wire x1="28.105609375" y1="10.188371875" x2="28.5075" y2="3.9069" width="0" layer="19" extent="16-16"/>
+<wire x1="26.33784375" y1="11.956140625" x2="28.105609375" y2="10.188371875" width="0" layer="19" extent="16-16"/>
 <wire x1="26.691396875" y1="15.067409375" x2="26.33784375" y2="11.956140625" width="0" layer="19" extent="16-16"/>
+<wire x1="27.04495" y1="15.4209625" x2="26.691396875" y2="15.067409375" width="0" layer="19" extent="16-16"/>
 <wire x1="28.4591625" y1="16.835178125" x2="27.04495" y2="15.4209625" width="0" layer="19" extent="16-16"/>
-<wire x1="38.995053125" y1="11.249034375" x2="42.4496" y2="10.885" width="0" layer="19" extent="16-16"/>
-<wire x1="35.813071875" y1="8.067053125" x2="38.995053125" y2="11.249034375" width="0" layer="19" extent="16-16"/>
+<wire x1="20.7518" y1="11.923" x2="26.33784375" y2="11.956140625" width="0" layer="19" extent="16-16"/>
+<wire x1="17.8617" y1="11.5364" x2="20.7518" y2="11.923" width="0" layer="19" extent="16-16"/>
+<wire x1="16.1221" y1="11.3434" x2="17.8617" y2="11.5364" width="0" layer="19" extent="16-16"/>
+<wire x1="20.97" y1="16.0782" x2="20.7518" y2="11.923" width="0" layer="19" extent="16-16"/>
+<wire x1="16.0528" y1="6.1826" x2="16.1221" y2="11.3434" width="0" layer="19" extent="1-16"/>
+<wire x1="14.3002" y1="4.7388" x2="16.0528" y2="6.1826" width="0" layer="19" extent="1-1"/>
+<wire x1="12.5222" y1="5.9286" x2="14.3002" y2="4.7388" width="0" layer="19" extent="1-1"/>
+<wire x1="10.7442" y1="6.7414" x2="12.5222" y2="5.9286" width="0" layer="19" extent="1-1"/>
+<wire x1="13.6398" y1="17.6888" x2="16.1221" y2="11.3434" width="0" layer="19" extent="1-16"/>
+<wire x1="11.5394" y1="17.2872" x2="13.6398" y2="17.6888" width="0" layer="19" extent="1-1"/>
+<wire x1="7.2644" y1="17.4094" x2="11.5394" y2="17.2872" width="0" layer="19" extent="1-1"/>
+<wire x1="4.9328" y1="12.0604" x2="7.2644" y2="17.4094" width="0" layer="19" extent="1-1"/>
+<wire x1="22.0726" y1="23.0378" x2="20.97" y2="16.0782" width="0" layer="19" extent="1-16"/>
+<wire x1="25.7706" y1="23.876" x2="22.0726" y2="23.0378" width="0" layer="19" extent="1-16"/>
 </signal>
 <signal name="VSS">
@@
 <contactref element="C10" pad="2"/>
 <contactref element="IC1" pad="3"/>
+<contactref element="U2" pad="VBUS"/>
 <wire x1="7.2644" y1="18.7094" x2="9.3394" y2="18.2372" width="0" layer="19" extent="1-1"/>
+<wire x1="4.9328" y1="14.6604" x2="7.2644" y2="18.7094" width="0" layer="19" extent="1-1"/>
 </signal>
 <signal name="SDA">

Commit message: wip
Parts:
- added TP5, TP6: (no value), microbuilder:TESTPOINT_ROUND_0.5MM
- TP1, TP2, TP3, TP4: value PTR1TP10R -> (none); device testpad:TP10R -> microbuilder:TESTPOINT_ROUND_0.5MM
- moved C17 30.8 mm to (18.4, 24.9), flipped to the top, turned to 180 degrees
- moved U1 28.1 mm to (6.93, 8.76), flipped to the top
- moved R3 27.1 mm to (15.6, 5.05), flipped to the top, turned to 0 degrees
- moved C16 25.9 mm to (24.2, 1.80), flipped to the top, turned to 0 degrees
- moved TP1 25.2 mm to (11.6, 10.2), flipped to the top
- moved C6 24.6 mm to (12.4, 5.00), flipped to the top, turned to 0 degrees
- moved R4 23.0 mm to (19.2, 5.00), flipped to the top, turned to 0 degrees
- moved R2 22.4 mm to (9.58, 6.48), flipped to the top, turned to 0 degrees
- moved TP2 21.3 mm to (14.8, 10.2), flipped to the top
- moved TP3 20.7 mm to (14.0, 10.2), flipped to the top
- moved TP4 20.2 mm to (13.2, 10.2), flipped to the top
- moved C19 18.5 mm to (15.2, 24.9), turned to 0 degrees
- moved U$1 17.9 mm to (15.1, 13.3), flipped to the top, turned to 180 degrees
- moved C12 15.4 mm to (13.8, 2.64), flipped to the top, turned to 270 degrees
- moved C4 14.8 mm to (46.9, 11.6), flipped to the top, turned to 90 degrees
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Connections:
- net GND: now also TP6.P$1
- net N$16: now also TP3.P$1; no longer TP2.TP
- net N$17: now also TP2.P$1; no longer TP1.TP
- net N$19: now also TP4.P$1; no longer TP3.TP
- net N$20: now also TP5.P$1; no longer TP4.TP
- net N$21: now also TP1.P$1
Routing:
- net USB_D_N: track 0.00 -> 5.30 mm
- net USB_D_P: track 0.00 -> 5.24 mm
Other:
- outline, holes or cut-outs redrawn

Commit message: wip
Parts:
- removed TP1, TP2, TP3, TP4, TP5, TP6: (no value), microbuilder:TESTPOINT_ROUND_0.5MM
- added X3: SSW-103-02-S-D, con-samtec:SSW-103-02-S-D
Connections:
- net GND: now also X3.6; no longer TP6.P$1
- net N$16: now also X3.3; no longer TP3.P$1
- net N$17: now also X3.5; no longer TP2.P$1
- net N$19: now also X3.4; no longer TP4.P$1
- net N$20: now also X3.1; no longer TP5.P$1
- net N$21: now also X3.2; no longer TP1.P$1
Changed lines of the file:
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@@
 <element name="R5" library="SparkFun-Passives" package="0402-RES" value="10k" x="20.701" y="20.447" rot="R90"/>
 <element name="IC1" library="linear" package="SOT23" value="MCP1703CB" x="6.858" y="17.399"/>
-<element name="TP1" library="microbuilder" package="TESTPOINT_ROUND_0.5MM" value="" x="11.5824" y="10.16"/>
-<element name="TP2" library="microbuilder" package="TESTPOINT_ROUND_0.5MM" value="" x="14.8336" y="10.16"/>
-<element name="TP3" library="microbuilder" package="TESTPOINT_ROUND_0.5MM" value="" x="14.0208" y="10.16"/>
-<element name="TP4" library="microbuilder" package="TESTPOINT_ROUND_0.5MM" value="" x="13.208" y="10.16"/>
-<element name="TP5" library="microbuilder" package="TESTPOINT_ROUND_0.5MM" value="" x="12.3952" y="10.16"/>
-<element name="TP6" library="microbuilder" package="TESTPOINT_ROUND_0.5MM" value="" x="15.6464" y="10.16"/>
+<element name="X3" library="con-samtec" package="SSW-103-02-S-D" value="SSW-103-02-S-D" x="15.1384" y="13.3096">
+<attribute name="OC_NEWARK" value="11P9365" x="15.1384" y="13.3096" size="1.778" layer="27" display="off"/>
+<attribute name="MPN" value="SSW-103-02-S-D" x="15.1384" y="13.3096" size="1.778" layer="27" display="off"/>
+<attribute name="MF" value="" x="15.1384" y="13.3096" size="1.778" layer="27" display="off"/>
+<attribute name="OC_FARNELL" value="unknown" x="15.1384" y="13.3096" size="1.778" layer="27" display="off"/>
+</element>
 </elements>
 <signals>
@@
 </polygon>
 <contactref element="U2" pad="GND"/>
-<contactref element="TP6" pad="P$1"/>
+<contactref element="X3" pad="6"/>
 <wire x1="5.908" y1="16.299" x2="6.5128" y2="14.8082" width="0" layer="19" extent="1-1"/>
 <wire x1="18.7706" y1="1.2844" x2="20.3962" y2="1.6614" width="0" layer="19" extent="1-1"/>
 <wire x1="9.4384" y1="16.085" x2="9.4384" y2="14.085" width="0" layer="19" extent="1-1"/>
-<wire x1="42.4496" y1="23.485" x2="46.8884" y2="24.5514" width="0" layer="19" extent="1-16"/>
 </signal>
 <signal name="VSS">
@@
 <contactref element="U$1" pad="52"/>
 <contactref element="R3" pad="1"/>
-<contactref element="TP2" pad="P$1"/>
-<wire x1="12.8884" y1="7.635" x2="14.8336" y2="10.16" width="0" layer="19" extent="1-1"/>
+<contactref element="X3" pad="5"/>
+<wire x1="12.8884" y1="7.635" x2="17.6784" y2="12.0396" width="0" layer="19" extent="1-1"/>
 <wire x1="14.9964" y1="5.0546" x2="12.8884" y2="7.635" width="0" layer="19" extent="1-1"/>
 </signal>
@@
 <contactref element="U$1" pad="51"/>
 <contactref element="R4" pad="1"/>
-<contactref element="TP3" pad="P$1"/>
-<wire x1="12.3884" y1="7.635" x2="14.0208" y2="10.16" width="0" layer="19" extent="1-1"/>
+<contactref element="X3" pad="3"/>
+<wire x1="12.3884" y1="7.635" x2="15.1384" y2="12.0396" width="0" layer="19" extent="1-1"/>
 <wire x1="18.5016" y1="5.0038" x2="12.3884" y2="7.635" width="0" layer="19" extent="1-1"/>
 </signal>
 <signal name="N$19">
 <contactref element="U$1" pad="50"/>
-<contactref element="TP4" pad="P$1"/>
-<wire x1="11.8884" y1="7.635" x2="13.208" y2="10.16" width="0" layer="19" extent="1-1"/>
+<contactref element="X3" pad="4"/>
+<wire x1="11.8884" y1="7.635" x2="15.1384" y2="14.5796" width="0" layer="19" extent="1-1"/>
 </signal>
 <signal name="N$20">
 <contactref element="U$1" pad="49"/>
-<contactref element="TP5" pad="P$1"/>
-<wire x1="11.3884" y1="7.635" x2="12.3952" y2="10.16" width="0" layer="19" extent="1-1"/>
+<contactref element="X3" pad="1"/>
+<wire x1="11.3884" y1="7.635" x2="12.5984" y2="12.0396" width="0" layer="19" extent="1-1"/>
 </signal>
 <signal name="N$23">
@@
 <contactref element="U$1" pad="38"/>
 <contactref element="C9" pad="2"/>
-<contactref element="TP1" pad="P$1"/>
+<contactref element="X3" pad="2"/>
 <wire x1="20.701" y1="19.797" x2="20.701" y2="22.9466" width="0" layer="19" extent="1-1"/>
-<wire x1="9.4384" y1="14.585" x2="20.701" y2="19.797" width="0" layer="19" extent="1-1"/>
-<wire x1="11.5824" y1="10.16" x2="9.4384" y2="14.585" width="0" layer="19" extent="1-1"/>
+<wire x1="12.5984" y1="14.5796" x2="20.701" y2="19.797" width="0" layer="19" extent="1-1"/>
+<wire x1="9.4384" y1="14.585" x2="12.5984" y2="14.5796" width="0" layer="19" extent="1-1"/>
 </signal>
 <signal name="USB_D_N">

Commit message: wip
Parts:
- C5: value 1uF -> 2.2uF
- R1: value 390k/560k -> 390k
Connections:
- net +3V3: now also U3.6
Changed lines of the file:
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@@
 <element name="C3" library="SparkFun-Passives" package="0402-CAP" value="0.1uF" x="46.8884" y="15.0368" rot="R90"/>
 <element name="C4" library="SparkFun-Passives" package="0402-CAP" value="1uF" x="46.9392" y="11.6332" rot="R90"/>
-<element name="C5" library="SparkFun-Passives" package="0402-CAP" value="1uF" x="46.8884" y="23.9014" rot="R90"/>
-<element name="R1" library="SparkFun-Passives" package="0402-RES" value="390k/560k" x="46.8884" y="18.542" rot="R270"/>
+<element name="C5" library="SparkFun-Passives" package="0402-CAP" value="2.2uF" x="46.8884" y="23.9014" rot="R90"/>
+<element name="R1" library="SparkFun-Passives" package="0402-RES" value="390k" x="46.8884" y="18.542" rot="R270"/>
 <element name="U1" library="SparkFun-DigitalIC" package="SOT23-3" value="ATSHA204-TSU" x="6.9342" y="8.763" rot="R90"/>
 <element name="R2" library="SparkFun-Passives" package="0402-RES" value="100k" x="9.5758" y="6.477"/>
@@
 <contactref element="U$1" pad="39"/>
 <contactref element="U$1" pad="12"/>
-<contactref element="U3" pad="30"/>
-<contactref element="U3" pad="29"/>
-<contactref element="C5" pad="2"/>
-<contactref element="R1" pad="2"/>
-<contactref element="U3" pad="10"/>
-<contactref element="U3" pad="12"/>
-<contactref element="U3" pad="11"/>
 <contactref element="U3" pad="1"/>
-<contactref element="C3" pad="2"/>
-<contactref element="C4" pad="2"/>
 <contactref element="U1" pad="3"/>
 <contactref element="C6" pad="2"/>
@@
 <contactref element="U2" pad="GND"/>
 <contactref element="X3" pad="6"/>
+<contactref element="U3" pad="30"/>
+<contactref element="U3" pad="29"/>
+<contactref element="C5" pad="2"/>
+<contactref element="R1" pad="2"/>
+<contactref element="U3" pad="12"/>
+<contactref element="U3" pad="11"/>
+<contactref element="U3" pad="10"/>
+<contactref element="C3" pad="2"/>
+<contactref element="C4" pad="2"/>
+<wire x1="42.4496" y1="23.485" x2="46.8884" y2="24.5514" width="0" layer="19" extent="1-16"/>
+<wire x1="42.4496" y1="22.785" x2="42.4496" y2="23.485" width="0" layer="19" extent="16-16"/>
+<wire x1="46.8884" y1="17.892" x2="42.4496" y2="22.785" width="0" layer="19" extent="1-16"/>
+<wire x1="46.8884" y1="15.6868" x2="46.8884" y2="17.892" width="0" layer="19" extent="1-1"/>
+<wire x1="46.9392" y1="12.2832" x2="46.8884" y2="15.6868" width="0" layer="19" extent="1-1"/>
+<wire x1="42.4496" y1="10.885" x2="46.9392" y2="12.2832" width="0" layer="19" extent="1-16"/>
+<wire x1="42.4496" y1="10.185" x2="42.4496" y2="10.885" width="0" layer="19" extent="16-16"/>
+<wire x1="42.4496" y1="9.485" x2="42.4496" y2="10.185" width="0" layer="19" extent="16-16"/>
+<wire x1="42.4496" y1="3.185" x2="42.4496" y2="9.485" width="0" layer="19" extent="16-16"/>
+<wire x1="25.9842" y1="3.5306" x2="42.4496" y2="3.185" width="0" layer="19" extent="1-16"/>
+<wire x1="24.8054" y1="1.8034" x2="25.9842" y2="3.5306" width="0" layer="19" extent="1-1"/>
+<wire x1="20.3962" y1="1.6614" x2="24.8054" y2="1.8034" width="0" layer="19" extent="1-1"/>
+<wire x1="18.7706" y1="1.2844" x2="20.3962" y2="1.6614" width="0" layer="19" extent="1-1"/>
+<wire x1="17.0887" y1="1.57" x2="18.7706" y2="1.2844" width="0" layer="19" extent="1-1"/>
+<wire x1="15.4363" y1="1.6128" x2="17.0887" y2="1.57" width="0" layer="19" extent="1-1"/>
+<wire x1="13.7621" y1="1.9933" x2="15.4363" y2="1.6128" width="0" layer="19" extent="1-1"/>
+<wire x1="13.0706" y1="5.0038" x2="13.7621" y2="1.9933" width="0" layer="19" extent="1-1"/>
+<wire x1="14.3884" y1="7.635" x2="13.0706" y2="5.0038" width="0" layer="19" extent="1-1"/>
+<wire x1="23.4038" y1="10.1277" x2="25.9842" y2="3.5306" width="0" layer="19" extent="1-1"/>
+<wire x1="20.8384" y1="10.585" x2="23.4038" y2="10.1277" width="0" layer="19" extent="1-1"/>
+<wire x1="20.8384" y1="15.085" x2="20.8384" y2="10.585" width="0" layer="19" extent="1-1"/>
+<wire x1="23.4546" y1="16.5608" x2="20.8384" y2="15.085" width="0" layer="19" extent="1-1"/>
+<wire x1="17.6784" y1="14.5796" x2="20.8384" y2="15.085" width="0" layer="19" extent="1-1"/>
+<wire x1="13.8884" y1="19.035" x2="17.6784" y2="14.5796" width="0" layer="19" extent="1-1"/>
+<wire x1="11.3884" y1="19.035" x2="13.8884" y2="19.035" width="0" layer="19" extent="1-1"/>
+<wire x1="9.6116" y1="20.447" x2="11.3884" y2="19.035" width="0" layer="19" extent="1-1"/>
+<wire x1="9.4384" y1="16.585" x2="11.3884" y2="19.035" width="0" layer="19" extent="1-1"/>
+<wire x1="9.4384" y1="16.085" x2="9.4384" y2="16.585" width="0" layer="19" extent="1-1"/>
+<wire x1="9.4384" y1="14.085" x2="9.4384" y2="16.085" width="0" layer="19" extent="1-1"/>
+<wire x1="6.5128" y1="14.8082" x2="9.4384" y2="14.085" width="0" layer="19" extent="1-1"/>
 <wire x1="5.908" y1="16.299" x2="6.5128" y2="14.8082" width="0" layer="19" extent="1-1"/>
-<wire x1="18.7706" y1="1.2844" x2="20.3962" y2="1.6614" width="0" layer="19" extent="1-1"/>
-<wire x1="9.4384" y1="16.085" x2="9.4384" y2="14.085" width="0" layer="19" extent="1-1"/>
+<wire x1="4.9328" y1="12.0604" x2="6.5128" y2="14.8082" width="0" layer="19" extent="1-1"/>
+<wire x1="3.9982" y1="18.9484" x2="5.908" y2="16.299" width="0" layer="19" extent="1-1"/>
+<wire x1="5.8342" y1="8.763" x2="4.9328" y2="12.0604" width="0" layer="19" extent="1-1"/>
+<wire x1="19.304" y1="21.7274" x2="13.8884" y2="19.035" width="0" layer="19" extent="1-1"/>
+<wire x1="20.701" y1="24.2466" x2="19.304" y2="21.7274" width="0" layer="19" extent="1-1"/>
+<wire x1="22.1742" y1="23.1394" x2="20.701" y2="24.2466" width="0" layer="19" extent="1-1"/>
+<wire x1="17.7283" y1="24.9059" x2="20.701" y2="24.2466" width="0" layer="19" extent="1-1"/>
+<wire x1="15.8138" y1="24.9174" x2="17.7283" y2="24.9059" width="0" layer="19" extent="1-1"/>
 </signal>
 <signal name="VSS">
@@
 <contactref element="R5" pad="2"/>
 <contactref element="IC1" pad="2"/>
+<contactref element="U3" pad="6"/>
 <wire x1="46.9392" y1="10.9832" x2="46.8884" y2="14.3868" width="0" layer="19" extent="1-1"/>
 <wire x1="42.4496" y1="8.785" x2="46.9392" y2="10.9832" width="0" layer="19" extent="1-16"/>
+<wire x1="42.4496" y1="6.685" x2="42.4496" y2="8.785" width="0" layer="19" extent="16-16"/>
 <wire x1="24.7038" y1="10.1277" x2="42.4496" y2="8.785" width="0" layer="19" extent="1-16"/>
 <wire x1="20.8384" y1="10.085" x2="24.7038" y2="10.1277" width="0" layer="19" extent="1-1"/>

Commit message: rework to STM32 (WIP)
Parts:
- removed C18: 1uF, SparkFun-Passives:0402-CAP
- removed C19, C21: 0.1uF, SparkFun-Passives:0402-CAP
- removed C20: 2.2uF, SparkFun-Passives:0805
- removed R2: 100k, SparkFun-Passives:0402-RES
- removed R3, R4, R5: 10k, SparkFun-Passives:0402-RES
- removed U$1: LM4F120H5QR, stellaris:LQFP64
- removed X3: SSW-103-02-S-D, con-samtec:SSW-103-02-S-D
- C1, C10, C11, C2, C3, C4, C5: device SparkFun-Passives:0402-CAP -> SparkFun-Passives:0603-CAP
- C12, C14: value 0.1uF -> 100nF; device SparkFun-Passives:0402-CAP -> SparkFun-Passives:0603-CAP
- C13, C15, C16: value 0.01uF -> 100nF; device SparkFun-Passives:0402-CAP -> SparkFun-Passives:0603-CAP
- C17: value 1uF -> 2.2uF; device SparkFun-Passives:0402-CAP -> SparkFun-Passives:0603-CAP
- C6, C9: value 0.1uF -> 2.2uF; device SparkFun-Passives:0402-CAP -> SparkFun-Passives:0603-CAP
- C7, C8: value 10pF -> 22pF; device SparkFun-Passives:0402-CAP -> SparkFun-Passives:0603-CAP
- R1: device SparkFun-Passives:0402-RES -> SparkFun-Passives:0603-RES
- U1: value ATSHA204-TSU -> STM32F205RET6; device SparkFun-DigitalIC:SOT23-3 -> stm32:TQFP64
- moved C16 38.2 mm to (18.7, 39.6), turned to 270 degrees
- moved C14 38.0 mm to (15.5, 40.2)
- moved C15 37.9 mm to (12.8, 40.1)
- moved C12 37.6 mm to (10.1, 40.0)
- moved C6 35.3 mm to (6.71, 39.8)
- moved C13 28.3 mm to (22.0, 38.4)
- moved C9 19.3 mm to (6.10, 36.2), turned to 0 degrees
- moved C17 15.6 mm to (26.7, 38.1)
- moved C11 13.1 mm to (6.73, 27.9), turned to 90 degrees
- moved IC1 11.6 mm to (3.81, 28.6)
- moved C10 10.2 mm to (0.76, 28.4), turned to 90 degrees
- moved C7 10.2 mm to (11.0, 30.6), turned to 270 degrees
- moved U1 8.82 mm to (14.4, 13.4), turned to 45 degrees
- moved Q2 8.34 mm to (15.6, 30.5)
- moved C8 7.74 mm to (21.1, 29.9)
Connections:
- removed net N$15: S1.1, U$1.28
- removed net N$17: R3.1, U$1.52, X3.5
- removed net N$19: U$1.50, X3.4
- removed net N$20: U$1.49, X3.1
- removed net N$21: C9.2, R5.1, U$1.38, X3.2
- removed net N$23: C18.1, C19.1, C20.1, C21.1, U$1.25, U$1.56
- removed net SDA: R2.1, U$1.48, U1.1
- removed net USB_D_N: U$1.43, U2.D-
- removed net USB_D_P: U$1.44, U2.D+
- new net N$3: U1.26, U3.15
- new net N$7: U1.27, U3.14
- net +3V3: now also C12.2, C13.2, C14.2, C15.2, C16.2, C17.2, U1.1, U1.13, U1.19, U1.32, U1.48, U1.64; no longer C12.1, C13.1, C14.1, C15.1, C16.1, C17.1, C6.1, R2.2, R3.2, R4.2, R5.2, U$1.11, U$1.2, U$1.26, U$1.37, U$1.42, U$1.54, U1.2
- net GND: now also C12.1, C13.1, C14.1, C15.1, C16.1, C17.1, C9.2, U1.12, U1.18, U1.60, U1.63; no longer C12.2, C13.2, C14.2, C15.2, C16.2, C17.2, C18.2, C19.2, C20.2, C21.2, C9.1, U$1.12, U$1.27, U$1.3, U$1.32, U$1.34, U$1.35, U$1.39, U$1.55, U1.3, X3.6
- net N$1: now also U1.23; no longer U$1.22
- net N$14: now also U1.45, U2.D+; no longer S2.1, U$1.29
- net N$16: now also U1.20, U3.13; no longer R4.1, U$1.51, X3.3
- net N$2: now also U1.44, U2.D-; no longer U$1.9, U3.13
- net N$4: now also C6.1, U1.31; no longer U$1.7, U3.15
- net N$5: now also U1.21; no longer U$1.19
- net N$8: now also C9.1, U1.47; no longer U$1.8, U3.14
- net XTAL1: now also U1.6; no longer U$1.40
- net XTAL2: now also U1.5; no longer U$1.41
Routing:
- net USB_D_N: track 5.30 -> 0.00 mm
- net USB_D_P: track 5.24 -> 0.00 mm
Other:
- outline, holes or cut-outs redrawn
