File: trezor.brd (EAGLE design)
At the start: 50 x 26.7 mm, 25 parts, among them IC1 MCP1703CB, Q2 16MHz, U1 STM32F205RET6, U2 USB, U3 DISPLAY

Commit message: trezor WIP
Parts:
- added C18: 0.1uF, SparkFun-Passives:0603-CAP
- added U$1: PROGRAMMER, fabhack:PROGRAMMER
- C7: value 22pF -> 2.2uF
- C9: value 2.2uF -> 22pF
- U2: device SparkFun-Connectors:USB-AB-MICRO-SMD -> fabhack:MOLEX_47346-0001
- moved C9 38.7 mm to (23.2, 1.42)
- moved C15 31.6 mm to (24.2, 10.6), turned to 0 degrees
- moved C12 30.8 mm to (25.6, 13.4)
- moved C13 30.1 mm to (6.91, 12.4), turned to 270 degrees
- moved Q2 27.7 mm to (17.7, 2.84), turned to 180 degrees
- moved C8 27.5 mm to (13.0, 3.66), turned to 90 degrees
- moved C17 25.0 mm to (23.6, 13.4), turned to 270 degrees
- moved C11 21.7 mm to (10.7, 6.50), turned to 270 degrees
- moved C6 21.3 mm to (17.9, 21.7), turned to 180 degrees
- moved IC1 20.1 mm to (7.11, 8.74), turned to 90 degrees
- moved C14 18.5 mm to (14.4, 21.7), turned to 0 degrees
- moved C16 16.7 mm to (13.6, 23.8), turned to 0 degrees
- moved C7 12.1 mm to (8.79, 18.7), turned to 0 degrees
- moved C10 11.0 mm to (5.08, 18.3), turned to 0 degrees
- moved U2 2.34 mm to (4.42, 13.4), turned to 270 degrees
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Connections:
- new net N$15: U$1.7, U1.46
- new net N$17: U$1.6, U1.49
- new net N$18: U$1.5, U1.50
- new net N$19: S1.1, U1.25
- new net N$20: S2.1, U1.10
- new net USB_D_N: U1.44, U2.2
- new net USB_D_P: U1.45, U2.3
- net +3V3: now also U$1.2
- net +5V: now also U2.1; no longer U2.VBUS
- net GND: now also C18.2, U$1.3, U2.5; no longer U2.GND
- net N$14: now also U$1.4, U1.55; no longer U1.45, U2.D+
- net N$2: now also C18.1, U$1.1, U1.7; no longer U1.44, U2.D-
- net N$8: now also C7.1; no longer C9.1
- net XTAL1: now also C9.1; no longer C7.1
Routing:
- net USB_D_N: track 0.00 -> 6.86 mm
- net USB_D_P: track 0.00 -> 6.59 mm
Other:
- outline, holes or cut-outs redrawn
