File: trezor.brd (EAGLE design)
At the start: 50 x 26.7 mm, 27 parts, among them IC1 MCP1703CB, Q2 16MHz, U1 STM32F205RET6, U2 USB, U3 DISPLAY

Commit message: wip
Routing:
- net N$8: track 12.6 -> 6.93 mm
- net +3V3: track 118.1 -> 119.4 mm
- net XTAL1: track 9.62 -> 8.65 mm

Commit message: wip
Routing:
- net GND: track 0.00 -> 8.93 mm, vias 0 -> 21
