File: trezor.brd (EAGLE design)
At the start: 50 x 26.7 mm, 27 parts, among them IC1 MCP1703CB, Q2 16MHz, U1 STM32F205RET6, U2 USB, U3 DISPLAY

Commit message: wip
Routing:
- net GND: vias 21 -> 22
Other:
- board text removed: "bitcointrezor.com"
Changed lines of the file:
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@@
 <wire x1="5.334" y1="19.9136" x2="5.9182" y2="19.8882" width="0.0254" layer="20"/>
 <wire x1="5.9182" y1="19.8882" x2="6.477" y2="20.0914" width="0.0254" layer="20"/>
-<text x="36.1696" y="13.5636" size="1.6764" layer="122" font="vector" ratio="12" rot="MR270" align="center">bitcointrezor.com</text>
 </plain>
 <attributes>
@@
 <via x="40.0304" y="10.16" extent="1-16" drill="0.4064"/>
 <via x="45.5168" y="24.9936" extent="1-16" drill="0.4064"/>
-<via x="40.4368" y="23.1648" extent="1-16" drill="0.4064"/>
+<via x="42.4688" y="24.7904" extent="1-16" drill="0.4064"/>
 <via x="45.5168" y="16.6624" extent="1-16" drill="0.4064"/>
 <via x="45.72" y="12.192" extent="1-16" drill="0.4064"/>
 <via x="12.192" y="22.1488" extent="1-16" drill="0.4064"/>
-<via x="22.9616" y="23.7744" extent="1-16" drill="0.4064"/>
+<via x="23.1648" y="23.5712" extent="1-16" drill="0.4064"/>
 <via x="16.8656" y="23.368" extent="1-16" drill="0.4064"/>
 <via x="9.5504" y="20.1168" extent="1-16" drill="0.4064"/>
@@
 <wire x1="21.0312" y1="10.0584" x2="21.844" y2="10.0584" width="0.2032" layer="1"/>
 <wire x1="21.844" y1="10.0584" x2="22.1488" y2="10.3632" width="0.2032" layer="1"/>
-<via x="32.3088" y="25.1968" extent="1-16" drill="0.4064"/>
-<via x="32.3088" y="1.6256" extent="1-16" drill="0.4064"/>
+<via x="32.3088" y="24.7904" extent="1-16" drill="0.4064"/>
+<via x="32.3088" y="2.032" extent="1-16" drill="0.4064"/>
 <via x="25.4" y="1.4224" extent="1-16" drill="0.4064"/>
 <via x="21.7424" y="5.8928" extent="1-16" drill="0.4064"/>
 <via x="3.6576" y="8.9408" extent="1-16" drill="0.4064"/>
+<via x="42.4688" y="2.032" extent="1-16" drill="0.4064"/>
 </signal>
 <signal name="VSS">

Commit message: move capacitors to the edge
Parts:
- moved C1 0.20 mm to (47.3, 2.64)
- moved C2 0.20 mm to (47.3, 8.13)
- moved C3 0.20 mm to (47.3, 15.0)
- moved C4 0.20 mm to (47.3, 11.6)
- moved C5 0.20 mm to (47.3, 24.2)
- moved R1 0.20 mm to (47.3, 18.3)
Changed lines of the file:
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@@
 </element>
 <element name="U3" library="microbuilder" package="UG-2864HSWEG01_0.96IN_WRAPAROUND" value="DISPLAY" x="41.2496" y="13.3604" rot="R90"/>
-<element name="C1" library="SparkFun-Passives" package="0603-CAP" value="1uF" x="47.1424" y="2.6416" rot="R90"/>
-<element name="C2" library="SparkFun-Passives" package="0603-CAP" value="1uF" x="47.1424" y="8.128" rot="R90"/>
-<element name="C3" library="SparkFun-Passives" package="0603-CAP" value="0.1uF" x="47.1424" y="15.0368" rot="R90"/>
-<element name="C4" library="SparkFun-Passives" package="0603-CAP" value="1uF" x="47.1424" y="11.5824" rot="R90"/>
-<element name="C5" library="SparkFun-Passives" package="0603-CAP" value="2.2uF" x="47.1424" y="24.1808" rot="R90"/>
-<element name="R1" library="SparkFun-Passives" package="0603-RES" value="390k" x="47.1424" y="18.288" rot="R270"/>
+<element name="C1" library="SparkFun-Passives" package="0603-CAP" value="1uF" x="47.3456" y="2.6416" rot="R90"/>
+<element name="C2" library="SparkFun-Passives" package="0603-CAP" value="1uF" x="47.3456" y="8.128" rot="R90"/>
+<element name="C3" library="SparkFun-Passives" package="0603-CAP" value="0.1uF" x="47.3456" y="15.0368" rot="R90"/>
+<element name="C4" library="SparkFun-Passives" package="0603-CAP" value="1uF" x="47.3456" y="11.5824" rot="R90"/>
+<element name="C5" library="SparkFun-Passives" package="0603-CAP" value="2.2uF" x="47.3456" y="24.1808" rot="R90"/>
+<element name="R1" library="SparkFun-Passives" package="0603-RES" value="390k" x="47.3456" y="18.288" rot="R270"/>
 <element name="S1" library="SparkFun-Electromechanical" package="TACTILE_SWITCH_SMD" value="SWITCH-MOMENTARY-2SMD" x="23.876" y="20.6248" rot="R270"/>
 <element name="S2" library="SparkFun-Electromechanical" package="TACTILE_SWITCH_SMD" value="SWITCH-MOMENTARY-2SMD" x="23.876" y="6.096" rot="R270"/>
@@
 <wire x1="15.2772" y1="21.7424" x2="15.2772" y2="22.9616" width="0.2032" layer="1"/>
 <wire x1="15.2772" y1="22.9616" x2="14.4644" y2="23.7744" width="0.2032" layer="1"/>
-<wire x1="47.1424" y1="10.7324" x2="45.8551" y2="10.7324" width="0.2032" layer="1"/>
+<wire x1="47.3456" y1="10.7324" x2="45.8551" y2="10.7324" width="0.2032" layer="1"/>
 <wire x1="24.8231" y1="26.0042" x2="28.1899" y2="26.0042" width="0.2032" layer="1"/>
-<wire x1="47.1424" y1="14.1868" x2="45.886" y2="14.1868" width="0.2032" layer="1"/>
+<wire x1="47.3456" y1="14.1868" x2="45.886" y2="14.1868" width="0.2032" layer="1"/>
 <wire x1="44.6584" y1="9.5357" x2="44.6584" y2="12.9592" width="0.2032" layer="1"/>
 <wire x1="44.6584" y1="12.9592" x2="45.886" y2="14.1868" width="0.2032" layer="1"/>
@@
 <contactref element="C1" pad="1"/>
 <wire x1="42.4496" y1="3.9104" x2="43.8037" y2="3.9104" width="0.2032" layer="16"/>
-<wire x1="47.1424" y1="1.7916" x2="46.3883" y2="1.7916" width="0.2032" layer="1"/>
+<wire x1="47.3456" y1="1.7916" x2="46.3883" y2="1.7916" width="0.2032" layer="1"/>
 <wire x1="44.8347" y1="3.3656" x2="46.3883" y2="1.812" width="0.2032" layer="1"/>
 <wire x1="46.3883" y1="1.812" x2="46.3883" y2="1.7916" width="0.2032" layer="1"/>
@@
 <contactref element="U3" pad="4"/>
 <contactref element="C2" pad="1"/>
-<wire x1="47.1424" y1="7.278" x2="46.3883" y2="7.278" width="0.2032" layer="1"/>
+<wire x1="47.3456" y1="7.278" x2="46.3883" y2="7.278" width="0.2032" layer="1"/>
 <wire x1="45.1528" y1="5.7014" x2="46.3883" y2="6.9369" width="0.2032" layer="1"/>
 <wire x1="46.3883" y1="6.9369" x2="46.3883" y2="7.278" width="0.2032" layer="1"/>
@@
 <contactref element="U3" pad="3"/>
 <contactref element="C1" pad="2"/>
-<wire x1="47.1424" y1="3.4916" x2="46.3883" y2="3.4916" width="0.2032" layer="1"/>
+<wire x1="47.3456" y1="3.4916" x2="46.3883" y2="3.4916" width="0.2032" layer="1"/>
 <wire x1="44.3512" y1="4.6104" x2="45.2695" y2="4.6104" width="0.2032" layer="1"/>
 <wire x1="45.2695" y1="4.6104" x2="46.3883" y2="3.4916" width="0.2032" layer="1"/>
@@
 <contactref element="C2" pad="2"/>
 <wire x1="42.4496" y1="6.0104" x2="43.8037" y2="6.0104" width="0.2032" layer="16"/>
-<wire x1="47.1424" y1="8.978" x2="46.3883" y2="8.978" width="0.2032" layer="1"/>
+<wire x1="47.3456" y1="8.978" x2="46.3883" y2="8.978" width="0.2032" layer="1"/>
 <wire x1="45.0324" y1="7.618" x2="45.6379" y2="8.2276" width="0.2032" layer="1"/>
 <wire x1="45.6379" y1="8.2276" x2="46.3883" y2="8.978" width="0.2032" layer="1"/>
@@
 <wire x1="42.4496" y1="21.4104" x2="45.0659" y2="21.4104" width="0.2032" layer="16"/>
 <wire x1="45.0659" y1="21.4104" x2="45.1344" y2="21.4789" width="0.2032" layer="16"/>
-<wire x1="47.1424" y1="23.3308" x2="46.9863" y2="23.3308" width="0.2032" layer="1"/>
+<wire x1="47.3456" y1="23.3308" x2="46.9863" y2="23.3308" width="0.2032" layer="1"/>
 <wire x1="46.9863" y1="23.3308" x2="45.1344" y2="21.4789" width="0.2032" layer="1"/>
 </signal>
@@
 <contactref element="U3" pad="26"/>
 <contactref element="R1" pad="1"/>
-<wire x1="47.1424" y1="19.138" x2="46.3883" y2="19.138" width="0.2032" layer="1"/>
+<wire x1="47.3456" y1="19.138" x2="46.3883" y2="19.138" width="0.2032" layer="1"/>
 <wire x1="45.6209" y1="19.7087" x2="45.8176" y2="19.7087" width="0.2032" layer="1"/>
 <wire x1="45.8176" y1="19.7087" x2="46.3883" y2="19.138" width="0.2032" layer="1"/>

Commit message: add items to trezor bom
Parts:
- C12, C13, C14, C15, C16: value 100nF -> 0.1uF
Changed lines of the file:
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@@
 <element name="C10" library="SparkFun-Passives" package="0603-CAP" value="1uF" x="5.08" y="18.288"/>
 <element name="C11" library="SparkFun-Passives" package="0603-CAP" value="1uF" x="10.668" y="6.5024" rot="R270"/>
-<element name="C13" library="SparkFun-Passives" package="0603-CAP" value="100nF" x="6.9088" y="12.3952" rot="R270"/>
-<element name="C12" library="SparkFun-Passives" package="0603-CAP" value="100nF" x="25.6032" y="13.3604" rot="R270"/>
-<element name="C15" library="SparkFun-Passives" package="0603-CAP" value="100nF" x="24.1808" y="10.5664"/>
-<element name="C16" library="SparkFun-Passives" package="0603-CAP" value="100nF" x="13.6144" y="23.7744"/>
-<element name="C14" library="SparkFun-Passives" package="0603-CAP" value="100nF" x="14.4272" y="21.7424"/>
+<element name="C13" library="SparkFun-Passives" package="0603-CAP" value="0.1uF" x="6.9088" y="12.3952" rot="R270"/>
+<element name="C12" library="SparkFun-Passives" package="0603-CAP" value="0.1uF" x="25.6032" y="13.3604" rot="R270"/>
+<element name="C15" library="SparkFun-Passives" package="0603-CAP" value="0.1uF" x="24.1808" y="10.5664"/>
+<element name="C16" library="SparkFun-Passives" package="0603-CAP" value="0.1uF" x="13.6144" y="23.7744"/>
+<element name="C14" library="SparkFun-Passives" package="0603-CAP" value="0.1uF" x="14.4272" y="21.7424"/>
 <element name="C17" library="SparkFun-Passives" package="0603-CAP" value="2.2uF" x="23.5712" y="13.3604" rot="R270"/>
 <element name="IC1" library="linear" package="SOT23" value="MCP1703CB" x="7.112" y="8.7376" rot="R90"/>

Commit message: connect vbus to mcu as well
Connections:
- net +5V: now also U1.42
Routing:
- net +5V: track 12.0 -> 18.5 mm, vias 2 -> 3
Changed lines of the file:
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@@
 <contactref element="IC1" pad="3"/>
 <contactref element="U2" pad="1"/>
-<via x="5.7912" y="15.748" extent="1-16" drill="0.4064" diameter="0.8128"/>
-<wire x1="5.7912" y1="15.748" x2="5.7912" y2="9.9568" width="0.2032" layer="16"/>
+<via x="5.7912" y="16.5608" extent="1-16" drill="0.4064" diameter="0.8128"/>
+<wire x1="5.7912" y1="16.5608" x2="5.7912" y2="9.9568" width="0.2032" layer="16"/>
 <via x="5.7912" y="9.9568" extent="1-16" drill="0.4064" diameter="0.8128"/>
 <wire x1="5.8928" y1="8.8568" x2="6.012" y2="8.7376" width="0.2032" layer="1"/>
 <wire x1="4.4196" y1="14.6604" x2="5.2116" y2="14.6604" width="0.2032" layer="1"/>
 <wire x1="5.2116" y1="14.6604" x2="5.7912" y2="15.24" width="0.2032" layer="1"/>
-<wire x1="5.7912" y1="15.24" x2="5.7912" y2="15.748" width="0.2032" layer="1"/>
+<wire x1="5.7912" y1="15.24" x2="5.7912" y2="16.5608" width="0.2032" layer="1"/>
 <wire x1="5.7912" y1="9.9568" x2="5.7912" y2="8.9584" width="0.2032" layer="1"/>
 <wire x1="5.7912" y1="8.9584" x2="6.012" y2="8.7376" width="0.2032" layer="1"/>
-<wire x1="5.7912" y1="15.748" x2="5.7912" y2="18.1492" width="0.2032" layer="1"/>
+<wire x1="5.7912" y1="16.5608" x2="5.7912" y2="18.1492" width="0.2032" layer="1"/>
 <wire x1="5.7912" y1="18.1492" x2="5.93" y2="18.288" width="0.2032" layer="1"/>
+<contactref element="U1" pad="42"/>
+<via x="9.2456" y="17.3736" extent="1-16" drill="0.4064" diameter="0.8128"/>
+<wire x1="10.679159375" y1="16.860578125" x2="10.1661375" y2="17.3736" width="0.2032" layer="1"/>
+<wire x1="10.1661375" y1="17.3736" x2="9.2456" y2="17.3736" width="0.2032" layer="1"/>
+<wire x1="9.2456" y1="17.3736" x2="8.9408" y2="17.6784" width="0.2032" layer="16"/>
+<wire x1="8.9408" y1="17.6784" x2="6.9088" y2="17.6784" width="0.2032" layer="16"/>
+<wire x1="6.9088" y1="17.6784" x2="5.7912" y2="16.5608" width="0.2032" layer="16"/>
 </signal>
 <signal name="XTAL1">

Commit message: rework swd programmer
Parts:
- removed U$1: PROGRAMMER, fabhack:PROGRAMMER
- added U$2: SWD, fabhack:SWD
Connections:
- removed net N$18: U$1.5, U1.50
- removed net VSS: U3.8
- net +3V3: now also U$2.6; no longer U$1.2
- net GND: now also U$2.2, U3.8; no longer U$1.3
- net N$14: now also U$2.3; no longer U$1.4
- net N$15: now also U$2.5; no longer U$1.7
- net N$17: now also U$2.4; no longer U$1.6
- net N$2: now also U$2.1; no longer U$1.1
Routing:
- net +3V3: track 119.4 -> 86.5 mm, vias 1 -> 2
- net N$18: track 18.3 -> 0.00 mm
- net N$15: track 13.8 -> 16.4 mm
- net N$17: track 17.0 -> 18.2 mm
- net N$14: track 19.5 -> 20.1 mm

Commit message: fix unconnected pin
Routing:
- net +3V3: track 86.5 -> 88.7 mm
- net N$17: track 18.2 -> 19.3 mm
- net N$15: track 16.4 -> 16.1 mm, vias 0 -> 1
Changed lines of the file:
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@@
 <wire x1="8.212" y1="10.0647" x2="9.9139" y2="8.3628" width="0.2032" layer="1"/>
 <wire x1="9.9139" y1="8.3628" x2="9.9139" y2="5.6524" width="0.2032" layer="1"/>
-<wire x1="16.6189" y1="20.0426" x2="16.0149" y2="19.4386" width="0.2032" layer="1"/>
+<wire x1="16.6189" y1="20.0426" x2="16.61885625" y2="20.04255625" width="0.2032" layer="1"/>
+<wire x1="16.61885625" y1="20.04255625" x2="16.0149" y2="19.4386" width="0.2032" layer="1"/>
 <wire x1="21.2151" y1="15.4464" x2="20.6111" y2="14.8424" width="0.2032" layer="1"/>
 <wire x1="25.0308" y1="12.5104" x2="25.6032" y2="12.5104" width="0.2032" layer="1"/>
@@
 <wire x1="40.8432" y1="8.5344" x2="28.448" y2="8.5344" width="0.2032" layer="16"/>
 <wire x1="28.448" y1="8.5344" x2="26.416" y2="10.5664" width="0.2032" layer="16"/>
+<wire x1="16.61885625" y1="20.04255625" x2="15.2772" y2="21.3842125" width="0.2032" layer="1"/>
+<wire x1="15.2772" y1="21.3842125" x2="15.2772" y2="21.7424" width="0.2032" layer="1"/>
 <wire x1="21.2151" y1="15.4464" x2="21.21505" y2="15.4463625" width="0" layer="19" extent="1-1"/>
-<wire x1="16.61885625" y1="20.04255625" x2="16.6189" y2="20.0426" width="0" layer="19" extent="1-1"/>
 <wire x1="20.861496875" y1="10.92088125" x2="20.8615" y2="10.9209" width="0" layer="19" extent="1-1"/>
 <wire x1="16.61885625" y1="6.678240625" x2="16.6189" y2="6.6782" width="0" layer="19" extent="1-1"/>
 <wire x1="8.557840625" y1="14.73925625" x2="8.5578" y2="14.7393" width="0" layer="19" extent="1-1"/>
 <wire x1="13.861140625" y1="6.678240625" x2="13.8611" y2="6.6782" width="0" layer="19" extent="1-1"/>
-<wire x1="15.2772" y1="21.7424" x2="16.6189" y2="20.0426" width="0" layer="19" extent="1-1"/>
 </signal>
 <signal name="N$1">
@@
 <wire x1="22.4282" y1="25.0952" x2="20.1168" y2="22.7838" width="0.2032" layer="16"/>
 <wire x1="20.1168" y1="22.7838" x2="20.1168" y2="20.5232" width="0.2032" layer="16"/>
-<wire x1="20.1168" y1="20.5232" x2="13.8176" y2="14.224" width="0.2032" layer="16"/>
-<wire x1="13.8176" y1="14.224" x2="13.8176" y2="13.6144" width="0.2032" layer="16"/>
 <wire x1="10.679159375" y1="9.86021875" x2="13.8176" y2="12.998659375" width="0.2032" layer="1"/>
-<wire x1="13.8176" y1="12.998659375" x2="13.8176" y2="13.6144" width="0.2032" layer="1"/>
-<via x="13.8176" y="13.6144" extent="1-16" drill="0.4064"/>
+<via x="14.4272" y="13.6144" extent="1-16" drill="0.4064"/>
+<wire x1="14.4272" y1="13.6144" x2="14.4272" y2="14.8336" width="0.2032" layer="16"/>
+<wire x1="14.4272" y1="14.8336" x2="20.1168" y2="20.5232" width="0.2032" layer="16"/>
+<wire x1="14.4272" y1="13.6144" x2="14.4272" y2="13.608259375" width="0.2032" layer="1"/>
+<wire x1="14.4272" y1="13.608259375" x2="13.8176" y2="12.998659375" width="0.2032" layer="1"/>
 </signal>
 <signal name="N$15">
 <contactref element="U1" pad="46"/>
 <contactref element="U$2" pad="5"/>
-<wire x1="9.264946875" y1="15.4463625" x2="9.877709375" y2="14.8336" width="0.2032" layer="1"/>
-<wire x1="9.877709375" y1="14.8336" x2="10.3632" y2="14.8336" width="0.2032" layer="1"/>
-<wire x1="10.3632" y1="14.8336" x2="16.1544" y2="20.6248" width="0.2032" layer="1"/>
-<wire x1="16.1544" y1="20.6248" x2="16.1544" y2="21.6408" width="0.2032" layer="1"/>
-<wire x1="19.2532" y1="25.0952" x2="18.3388" y2="24.1808" width="0.2032" layer="1"/>
-<wire x1="18.3388" y1="24.1808" x2="17.0688" y2="24.1808" width="0.2032" layer="1"/>
-<wire x1="17.0688" y1="24.1808" x2="16.4592" y2="24.1808" width="0.2032" layer="1"/>
-<wire x1="16.4592" y1="24.1808" x2="16.1544" y2="23.876" width="0.2032" layer="1"/>
-<wire x1="16.1544" y1="23.876" x2="16.1544" y2="21.6408" width="0.2032" layer="1"/>
+<wire x1="9.264946875" y1="15.4463625" x2="10.080909375" y2="14.6304" width="0.2032" layer="1"/>
+<wire x1="10.080909375" y1="14.6304" x2="11.176" y2="14.6304" width="0.2032" layer="1"/>
+<via x="11.176" y="14.6304" extent="1-16" drill="0.4064"/>
+<wire x1="11.176" y1="14.6304" x2="18.288" y2="21.7424" width="0.2032" layer="16"/>
+<wire x1="18.288" y1="21.7424" x2="18.288" y2="22.9616" width="0.2032" layer="16"/>
+<wire x1="18.288" y1="22.9616" x2="18.288" y2="24.13" width="0.2032" layer="16"/>
+<wire x1="18.288" y1="24.13" x2="19.2532" y2="25.0952" width="0.2032" layer="16"/>
 </signal>
 <signal name="N$17">
 <contactref element="U1" pad="49"/>
-<wire x1="10.053" y1="13.8368" x2="17.6657" y2="21.4495" width="0.2032" layer="16"/>
-<via x="10.053" y="13.8368" extent="1-16" drill="0.4064" diameter="0.8128"/>
-<wire x1="8.557840625" y1="11.981540625" x2="10.053" y2="13.4767" width="0.2032" layer="1"/>
-<wire x1="10.053" y1="13.4767" x2="10.053" y2="13.8368" width="0.2032" layer="1"/>
 <contactref element="U$2" pad="4"/>
-<wire x1="17.6657" y1="21.4495" x2="20.8407" y2="24.6245" width="0.2032" layer="16"/>
-<wire x1="20.8407" y1="24.6245" x2="20.8407" y2="25.0952" width="0.2032" layer="16"/>
+<via x="13.0048" y="14.6304" extent="1-16" drill="0.4064"/>
+<wire x1="13.0048" y1="14.6304" x2="19.304" y2="20.9296" width="0.2032" layer="16"/>
+<wire x1="19.304" y1="20.9296" x2="19.304" y2="22.9616" width="0.2032" layer="16"/>
+<wire x1="19.304" y1="22.9616" x2="19.304" y2="23.5585" width="0.2032" layer="16"/>
+<wire x1="19.304" y1="23.5585" x2="20.8407" y2="25.0952" width="0.2032" layer="16"/>
+<wire x1="8.557840625" y1="11.981540625" x2="9.5811" y2="13.0048" width="0.2032" layer="1"/>
+<wire x1="9.5811" y1="13.0048" x2="10.3632" y2="13.0048" width="0.2032" layer="1"/>
+<wire x1="10.3632" y1="13.0048" x2="11.3792" y2="13.0048" width="0.2032" layer="1"/>
+<wire x1="11.3792" y1="13.0048" x2="13.0048" y2="14.6304" width="0.2032" layer="1"/>
 </signal>
 <signal name="N$19">

Commit message: change crystal
Parts:
- Q2: value 16MHz -> 8MHz
Changed lines of the file:
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@@
 <element name="S1" library="SparkFun-Electromechanical" package="TACTILE_SWITCH_SMD" value="SWITCH-MOMENTARY-2SMD" x="23.876" y="20.6248" rot="R270"/>
 <element name="S2" library="SparkFun-Electromechanical" package="TACTILE_SWITCH_SMD" value="SWITCH-MOMENTARY-2SMD" x="23.876" y="6.096" rot="R270"/>
-<element name="Q2" library="crystal" package="CTS406" value="16MHz" x="17.6784" y="2.8448" rot="R180"/>
+<element name="Q2" library="crystal" package="CTS406" value="8MHz" x="17.6784" y="2.8448" rot="R180"/>
 <element name="C9" library="SparkFun-Passives" package="0603-CAP" value="22pF" x="23.1648" y="1.4224"/>
 <element name="C8" library="SparkFun-Passives" package="0603-CAP" value="22pF" x="13.0048" y="3.6576" rot="R90"/>
