File: trezor.sch (EAGLE design)
At the start: 39 parts, among them IC1 MCP1703CB, Q2 16MHz, U1 ATSHA204-TSU, U2 USB, U3 DISPLAY, U5 TPD4S012_DRY_6

Commit message: work snapshot
Parts:
- removed U5: TPD4S012_DRY_6, imported:TPD4S012_DRY_6
- C20: device SparkFun-Passives:CAP0402-CAP -> SparkFun-Passives:CAP0805
- C3: value 104 -> 0.1uF
Connections:
- removed net N$3: U2.USBID, U5.ID
- net +5V: no longer U2.VBUS, U5.VBUS
- net GND: no longer U2.GND, U5.GND
- net USB_D_N: no longer U5.D-
- net USB_D_P: no longer U5.D+
Changed lines of the file:
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@@
 <part name="C1" library="SparkFun-Passives" deviceset="CAP" device="0402-CAP" value="1uF"/>
 <part name="C2" library="SparkFun-Passives" deviceset="CAP" device="0402-CAP" value="1uF"/>
-<part name="C3" library="SparkFun-Passives" deviceset="CAP" device="0402-CAP" value="104"/>
+<part name="C3" library="SparkFun-Passives" deviceset="CAP" device="0402-CAP" value="0.1uF"/>
 <part name="C4" library="SparkFun-Passives" deviceset="CAP" device="0402-CAP" value="1uF"/>
 <part name="GND6" library="supply1" deviceset="GND" device=""/>
@@
 <part name="C18" library="SparkFun-Passives" deviceset="CAP" device="0402-CAP" value="1uF"/>
 <part name="C19" library="SparkFun-Passives" deviceset="CAP" device="0402-CAP" value="0.1uF"/>
-<part name="C20" library="SparkFun-Passives" deviceset="CAP" device="0402-CAP" value="2.2uF"/>
+<part name="C20" library="SparkFun-Passives" deviceset="CAP" device="0805" value="2.2uF"/>
 <part name="C21" library="SparkFun-Passives" deviceset="CAP" device="0402-CAP" value="0.1uF"/>
 <part name="GND15" library="supply1" deviceset="GND" device=""/>
@@
 </part>
 <part name="IC1" library="linear" deviceset="MCP1703" device="CB"/>
-<part name="U5" library="imported" deviceset="TPD4S012_DRY_6" device=""/>
-<part name="P+3" library="supply1" deviceset="+5V" device=""/>
-<part name="GND17" library="supply1" deviceset="GND" device=""/>
 <part name="P+1" library="supply1" deviceset="+5V" device=""/>
 <part name="GND1" library="supply1" deviceset="GND" device=""/>
@@
 <instances>
 <instance part="U$1" gate="G$1" x="22.86" y="60.96"/>
-<instance part="U2" gate="G$1" x="86.36" y="-38.1" rot="R180"/>
+<instance part="U2" gate="G$1" x="104.14" y="-30.48" rot="MR270"/>
 <instance part="GND2" gate="1" x="170.18" y="63.5" rot="R180"/>
 <instance part="U3" gate="G$1" x="132.08" y="20.32" rot="MR270"/>
@@
 <instance part="TP4" gate="G$1" x="-33.02" y="27.94"/>
 <instance part="IC1" gate="G$1" x="-30.48" y="10.16"/>
-<instance part="U5" gate="A" x="109.22" y="-38.1"/>
-<instance part="P+3" gate="1" x="170.18" y="-33.02"/>
-<instance part="GND17" gate="1" x="170.18" y="-48.26"/>
-<instance part="P+1" gate="1" x="93.98" y="-25.4"/>
-<instance part="GND1" gate="1" x="93.98" y="-48.26"/>
+<instance part="P+1" gate="1" x="114.3" y="-17.78"/>
+<instance part="GND1" gate="1" x="93.98" y="-27.94"/>
 </instances>
 <busses>
@@
 </segment>
 <segment>
-<pinref part="U5" gate="A" pin="GND"/>
-<pinref part="GND17" gate="1" pin="GND"/>
-<wire x1="165.1" y1="-43.18" x2="170.18" y2="-43.18" width="0.1524" layer="91"/>
-<wire x1="170.18" y1="-43.18" x2="170.18" y2="-45.72" width="0.1524" layer="91"/>
-</segment>
-<segment>
-<pinref part="U2" gate="G$1" pin="GND"/>
 <pinref part="GND1" gate="1" pin="GND"/>
-<wire x1="91.44" y1="-43.18" x2="93.98" y2="-43.18" width="0.1524" layer="91"/>
-<wire x1="93.98" y1="-43.18" x2="93.98" y2="-45.72" width="0.1524" layer="91"/>
+<wire x1="99.06" y1="-25.4" x2="99.06" y2="-20.32" width="0.1524" layer="91"/>
+<wire x1="99.06" y1="-20.32" x2="93.98" y2="-20.32" width="0.1524" layer="91"/>
+<wire x1="93.98" y1="-20.32" x2="93.98" y2="-25.4" width="0.1524" layer="91"/>
 </segment>
 </net>
@@
 </segment>
 <segment>
-<pinref part="U5" gate="A" pin="VBUS"/>
-<pinref part="P+3" gate="1" pin="+5V"/>
-<wire x1="165.1" y1="-38.1" x2="170.18" y2="-38.1" width="0.1524" layer="91"/>
-<wire x1="170.18" y1="-38.1" x2="170.18" y2="-35.56" width="0.1524" layer="91"/>
-</segment>
-<segment>
-<pinref part="U2" gate="G$1" pin="VBUS"/>
 <pinref part="P+1" gate="1" pin="+5V"/>
-<wire x1="91.44" y1="-33.02" x2="93.98" y2="-33.02" width="0.1524" layer="91"/>
-<wire x1="93.98" y1="-33.02" x2="93.98" y2="-27.94" width="0.1524" layer="91"/>
+<wire x1="109.22" y1="-25.4" x2="109.22" y2="-22.86" width="0.1524" layer="91"/>
+<wire x1="109.22" y1="-22.86" x2="114.3" y2="-22.86" width="0.1524" layer="91"/>
+<wire x1="114.3" y1="-22.86" x2="114.3" y2="-20.32" width="0.1524" layer="91"/>
 </segment>
 </net>
@@
 <pinref part="U$1" gate="G$1" pin="PD4"/>
 <wire x1="86.36" y1="30.48" x2="45.72" y2="30.48" width="0.1524" layer="91"/>
+<wire x1="86.36" y1="-7.62" x2="106.68" y2="-7.62" width="0.1524" layer="91"/>
 <pinref part="U2" gate="G$1" pin="D-"/>
-<wire x1="91.44" y1="-35.56" x2="101.6" y2="-35.56" width="0.1524" layer="91"/>
-<wire x1="101.6" y1="-35.56" x2="101.6" y2="-40.64" width="0.1524" layer="91"/>
-<pinref part="U5" gate="A" pin="D-"/>
-<wire x1="101.6" y1="-40.64" x2="106.68" y2="-40.64" width="0.1524" layer="91"/>
-<wire x1="106.68" y1="-40.64" x2="109.22" y2="-40.64" width="0.1524" layer="91"/>
-<wire x1="86.36" y1="-7.62" x2="106.68" y2="-7.62" width="0.1524" layer="91"/>
-<wire x1="106.68" y1="-7.62" x2="106.68" y2="-40.64" width="0.1524" layer="91"/>
-<junction x="106.68" y="-40.64"/>
+<wire x1="106.68" y1="-7.62" x2="106.68" y2="-25.4" width="0.1524" layer="91"/>
 </segment>
 </net>
@@
 <pinref part="U$1" gate="G$1" pin="PD5"/>
 <wire x1="83.82" y1="27.94" x2="45.72" y2="27.94" width="0.1524" layer="91"/>
+<wire x1="83.82" y1="-10.16" x2="104.14" y2="-10.16" width="0.1524" layer="91"/>
 <pinref part="U2" gate="G$1" pin="D+"/>
-<wire x1="91.44" y1="-38.1" x2="101.6" y2="-38.1" width="0.1524" layer="91"/>
-<wire x1="101.6" y1="-38.1" x2="104.14" y2="-38.1" width="0.1524" layer="91"/>
-<pinref part="U5" gate="A" pin="D+"/>
-<wire x1="104.14" y1="-38.1" x2="109.22" y2="-38.1" width="0.1524" layer="91"/>
-<wire x1="83.82" y1="-10.16" x2="104.14" y2="-10.16" width="0.1524" layer="91"/>
-<wire x1="104.14" y1="-10.16" x2="104.14" y2="-38.1" width="0.1524" layer="91"/>
-<junction x="104.14" y="-38.1"/>
-</segment>
-</net>
-<net name="N$3" class="0">
-<segment>
-<pinref part="U2" gate="G$1" pin="USBID"/>
-<pinref part="U5" gate="A" pin="ID"/>
-<wire x1="91.44" y1="-40.64" x2="96.52" y2="-40.64" width="0.1524" layer="91"/>
-<wire x1="96.52" y1="-40.64" x2="96.52" y2="-43.18" width="0.1524" layer="91"/>
-<wire x1="96.52" y1="-43.18" x2="109.22" y2="-43.18" width="0.1524" layer="91"/>
-</segment>
-</net>
+<wire x1="104.14" y1="-25.4" x2="104.14" y2="-10.16" width="0.1524" layer="91"/>
+</segment>
+</net>

Commit message: forgot to connect usb gnd/vcc
Connections:
- net +5V: now also U2.VBUS
- net GND: now also U2.GND
Changed lines of the file:
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@@
 <wire x1="99.06" y1="-20.32" x2="93.98" y2="-20.32" width="0.1524" layer="91"/>
 <wire x1="93.98" y1="-20.32" x2="93.98" y2="-25.4" width="0.1524" layer="91"/>
+<pinref part="U2" gate="G$1" pin="GND"/>
 </segment>
 </net>
@@
 <wire x1="109.22" y1="-22.86" x2="114.3" y2="-22.86" width="0.1524" layer="91"/>
 <wire x1="114.3" y1="-22.86" x2="114.3" y2="-20.32" width="0.1524" layer="91"/>
+<pinref part="U2" gate="G$1" pin="VBUS"/>
 </segment>
 </net>

Commit message: wip
Parts:
- added TP5, TP6: (no value), microbuilder:TESTPOINTROUND0.5MM
- TP1, TP2, TP3, TP4: value PTR1TP10R -> (none); device testpad:PTR1TP10R -> microbuilder:TESTPOINTROUND0.5MM
Connections:
- net GND: now also TP6.P$1
- net N$16: now also TP3.P$1; no longer TP2.TP
- net N$17: now also TP2.P$1; no longer TP1.TP
- net N$19: now also TP4.P$1; no longer TP3.TP
- net N$20: now also TP5.P$1; no longer TP4.TP
- net N$21: now also TP1.P$1
Changed lines of the file:
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@@
 <part name="GND16" library="supply1" deviceset="GND" device=""/>
 <part name="+3V6" library="supply1" deviceset="+3V3" device=""/>
-<part name="TP1" library="testpad" deviceset="PTR1" device="TP10R"/>
-<part name="TP2" library="testpad" deviceset="PTR1" device="TP10R">
-<attribute name="TP_SIGNAL_NAME" value=""/>
-</part>
-<part name="TP3" library="testpad" deviceset="PTR1" device="TP10R">
-<attribute name="TP_SIGNAL_NAME" value=""/>
-</part>
-<part name="TP4" library="testpad" deviceset="PTR1" device="TP10R">
-<attribute name="TP_SIGNAL_NAME" value=""/>
-</part>
 <part name="IC1" library="linear" deviceset="MCP1703" device="CB"/>
 <part name="P+1" library="supply1" deviceset="+5V" device=""/>
 <part name="GND1" library="supply1" deviceset="GND" device=""/>
+<part name="GND17" library="supply1" deviceset="GND" device=""/>
+<part name="TP1" library="microbuilder" deviceset="TESTPOINT" device="ROUND0.5MM"/>
+<part name="TP2" library="microbuilder" deviceset="TESTPOINT" device="ROUND0.5MM"/>
+<part name="TP3" library="microbuilder" deviceset="TESTPOINT" device="ROUND0.5MM"/>
+<part name="TP4" library="microbuilder" deviceset="TESTPOINT" device="ROUND0.5MM"/>
+<part name="TP5" library="microbuilder" deviceset="TESTPOINT" device="ROUND0.5MM"/>
+<part name="TP6" library="microbuilder" deviceset="TESTPOINT" device="ROUND0.5MM"/>
 </parts>
 <sheets>
@@
 <instance part="GND16" gate="1" x="55.88" y="91.44"/>
 <instance part="+3V6" gate="G$1" x="55.88" y="114.3"/>
-<instance part="TP1" gate="G$1" x="-40.64" y="35.56"/>
-<instance part="TP2" gate="G$1" x="-38.1" y="33.02"/>
-<instance part="TP3" gate="G$1" x="-35.56" y="30.48"/>
-<instance part="TP4" gate="G$1" x="-33.02" y="27.94"/>
 <instance part="IC1" gate="G$1" x="-30.48" y="10.16"/>
 <instance part="P+1" gate="1" x="114.3" y="-17.78"/>
 <instance part="GND1" gate="1" x="93.98" y="-27.94"/>
+<instance part="GND17" gate="1" x="-43.18" y="25.4"/>
+<instance part="TP1" gate="G$1" x="-45.72" y="43.18" rot="R90"/>
+<instance part="TP2" gate="G$1" x="-48.26" y="40.64" rot="R90"/>
+<instance part="TP3" gate="G$1" x="-45.72" y="38.1" rot="R90"/>
+<instance part="TP4" gate="G$1" x="-48.26" y="35.56" rot="R90"/>
+<instance part="TP5" gate="G$1" x="-45.72" y="33.02" rot="R90"/>
+<instance part="TP6" gate="G$1" x="-48.26" y="30.48" rot="R90"/>
 </instances>
 <busses>
@@
 <pinref part="U2" gate="G$1" pin="GND"/>
 </segment>
+<segment>
+<pinref part="GND17" gate="1" pin="GND"/>
+<wire x1="-43.18" y1="27.94" x2="-43.18" y2="30.48" width="0.1524" layer="91"/>
+<wire x1="-43.18" y1="30.48" x2="-48.26" y2="30.48" width="0.1524" layer="91"/>
+<pinref part="TP6" gate="G$1" pin="P$1"/>
+</segment>
 </net>
 <net name="N$8" class="0">
@@
 <pinref part="R3" gate="G$1" pin="1"/>
 <wire x1="-22.86" y1="43.18" x2="-22.86" y2="40.64" width="0.1524" layer="91"/>
+<wire x1="-22.86" y1="40.64" x2="-33.02" y2="40.64" width="0.1524" layer="91"/>
 <junction x="-22.86" y="40.64"/>
-<pinref part="TP1" gate="G$1" pin="TP"/>
-<wire x1="-22.86" y1="40.64" x2="-40.64" y2="40.64" width="0.1524" layer="91"/>
-<wire x1="-40.64" y1="40.64" x2="-40.64" y2="38.1" width="0.1524" layer="91"/>
+<wire x1="-33.02" y1="40.64" x2="-48.26" y2="40.64" width="0.1524" layer="91"/>
+<pinref part="TP2" gate="G$1" pin="P$1"/>
 </segment>
 </net>
@@
 <pinref part="R4" gate="G$1" pin="1"/>
 <wire x1="-15.24" y1="43.18" x2="-15.24" y2="38.1" width="0.1524" layer="91"/>
+<wire x1="-15.24" y1="38.1" x2="-33.02" y2="38.1" width="0.1524" layer="91"/>
 <junction x="-15.24" y="38.1"/>
-<pinref part="TP2" gate="G$1" pin="TP"/>
-<wire x1="-15.24" y1="38.1" x2="-38.1" y2="38.1" width="0.1524" layer="91"/>
-<wire x1="-38.1" y1="38.1" x2="-38.1" y2="35.56" width="0.1524" layer="91"/>
+<wire x1="-33.02" y1="38.1" x2="-45.72" y2="38.1" width="0.1524" layer="91"/>
+<pinref part="TP3" gate="G$1" pin="P$1"/>
 </segment>
 </net>
@@
 <segment>
 <pinref part="U$1" gate="G$1" pin="PC2/TDI"/>
-<wire x1="-2.54" y1="35.56" x2="-35.56" y2="35.56" width="0.1524" layer="91"/>
-<pinref part="TP3" gate="G$1" pin="TP"/>
-<wire x1="-35.56" y1="35.56" x2="-35.56" y2="33.02" width="0.1524" layer="91"/>
+<wire x1="-2.54" y1="35.56" x2="-30.48" y2="35.56" width="0.1524" layer="91"/>
+<wire x1="-30.48" y1="35.56" x2="-33.02" y2="35.56" width="0.1524" layer="91"/>
+<wire x1="-33.02" y1="35.56" x2="-48.26" y2="35.56" width="0.1524" layer="91"/>
+<pinref part="TP4" gate="G$1" pin="P$1"/>
 </segment>
 </net>
@@
 <segment>
 <pinref part="U$1" gate="G$1" pin="PC3/TDO/SWO"/>
-<wire x1="-2.54" y1="33.02" x2="-33.02" y2="33.02" width="0.1524" layer="91"/>
-<wire x1="-33.02" y1="33.02" x2="-33.02" y2="30.48" width="0.1524" layer="91"/>
-<pinref part="TP4" gate="G$1" pin="TP"/>
+<wire x1="-2.54" y1="33.02" x2="-30.48" y2="33.02" width="0.1524" layer="91"/>
+<wire x1="-30.48" y1="33.02" x2="-35.56" y2="33.02" width="0.1524" layer="91"/>
+<wire x1="-35.56" y1="33.02" x2="-45.72" y2="33.02" width="0.1524" layer="91"/>
+<pinref part="TP5" gate="G$1" pin="P$1"/>
 </segment>
 </net>
@@
 <junction x="55.88" y="101.6"/>
 <junction x="55.88" y="101.6"/>
-</segment>
-</net>
+<wire x1="55.88" y1="101.6" x2="60.96" y2="101.6" width="0.1524" layer="91"/>
+<wire x1="60.96" y1="101.6" x2="60.96" y2="121.92" width="0.1524" layer="91"/>
+<wire x1="60.96" y1="121.92" x2="-43.18" y2="121.92" width="0.1524" layer="91"/>
+<wire x1="-43.18" y1="121.92" x2="-43.18" y2="43.18" width="0.1524" layer="91"/>
+<wire x1="-43.18" y1="43.18" x2="-45.72" y2="43.18" width="0.1524" layer="91"/>
+<pinref part="TP1" gate="G$1" pin="P$1"/>
+</segment>
+</net>

Commit message: wip
Parts:
- removed TP1, TP2, TP3, TP4, TP5, TP6: (no value), microbuilder:TESTPOINTROUND0.5MM
- added X3: SSW-103-02-S-D, con-samtec:SSW-103-02-S-D
Connections:
- net GND: now also X3-6.1; no longer TP6.P$1
- net N$16: now also X3-3.1; no longer TP3.P$1
- net N$17: now also X3-5.1; no longer TP2.P$1
- net N$19: now also X3-4.1; no longer TP4.P$1
- net N$20: now also X3-1.1; no longer TP5.P$1
- net N$21: now also X3-2.1; no longer TP1.P$1
Changed lines of the file:
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@@
 <part name="GND1" library="supply1" deviceset="GND" device=""/>
 <part name="GND17" library="supply1" deviceset="GND" device=""/>
-<part name="TP1" library="microbuilder" deviceset="TESTPOINT" device="ROUND0.5MM"/>
-<part name="TP2" library="microbuilder" deviceset="TESTPOINT" device="ROUND0.5MM"/>
-<part name="TP3" library="microbuilder" deviceset="TESTPOINT" device="ROUND0.5MM"/>
-<part name="TP4" library="microbuilder" deviceset="TESTPOINT" device="ROUND0.5MM"/>
-<part name="TP5" library="microbuilder" deviceset="TESTPOINT" device="ROUND0.5MM"/>
-<part name="TP6" library="microbuilder" deviceset="TESTPOINT" device="ROUND0.5MM"/>
+<part name="X3" library="con-samtec" deviceset="SSW-103-02-S-D" device=""/>
 </parts>
 <sheets>
@@
 <instance part="GND1" gate="1" x="93.98" y="-27.94"/>
 <instance part="GND17" gate="1" x="-43.18" y="25.4"/>
-<instance part="TP1" gate="G$1" x="-45.72" y="43.18" rot="R90"/>
-<instance part="TP2" gate="G$1" x="-48.26" y="40.64" rot="R90"/>
-<instance part="TP3" gate="G$1" x="-45.72" y="38.1" rot="R90"/>
-<instance part="TP4" gate="G$1" x="-48.26" y="35.56" rot="R90"/>
-<instance part="TP5" gate="G$1" x="-45.72" y="33.02" rot="R90"/>
-<instance part="TP6" gate="G$1" x="-48.26" y="30.48" rot="R90"/>
+<instance part="X3" gate="-1" x="-55.88" y="43.18"/>
+<instance part="X3" gate="-2" x="-55.88" y="40.64"/>
+<instance part="X3" gate="-3" x="-55.88" y="38.1"/>
+<instance part="X3" gate="-4" x="-55.88" y="35.56"/>
+<instance part="X3" gate="-5" x="-55.88" y="33.02"/>
+<instance part="X3" gate="-6" x="-55.88" y="30.48"/>
 </instances>
 <busses>
@@
 </segment>
 <segment>
+<pinref part="X3" gate="-6" pin="1"/>
 <pinref part="GND17" gate="1" pin="GND"/>
-<wire x1="-43.18" y1="27.94" x2="-43.18" y2="30.48" width="0.1524" layer="91"/>
-<wire x1="-43.18" y1="30.48" x2="-48.26" y2="30.48" width="0.1524" layer="91"/>
-<pinref part="TP6" gate="G$1" pin="P$1"/>
+<wire x1="-53.34" y1="30.48" x2="-43.18" y2="30.48" width="0.1524" layer="91"/>
+<wire x1="-43.18" y1="30.48" x2="-43.18" y2="27.94" width="0.1524" layer="91"/>
 </segment>
 </net>
@@
 <wire x1="-22.86" y1="40.64" x2="-33.02" y2="40.64" width="0.1524" layer="91"/>
 <junction x="-22.86" y="40.64"/>
-<wire x1="-33.02" y1="40.64" x2="-48.26" y2="40.64" width="0.1524" layer="91"/>
-<pinref part="TP2" gate="G$1" pin="P$1"/>
+<wire x1="-33.02" y1="40.64" x2="-40.64" y2="40.64" width="0.1524" layer="91"/>
+<wire x1="-40.64" y1="40.64" x2="-40.64" y2="33.02" width="0.1524" layer="91"/>
+<pinref part="X3" gate="-5" pin="1"/>
+<wire x1="-40.64" y1="33.02" x2="-53.34" y2="33.02" width="0.1524" layer="91"/>
 </segment>
 </net>
@@
 <wire x1="-15.24" y1="38.1" x2="-33.02" y2="38.1" width="0.1524" layer="91"/>
 <junction x="-15.24" y="38.1"/>
-<wire x1="-33.02" y1="38.1" x2="-45.72" y2="38.1" width="0.1524" layer="91"/>
-<pinref part="TP3" gate="G$1" pin="P$1"/>
+<wire x1="-33.02" y1="38.1" x2="-43.18" y2="38.1" width="0.1524" layer="91"/>
+<pinref part="X3" gate="-3" pin="1"/>
+<wire x1="-43.18" y1="38.1" x2="-53.34" y2="38.1" width="0.1524" layer="91"/>
 </segment>
 </net>
@@
 <wire x1="-2.54" y1="35.56" x2="-30.48" y2="35.56" width="0.1524" layer="91"/>
 <wire x1="-30.48" y1="35.56" x2="-33.02" y2="35.56" width="0.1524" layer="91"/>
-<wire x1="-33.02" y1="35.56" x2="-48.26" y2="35.56" width="0.1524" layer="91"/>
-<pinref part="TP4" gate="G$1" pin="P$1"/>
+<wire x1="-33.02" y1="35.56" x2="-45.72" y2="35.56" width="0.1524" layer="91"/>
+<pinref part="X3" gate="-4" pin="1"/>
+<wire x1="-45.72" y1="35.56" x2="-53.34" y2="35.56" width="0.1524" layer="91"/>
 </segment>
 </net>
@@
 <wire x1="-2.54" y1="33.02" x2="-30.48" y2="33.02" width="0.1524" layer="91"/>
 <wire x1="-30.48" y1="33.02" x2="-35.56" y2="33.02" width="0.1524" layer="91"/>
-<wire x1="-35.56" y1="33.02" x2="-45.72" y2="33.02" width="0.1524" layer="91"/>
-<pinref part="TP5" gate="G$1" pin="P$1"/>
+<wire x1="-35.56" y1="33.02" x2="-35.56" y2="43.18" width="0.1524" layer="91"/>
+<pinref part="X3" gate="-1" pin="1"/>
+<wire x1="-35.56" y1="43.18" x2="-53.34" y2="43.18" width="0.1524" layer="91"/>
 </segment>
 </net>
@@
 <wire x1="60.96" y1="101.6" x2="60.96" y2="121.92" width="0.1524" layer="91"/>
 <wire x1="60.96" y1="121.92" x2="-43.18" y2="121.92" width="0.1524" layer="91"/>
-<wire x1="-43.18" y1="121.92" x2="-43.18" y2="43.18" width="0.1524" layer="91"/>
-<wire x1="-43.18" y1="43.18" x2="-45.72" y2="43.18" width="0.1524" layer="91"/>
-<pinref part="TP1" gate="G$1" pin="P$1"/>
-</segment>
-</net>
+<wire x1="-43.18" y1="121.92" x2="-43.18" y2="40.64" width="0.1524" layer="91"/>
+<pinref part="X3" gate="-2" pin="1"/>
+<wire x1="-43.18" y1="40.64" x2="-53.34" y2="40.64" width="0.1524" layer="91"/>
+</segment>
+</net>

Commit message: wip
Parts:
- C5: value 1uF -> 2.2uF
- R1: value 390k/560k -> 390k
Connections:
- net +3V3: now also U3.VBAT
Other:
- moved on the sheet: C3, C4

Commit message: rework to STM32 (WIP)
Parts:
- removed C18: 1uF, SparkFun-Passives:CAP0402-CAP
- removed C19, C21: 0.1uF, SparkFun-Passives:CAP0402-CAP
- removed C20: 2.2uF, SparkFun-Passives:CAP0805
- removed R2: 100k, SparkFun-Passives:RESISTOR0402-RES
- removed R3, R4, R5: 10k, SparkFun-Passives:RESISTOR0402-RES
- removed U$1: LM4F120H5QR, stellaris:LM4F120H5QR
- removed X3: SSW-103-02-S-D, con-samtec:SSW-103-02-S-D
- C1, C10, C11, C2, C3, C4, C5: device SparkFun-Passives:CAP0402-CAP -> SparkFun-Passives:CAP0603-CAP
- C12, C14: value 0.1uF -> 100nF; device SparkFun-Passives:CAP0402-CAP -> SparkFun-Passives:CAP0603-CAP
- C13, C15, C16: value 0.01uF -> 100nF; device SparkFun-Passives:CAP0402-CAP -> SparkFun-Passives:CAP0603-CAP
- C17: value 1uF -> 2.2uF; device SparkFun-Passives:CAP0402-CAP -> SparkFun-Passives:CAP0603-CAP
- C6, C9: value 0.1uF -> 2.2uF; device SparkFun-Passives:CAP0402-CAP -> SparkFun-Passives:CAP0603-CAP
- C7, C8: value 10pF -> 22pF; device SparkFun-Passives:CAP0402-CAP -> SparkFun-Passives:CAP0603-CAP
- R1: device SparkFun-Passives:RESISTOR0402-RES -> SparkFun-Passives:RESISTOR0603-RES
- U1: value ATSHA204-TSU -> STM32F205RET6; device SparkFun-DigitalIC:ATSHA204-TSU -> stm32:STM32F10XRXT6
Connections:
- removed net N$15: S1.1, U$1.PF0
- removed net N$17: R3.1, U$1.PC0/TCK/SWCLK, X3-5.1
- removed net N$19: U$1.PC2/TDI, X3-4.1
- removed net N$20: U$1.PC3/TDO/SWO, X3-1.1
- removed net N$21: C9.2, R5.1, U$1./RST, X3-2.1
- removed net N$23: C18.1, C19.1, C20.1, C21.1, U$1.VDDC
- removed net SDA: R2.1, U$1.PB3/I2C0SDA, U1.SDA
- removed net USB_D_N: U$1.PD4, U2.D-
- removed net USB_D_P: U$1.PD5, U2.D+
- new net N$3: U1PORTB_L.PB0, U3.DC/I2C_SA0
- new net N$7: U1PORTB_L.PB1, U3./RES
- net +3V3: now also C12.2, C13.2, C14.2, C15.2, C16.2, C17.2, U1AN_POWER.VBAT, U1AN_POWER.VDDA, U1POWER.VDD_1, U1POWER.VDD_2, U1POWER.VDD_3, U1POWER.VDD_4; no longer C12.1, C13.1, C14.1, C15.1, C16.1, C17.1, C6.1, R2.2, R3.2, R4.2, R5.2, U$1.VBAT, U$1.VDD, U$1.VDDA, U1.VCC
- net GND: now also C12.1, C13.1, C14.1, C15.1, C16.1, C17.1, C9.2, U1AN_POWER.VSSA, U1POWER.VSS_3, U1POWER.VSS_4, U1RESET.BOOT0; no longer C12.2, C13.2, C14.2, C15.2, C16.2, C17.2, C18.2, C19.2, C20.2, C21.2, C9.1, U$1./WAKE, U$1.GND, U$1.GNDA, U$1.GNDX, U$1.XOSC0, U1.GND, X3-6.1
- net N$1: now also U1PORTA_L.PA7; no longer U$1.PA5/SSI0TX
- net N$14: now also U1PORTA_H.PA12, U2.D+; no longer S2.1, U$1.PF1
- net N$16: now also U1PORTA_L.PA4, U3./CS; no longer R4.1, U$1.PC1/TMS/SWDIO, X3-3.1
- net N$2: now also U1PORTA_H.PA11, U2.D-; no longer U$1.PE0, U3./CS
- net N$4: now also C6.1, U1POWER.VSS_1; no longer U$1.PE2, U3.DC/I2C_SA0
- net N$5: now also U1PORTA_L.PA5; no longer U$1.PA2/SSI0CLK
- net N$8: now also C9.1, U1POWER.VSS_2; no longer U$1.PE1, U3./RES
- net XTAL1: now also U1PORTD/OSC.PD1/OSC=>; no longer U$1.OSC0
- net XTAL2: now also U1PORTD/OSC.PD0/OSC<=; no longer U$1.OSC1
Other:
- moved on the sheet: C1, C10, C11, C12, C13, C14, C15, C16, C17, C2, C3, C4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

Commit message: trezor WIP
Parts:
- added C18: 0.1uF, SparkFun-Passives:CAP0603-CAP
- added U$1: PROGRAMMER, fabhack:PROGRAMMER
- C7: value 22pF -> 2.2uF
- C9: value 2.2uF -> 22pF
- U2: device SparkFun-Connectors:USB-AB -> fabhack:47346-0001
Connections:
- net N$14 renamed USB_D_P
- net N$2 renamed USB_D_N
- new net N$14: U$1.TDO, U1PORTB_L.PB3
- new net N$15: U$1.TMS, U1PORTA_H.PA13
- new net N$17: U$1.TCK, U1PORTA_H.PA14
- new net N$18: U$1.TDI, U1PORTA_H.PA15
- new net N$19: S1.1, U1PORTC_L.PC5
- new net N$2: C18.1, U$1.RST, U1RESET.NRST
- new net N$20: S2.1, U1PORTC_L.PC2
- net +3V3: now also U$1.VDD
- net GND: now also C18.2, U$1.GND
- net N$8: now also C7.1; no longer C9.1
- net XTAL1: now also C9.1; no longer C7.1
Other:
- moved on the sheet: C12, C13, C14, C15, C16, C7, C9, S1, S2, U1PORTA_H, U1PORTC_L
