File: trezor.sch (EAGLE design)
At the start: 27 parts, among them IC1 MCP1703CB, Q2 16MHz, U1 STM32F205RET6, U2 USB, U3 DISPLAY

Commit message: add items to trezor bom
Parts:
- C12, C13, C14, C15, C16: value 100nF -> 0.1uF
Changed lines of the file:
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@@
 <part name="GND12" library="supply1" deviceset="GND" device=""/>
 <part name="GND13" library="supply1" deviceset="GND" device=""/>
-<part name="C13" library="SparkFun-Passives" deviceset="CAP" device="0603-CAP" value="100nF"/>
-<part name="C12" library="SparkFun-Passives" deviceset="CAP" device="0603-CAP" value="100nF"/>
-<part name="C15" library="SparkFun-Passives" deviceset="CAP" device="0603-CAP" value="100nF"/>
-<part name="C16" library="SparkFun-Passives" deviceset="CAP" device="0603-CAP" value="100nF"/>
-<part name="C14" library="SparkFun-Passives" deviceset="CAP" device="0603-CAP" value="100nF"/>
+<part name="C13" library="SparkFun-Passives" deviceset="CAP" device="0603-CAP" value="0.1uF"/>
+<part name="C12" library="SparkFun-Passives" deviceset="CAP" device="0603-CAP" value="0.1uF"/>
+<part name="C15" library="SparkFun-Passives" deviceset="CAP" device="0603-CAP" value="0.1uF"/>
+<part name="C16" library="SparkFun-Passives" deviceset="CAP" device="0603-CAP" value="0.1uF"/>
+<part name="C14" library="SparkFun-Passives" deviceset="CAP" device="0603-CAP" value="0.1uF"/>
 <part name="C17" library="SparkFun-Passives" deviceset="CAP" device="0603-CAP" value="2.2uF"/>
 <part name="IC1" library="linear" deviceset="MCP1703" device="CB"/>

Commit message: connect vbus to mcu as well
Connections:
- net +5V: now also U1PORTA_H.PA9
Changed lines of the file:
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@@
 <part name="GND10" library="supply1" deviceset="GND" device=""/>
 <part name="+3V6" library="supply1" deviceset="+3V3" device=""/>
+<part name="P+3" library="supply1" deviceset="+5V" device=""/>
 </parts>
 <sheets>
@@
 <instance part="+3V6" gate="G$1" x="83.82" y="134.62"/>
 <instance part="U1" gate="PORTC_L" x="132.08" y="132.08" rot="R180"/>
+<instance part="P+3" gate="1" x="20.32" y="132.08"/>
 </instances>
 <busses>
@@
 <wire x1="43.18" y1="124.46" x2="43.18" y2="127" width="0.1524" layer="91"/>
 </segment>
-</net>
+<segment>
+<pinref part="U1" gate="PORTA_H" pin="PA9"/>
+<pinref part="P+3" gate="1" pin="+5V"/>
+<wire x1="15.24" y1="127" x2="20.32" y2="127" width="0.1524" layer="91"/>
+<wire x1="20.32" y1="127" x2="20.32" y2="129.54" width="0.1524" layer="91"/>
+</segment>
+</net>

Commit message: rework swd programmer
Parts:
- removed U$1: PROGRAMMER, fabhack:PROGRAMMER
- added U$2: SWD, fabhack:SWD
Connections:
- removed net N$18: U$1.TDI, U1PORTA_H.PA15
- net +3V3: now also U$2.VDD; no longer U$1.VDD
- net GND: now also U$2.GND, U3.VSS; no longer U$1.GND
- net N$14: now also U$2.SWO; no longer U$1.TDO
- net N$15: now also U$2.SWDIO; no longer U$1.TMS
- net N$17: now also U$2.SWCLK; no longer U$1.TCK
- net N$2: now also U$2.RST; no longer U$1.RST
Changed lines of the file:
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@@
 <part name="C18" library="SparkFun-Passives" deviceset="CAP" device="0603-CAP" value="0.1uF"/>
 <part name="GND9" library="supply1" deviceset="GND" device=""/>
-<part name="U$1" library="fabhack" deviceset="PROGRAMMER" device=""/>
 <part name="GND10" library="supply1" deviceset="GND" device=""/>
 <part name="+3V6" library="supply1" deviceset="+3V3" device=""/>
 <part name="P+3" library="supply1" deviceset="+5V" device=""/>
+<part name="U$2" library="fabhack" deviceset="SWD" device=""/>
 </parts>
 <sheets>
@@
 <instance part="C18" gate="G$1" x="76.2" y="96.52" rot="R90"/>
 <instance part="GND9" gate="1" x="81.28" y="86.36"/>
-<instance part="U$1" gate="G$1" x="111.76" y="132.08" rot="MR180"/>
-<instance part="GND10" gate="1" x="93.98" y="121.92"/>
-<instance part="+3V6" gate="G$1" x="83.82" y="134.62"/>
+<instance part="GND10" gate="1" x="96.52" y="119.38"/>
+<instance part="+3V6" gate="G$1" x="96.52" y="147.32"/>
 <instance part="U1" gate="PORTC_L" x="132.08" y="132.08" rot="R180"/>
 <instance part="P+3" gate="1" x="20.32" y="132.08"/>
+<instance part="U$2" gate="G$1" x="106.68" y="132.08" rot="MR180"/>
 </instances>
 <busses>
@@
 <pinref part="C4" gate="G$1" pin="1"/>
 <junction x="134.62" y="38.1"/>
+<wire x1="119.38" y1="38.1" x2="127" y2="38.1" width="0.1524" layer="91"/>
+<junction x="127" y="38.1"/>
 <pinref part="U3" gate="G$1" pin="VBAT"/>
 <wire x1="142.24" y1="30.48" x2="139.7" y2="30.48" width="0.1524" layer="91"/>
-<wire x1="139.7" y1="30.48" x2="139.7" y2="38.1" width="0.1524" layer="91"/>
-<junction x="139.7" y="38.1"/>
-<wire x1="119.38" y1="38.1" x2="127" y2="38.1" width="0.1524" layer="91"/>
-<junction x="127" y="38.1"/>
-</segment>
-<segment>
-<pinref part="U$1" gate="G$1" pin="VDD"/>
+<wire x1="139.7" y1="30.48" x2="134.62" y2="30.48" width="0.1524" layer="91"/>
+<wire x1="134.62" y1="30.48" x2="134.62" y2="38.1" width="0.1524" layer="91"/>
+</segment>
+<segment>
+<pinref part="U$2" gate="G$1" pin="VDD"/>
 <pinref part="+3V6" gate="G$1" pin="+3V3"/>
-<wire x1="104.14" y1="129.54" x2="83.82" y2="129.54" width="0.1524" layer="91"/>
-<wire x1="83.82" y1="129.54" x2="83.82" y2="132.08" width="0.1524" layer="91"/>
+<wire x1="99.06" y1="139.7" x2="96.52" y2="139.7" width="0.1524" layer="91"/>
+<wire x1="96.52" y1="139.7" x2="96.52" y2="144.78" width="0.1524" layer="91"/>
 </segment>
 </net>
@@
 <junction x="127" y="45.72"/>
 <pinref part="GND2" gate="1" pin="GND"/>
+<pinref part="U3" gate="G$1" pin="VSS"/>
+<wire x1="142.24" y1="35.56" x2="139.7" y2="35.56" width="0.1524" layer="91"/>
+<wire x1="139.7" y1="35.56" x2="139.7" y2="40.64" width="0.1524" layer="91"/>
+<junction x="139.7" y="40.64"/>
 </segment>
 <segment>
@@
 </segment>
 <segment>
-<pinref part="U$1" gate="G$1" pin="GND"/>
 <pinref part="GND10" gate="1" pin="GND"/>
-<wire x1="104.14" y1="132.08" x2="93.98" y2="132.08" width="0.1524" layer="91"/>
-<wire x1="93.98" y1="132.08" x2="93.98" y2="124.46" width="0.1524" layer="91"/>
+<wire x1="99.06" y1="129.54" x2="96.52" y2="129.54" width="0.1524" layer="91"/>
+<wire x1="96.52" y1="129.54" x2="96.52" y2="121.92" width="0.1524" layer="91"/>
+<pinref part="U$2" gate="G$1" pin="GND"/>
 </segment>
 </net>
@@
 <net name="N$2" class="0">
 <segment>
-<pinref part="U$1" gate="G$1" pin="RST"/>
-<wire x1="104.14" y1="127" x2="68.58" y2="127" width="0.1524" layer="91"/>
+<wire x1="99.06" y1="127" x2="68.58" y2="127" width="0.1524" layer="91"/>
 <pinref part="C18" gate="G$1" pin="1"/>
 <wire x1="68.58" y1="96.52" x2="71.12" y2="96.52" width="0.1524" layer="91"/>
@@
 <wire x1="68.58" y1="127" x2="68.58" y2="96.52" width="0.1524" layer="91"/>
 <junction x="68.58" y="96.52"/>
+<pinref part="U$2" gate="G$1" pin="RST"/>
 </segment>
 </net>
@@
 <wire x1="114.3" y1="83.82" x2="114.3" y2="76.2" width="0.1524" layer="91"/>
 <wire x1="114.3" y1="76.2" x2="88.9" y2="76.2" width="0.1524" layer="91"/>
-<wire x1="88.9" y1="76.2" x2="88.9" y2="134.62" width="0.1524" layer="91"/>
-<pinref part="U$1" gate="G$1" pin="TDO"/>
-<wire x1="88.9" y1="134.62" x2="104.14" y2="134.62" width="0.1524" layer="91"/>
+<wire x1="88.9" y1="76.2" x2="88.9" y2="132.08" width="0.1524" layer="91"/>
+<wire x1="88.9" y1="132.08" x2="99.06" y2="132.08" width="0.1524" layer="91"/>
+<pinref part="U$2" gate="G$1" pin="SWO"/>
 </segment>
 </net>
 <net name="N$15" class="0">
 <segment>
-<pinref part="U$1" gate="G$1" pin="TMS"/>
-<wire x1="104.14" y1="142.24" x2="22.86" y2="142.24" width="0.1524" layer="91"/>
-<wire x1="22.86" y1="142.24" x2="22.86" y2="116.84" width="0.1524" layer="91"/>
+<wire x1="99.06" y1="137.16" x2="22.86" y2="137.16" width="0.1524" layer="91"/>
+<wire x1="22.86" y1="137.16" x2="22.86" y2="116.84" width="0.1524" layer="91"/>
 <pinref part="U1" gate="PORTA_H" pin="PA13"/>
 <wire x1="22.86" y1="116.84" x2="15.24" y2="116.84" width="0.1524" layer="91"/>
+<pinref part="U$2" gate="G$1" pin="SWDIO"/>
 </segment>
 </net>
@@
 <pinref part="U1" gate="PORTA_H" pin="PA14"/>
 <wire x1="15.24" y1="114.3" x2="25.4" y2="114.3" width="0.1524" layer="91"/>
-<wire x1="25.4" y1="114.3" x2="25.4" y2="139.7" width="0.1524" layer="91"/>
-<pinref part="U$1" gate="G$1" pin="TCK"/>
-<wire x1="25.4" y1="139.7" x2="104.14" y2="139.7" width="0.1524" layer="91"/>
-</segment>
-</net>
-<net name="N$18" class="0">
-<segment>
-<pinref part="U$1" gate="G$1" pin="TDI"/>
-<wire x1="104.14" y1="137.16" x2="27.94" y2="137.16" width="0.1524" layer="91"/>
-<wire x1="27.94" y1="137.16" x2="27.94" y2="111.76" width="0.1524" layer="91"/>
-<pinref part="U1" gate="PORTA_H" pin="PA15"/>
-<wire x1="27.94" y1="111.76" x2="15.24" y2="111.76" width="0.1524" layer="91"/>
-</segment>
-</net>
+<wire x1="25.4" y1="114.3" x2="25.4" y2="134.62" width="0.1524" layer="91"/>
+<wire x1="25.4" y1="134.62" x2="99.06" y2="134.62" width="0.1524" layer="91"/>
+<pinref part="U$2" gate="G$1" pin="SWCLK"/>
+</segment>
+</net>

Commit message: change crystal
Parts:
- Q2: value 16MHz -> 8MHz
Changed lines of the file:
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@@
 <part name="S1" library="SparkFun-Electromechanical" deviceset="SWITCH-MOMENTARY-2" device="SMD"/>
 <part name="S2" library="SparkFun-Electromechanical" deviceset="SWITCH-MOMENTARY-2" device="SMD"/>
-<part name="Q2" library="crystal" deviceset="CRYSTAL" device="CTS406" value="16MHz"/>
+<part name="Q2" library="crystal" deviceset="CRYSTAL" device="CTS406" value="8MHz"/>
 <part name="C9" library="SparkFun-Passives" deviceset="CAP" device="0603-CAP" value="22pF"/>
 <part name="C8" library="SparkFun-Passives" deviceset="CAP" device="0603-CAP" value="22pF"/>
