File: programmer-old.brd (EAGLE design)
At the start: 27.9 x 12.7 mm, 2 parts

Commit message: rework swd programmer
Parts:
- removed U$1: SWD, fabhack:SWD
- added U$2: PROGRAMMER, fabhack:PROGRAMMER
Connections:
- net GND: now also U$2.3; no longer U$1.2
- net N$1: now also U$2.7; no longer U$1.5
- net N$2: now also U$2.6; no longer U$1.4
- net N$3: now also U$2.4; no longer U$1.3
- net N$4: now also U$2.1; no longer U$1.1
- net VCC: now also U$2.2; no longer U$1.6
Routing:
- net VCC: track 14.7 -> 26.3 mm
- net N$3: track 5.34 -> 11.6 mm
- net N$4: track 5.08 -> 10.7 mm
- net N$2: track 6.26 -> 10.8 mm
- net N$1: track 6.66 -> 10.4 mm
Other:
- board size 27.9 x 12.7 mm -> 27.9 x 17.8 mm
