File: programmer-old.sch (EAGLE design)
At the start: 2 parts

Commit message: rework swd programmer
Parts:
- removed U$1: SWD, fabhack:SWD
- added U$2: PROGRAMMER, fabhack:PROGRAMMER
Connections:
- net GND: now also U$2.GND; no longer U$1.GND
- net N$1: now also U$2.TMS; no longer U$1.SWDIO
- net N$2: now also U$2.TCK; no longer U$1.SWCLK
- net N$3: now also U$2.TDO; no longer U$1.SWO
- net N$4: now also U$2.RST; no longer U$1.RST
- net VCC: now also U$2.VDD; no longer U$1.VDD
Changed lines of the file:
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@@
 </classes>
 <parts>
+<part name="U$2" library="fabhack" deviceset="PROGRAMMER" device=""/>
 <part name="JP1" library="pinhead" deviceset="PINHD-2X10" device=""/>
 <part name="P+1" library="supply1" deviceset="VCC" device=""/>
@@
 <part name="GND2" library="supply1" deviceset="GND" device=""/>
 <part name="GND3" library="supply1" deviceset="GND" device=""/>
-<part name="U$1" library="fabhack" deviceset="SWD" device=""/>
 </parts>
 <sheets>
@@
 </plain>
 <instances>
+<instance part="U$2" gate="G$1" x="5.08" y="12.7" rot="R180"/>
 <instance part="JP1" gate="A" x="83.82" y="17.78"/>
-<instance part="P+1" gate="VCC" x="60.96" y="38.1"/>
-<instance part="GND1" gate="1" x="60.96" y="-2.54"/>
+<instance part="P+1" gate="VCC" x="15.24" y="38.1"/>
+<instance part="GND1" gate="1" x="17.78" y="0"/>
 <instance part="P+2" gate="VCC" x="73.66" y="38.1"/>
 <instance part="P+3" gate="VCC" x="96.52" y="38.1"/>
 <instance part="GND2" gate="1" x="73.66" y="-2.54"/>
 <instance part="GND3" gate="1" x="96.52" y="-2.54"/>
-<instance part="U$1" gate="G$1" x="50.8" y="12.7" rot="R180"/>
 </instances>
 <busses>
@@
 <nets>
 <net name="VCC" class="0">
+<segment>
+<pinref part="U$2" gate="G$1" pin="VDD"/>
+<pinref part="P+1" gate="VCC" pin="VCC"/>
+<wire x1="12.7" y1="10.16" x2="15.24" y2="10.16" width="0.1524" layer="91"/>
+<wire x1="15.24" y1="10.16" x2="15.24" y2="35.56" width="0.1524" layer="91"/>
+</segment>
 <segment>
 <pinref part="JP1" gate="A" pin="1"/>
@@
 <wire x1="96.52" y1="27.94" x2="96.52" y2="35.56" width="0.1524" layer="91"/>
 </segment>
-<segment>
-<pinref part="U$1" gate="G$1" pin="VDD"/>
-<pinref part="P+1" gate="VCC" pin="VCC"/>
-<wire x1="58.42" y1="20.32" x2="60.96" y2="20.32" width="0.1524" layer="91"/>
-<wire x1="60.96" y1="20.32" x2="60.96" y2="35.56" width="0.1524" layer="91"/>
-</segment>
 </net>
 <net name="GND" class="0">
+<segment>
+<pinref part="U$2" gate="G$1" pin="GND"/>
+<pinref part="GND1" gate="1" pin="GND"/>
+<wire x1="12.7" y1="12.7" x2="17.78" y2="12.7" width="0.1524" layer="91"/>
+<wire x1="17.78" y1="12.7" x2="17.78" y2="2.54" width="0.1524" layer="91"/>
+</segment>
 <segment>
 <pinref part="JP1" gate="A" pin="3"/>
@@
 <junction x="96.52" y="5.08"/>
 </segment>
-<segment>
-<pinref part="U$1" gate="G$1" pin="GND"/>
-<pinref part="GND1" gate="1" pin="GND"/>
-<wire x1="58.42" y1="10.16" x2="60.96" y2="10.16" width="0.1524" layer="91"/>
-<wire x1="60.96" y1="10.16" x2="60.96" y2="0" width="0.1524" layer="91"/>
-</segment>
 </net>
 <net name="N$1" class="0">
 <segment>
 <pinref part="JP1" gate="A" pin="7"/>
-<wire x1="81.28" y1="20.32" x2="66.04" y2="20.32" width="0.1524" layer="91"/>
-<wire x1="66.04" y1="20.32" x2="66.04" y2="17.78" width="0.1524" layer="91"/>
-<pinref part="U$1" gate="G$1" pin="SWDIO"/>
-<wire x1="66.04" y1="17.78" x2="58.42" y2="17.78" width="0.1524" layer="91"/>
+<wire x1="81.28" y1="20.32" x2="43.18" y2="20.32" width="0.1524" layer="91"/>
+<wire x1="43.18" y1="20.32" x2="43.18" y2="22.86" width="0.1524" layer="91"/>
+<pinref part="U$2" gate="G$1" pin="TMS"/>
+<wire x1="43.18" y1="22.86" x2="12.7" y2="22.86" width="0.1524" layer="91"/>
 </segment>
 </net>
@@
 <segment>
 <pinref part="JP1" gate="A" pin="9"/>
-<wire x1="81.28" y1="17.78" x2="68.58" y2="17.78" width="0.1524" layer="91"/>
-<wire x1="68.58" y1="17.78" x2="68.58" y2="15.24" width="0.1524" layer="91"/>
-<pinref part="U$1" gate="G$1" pin="SWCLK"/>
-<wire x1="68.58" y1="15.24" x2="58.42" y2="15.24" width="0.1524" layer="91"/>
+<wire x1="81.28" y1="17.78" x2="40.64" y2="17.78" width="0.1524" layer="91"/>
+<pinref part="U$2" gate="G$1" pin="TCK"/>
+<wire x1="40.64" y1="17.78" x2="40.64" y2="20.32" width="0.1524" layer="91"/>
+<wire x1="40.64" y1="20.32" x2="12.7" y2="20.32" width="0.1524" layer="91"/>
 </segment>
 </net>
@@
 <segment>
 <pinref part="JP1" gate="A" pin="13"/>
-<wire x1="81.28" y1="12.7" x2="58.42" y2="12.7" width="0.1524" layer="91"/>
-<pinref part="U$1" gate="G$1" pin="SWO"/>
+<wire x1="81.28" y1="12.7" x2="40.64" y2="12.7" width="0.1524" layer="91"/>
+<wire x1="40.64" y1="12.7" x2="40.64" y2="15.24" width="0.1524" layer="91"/>
+<pinref part="U$2" gate="G$1" pin="TDO"/>
+<wire x1="40.64" y1="15.24" x2="12.7" y2="15.24" width="0.1524" layer="91"/>
 </segment>
 </net>
@@
 <segment>
 <pinref part="JP1" gate="A" pin="15"/>
-<wire x1="81.28" y1="10.16" x2="68.58" y2="10.16" width="0.1524" layer="91"/>
-<wire x1="68.58" y1="10.16" x2="68.58" y2="7.62" width="0.1524" layer="91"/>
-<pinref part="U$1" gate="G$1" pin="RST"/>
-<wire x1="68.58" y1="7.62" x2="58.42" y2="7.62" width="0.1524" layer="91"/>
+<wire x1="81.28" y1="10.16" x2="40.64" y2="10.16" width="0.1524" layer="91"/>
+<wire x1="40.64" y1="10.16" x2="40.64" y2="7.62" width="0.1524" layer="91"/>
+<pinref part="U$2" gate="G$1" pin="RST"/>
+<wire x1="40.64" y1="7.62" x2="12.7" y2="7.62" width="0.1524" layer="91"/>
 </segment>
 </net>
