File: electronics/trezor_v1.1.brd (EAGLE design)
At the start: 50 x 26.7 mm, 47 parts, among them IC1 MCP1703T-3302E/CB, K1 USB5_USB_MICRO_MOLEX475890001, K2 SWD, Q2 8MHz, U1 STM32F205RET6, U3 DISPLAY

Commit message: cleanup eagle filenames (trezor -> trezor_v1.0, trezor_v1 -> trezor_v1.1)
Parts:
- removed U$5: (no value), vyber:RAM_BRD
Other:
- board text removed: "1,5mm / 35µm"
- board text removed: "1.00"
- board text removed: "49.99x26.70 mm"
- board text removed: "FR4"
- board text removed: "Galv. Au"
- board text removed: "Krelina"
- board text removed: "TREZOR"
- board text removed: "frézovat"
- board text removed: "±0,2mm"
Changed lines of the file:
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@@
 <wire x1="62.3" y1="0" x2="62.3" y2="26.7" width="0.2" layer="47"/>
 <wire x1="-18.14" y1="0" x2="-18.14" y2="26.64" width="0.2" layer="47"/>
-<text x="68.4784" y="-76.5048" size="1.778" layer="48">Krelina</text>
-<text x="68.4784" y="-58.4708" size="1.778" layer="48">TREZOR</text>
-<text x="65.6336" y="-68.834" size="1.778" layer="48">1.00</text>
-<text x="-83.4136" y="-57.4548" size="1.524" layer="48">49.99x26.70 mm</text>
-<text x="-76.5556" y="-61.2648" size="1.524" layer="48">±0,2mm</text>
-<text x="-80.8736" y="-64.5668" size="1.524" layer="48">1,5mm / 35µm</text>
-<text x="-73.7616" y="-68.8848" size="1.524" layer="48">FR4</text>
-<text x="-78.3336" y="-72.6948" size="1.524" layer="48">Galv. Au</text>
-<text x="-78.3336" y="-76.5048" size="1.524" layer="48">frézovat</text>
 <wire x1="-60.5536" y1="-80.1878" x2="-58.5216" y2="-80.1878" width="0.0762" layer="144"/>
 <wire x1="-59.5376" y1="-79.1718" x2="-59.5376" y2="-81.2038" width="0.0762" layer="144"/>
@@
 <pass name="Default">
 <param name="RoutingGrid" value="50mil"/>
+<param name="AutoGrid" value="1"/>
+<param name="Efforts" value="0"/>
+<param name="TopRouterVariant" value="1"/>
 <param name="tpViaShape" value="round"/>
 <param name="PrefDir.1" value="|"/>
@@
 <attribute name="VALUE" x="46.9646" y="25.1714" size="0.8128" layer="27" rot="R270"/>
 </element>
-<element name="U$5" library="vyber" package="RAM_BRD" value="" x="-114.4016" y="-82.6008"/>
 </elements>
 <signals>
