File: electronics/trezor_v1.1.sch (EAGLE design)
At the start: 44 parts, among them IC1 MCP1703T-3302E/CB, K1 USB5_USB_MICRO_MOLEX475890001, K2 SWD, Q2 8MHz, U1 STM32F205RET6, U3 DISPLAY

Commit message: cleanup eagle filenames (trezor -> trezor_v1.0, trezor_v1 -> trezor_v1.1)
Other:
- note removed: "1.00"
- note removed: "Krelina"
- note removed: "TREZOR"
Changed lines of the file:
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@@
 <part name="K2" library="fabhack" deviceset="SWD" device=""/>
 <part name="K1" library="vyber" deviceset="USB5" device="_USB_MICRO_MOLEX475890001"/>
-<part name="U$1" library="vyber" deviceset="RAM_A3" device=""/>
 <part name="R2" library="vyber" deviceset="POLYSWITCH" device="_0603" value="MF-FSMF020X-2 "/>
 <part name="GND14" library="supply1" deviceset="GND" device=""/>
@@
 <sheet>
 <plain>
-<text x="205.74" y="-47.244" size="1.9304" layer="97">Krelina</text>
-<text x="213.36" y="-30.48" size="1.9304" layer="97">TREZOR</text>
-<text x="205.74" y="-39.37" size="1.9304" layer="97">1.00</text>
 </plain>
 <instances>
@@
 <attribute name="NAME" x="55.88" y="155.194" size="1.27" layer="95" rot="MR0"/>
 </instance>
-<instance part="U$1" gate="G$1" x="-76.2" y="-58.42"/>
-<instance part="U$1" gate="G$2" x="175.26" y="-53.34"/>
 <instance part="R2" gate="G$1" x="10.16" y="152.4" smashed="yes">
 <attribute name="NAME" x="12.065" y="150.495" size="1.27" layer="95" rot="R180"/>
