File: electronics/trezor_model_t/kicad/CYM1A113.kicad_pcb (KiCad board)
At the start: 4 copper layers, 59 x 33.8 mm, 132 parts, among them IC1 MIC803-29D2VC3, IC2 STM32F427VIT6, IC5 TPS61043, IC6 XC6210B332PR, K1 DX07B024XJ1R1300, K3 ATTEND_112J-TDAR-R01, K4 DF37NB-24DS-0.4V, K5 SWD, K6 DF37NB-10DS-0.4V, T1 DMG3415U-7, T2 DMG3415U-7, X1 CTS406 8MHz

Commit message: Board edge rendering correction on kicad
Parts:
- added REF**: OSHW-Logo_5.7x6mm_SilkScreen, Symbol:OSHW-Logo_5.7x6mm_SilkScreen, F.Cu at (159.5, 95.7)
- moved K1 0.14 mm to (120.7, 105.1)
Connections:
- K1 pad A1: GND -> (no net)
- K1 pad A10: Net-(K1-PadA10) -> (no net)
- K1 pad A11: Net-(K1-PadA11) -> (no net)
- K1 pad A12: GND -> (no net)
- K1 pad A2: Net-(K1-PadA2) -> (no net)
- K1 pad A3: Net-(K1-PadA3) -> (no net)
- K1 pad A4: /VBUS -> (no net)
- K1 pad A5: /CC1 -> (no net)
- K1 pad A6: /DP -> (no net)
- K1 pad A7: /DN -> (no net)
- K1 pad A8: /SBU1 -> (no net)
- K1 pad A9: /VBUS -> (no net)
- K1 pad B1: GND -> (no net)
- K1 pad B10: Net-(K1-PadB10) -> (no net)
- K1 pad B11: Net-(K1-PadB11) -> (no net)
- K1 pad B12: GND -> (no net)
- K1 pad B2: Net-(K1-PadB2) -> (no net)
- K1 pad B3: Net-(K1-PadB3) -> (no net)
- K1 pad B4: /VBUS -> (no net)
- K1 pad B5: /CC2 -> (no net)
- K1 pad B6: /DP -> (no net)
- K1 pad B7: /DN -> (no net)
- K1 pad B8: /SBU2 -> (no net)
- K1 pad B9: /VBUS -> (no net)
- K1 pad SH1: Net-(C25-PadP$2) -> (no net)
- K1 pad SH2: Net-(C25-PadP$2) -> (no net)
- K1 pad SH3: Net-(C1-PadP$2) -> (no net)
- K1 pad SH4: Net-(C1-PadP$2) -> (no net)
Routing:
- net VCC-2: track 89.3 -> 97.2 mm
- net GND: track 35.4 -> 32.9 mm
- net (no net): track 0.00 -> 2.52 mm
- net /LEDA: track 36.6 -> 37.8 mm

Commit message: Fixed filled zones bug, connection issues
Connections:
- K1 pad A4: (no net) -> /VBUS
- K1 pad A5: (no net) -> /CC1
- K1 pad A6: (no net) -> /DP
- K1 pad A7: (no net) -> /DN
- K1 pad B6: (no net) -> /DP
- K1 pad B7: (no net) -> /DN
- K1 pad B9: (no net) -> /VBUS
- K1 pad SH1: (no net) -> Net-(C25-PadP$2)
- K1 pad SH2: (no net) -> Net-(C25-PadP$2)
Routing:
- net /VBUS: track 10.4 -> 4.72 mm
- net (no net): track 2.52 -> 8.12 mm
- net VCC-2: track 97.2 -> 102.8 mm, vias 20 -> 21
- net /DN: track 9.50 -> 10.1 mm
Other:
- net class smol added: clearance 0.12, trace_width 0.125, via_dia 0.8, via_drill 0.4
