File: electronics/trezor_model_t/kicad/CYM1A113.kicad_pcb (KiCad board)
At the start: 4 copper layers, 59 x 33.8 mm, 133 parts, among them IC1 MIC803-29D2VC3, IC2 STM32F427VIT6, IC5 TPS61043, IC6 XC6210B332PR, K1 DX07B024XJ1R1300, K3 ATTEND_112J-TDAR-R01, K4 DF37NB-24DS-0.4V, K5 SWD, K6 DF37NB-10DS-0.4V, T1 DMG3415U-7, T2 DMG3415U-7, X1 CTS406 8MHz

Commit message: update mosfet
Parts:
- T1, T2: value DMG3415U-7 -> DMP2045U
Changed lines of the file:
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@@
       (effects (font (size 0.9652 0.9652) (thickness 0.08128)) (justify right top))
     )
-    (fp_text value DMG3415U-7 (at -1.27 2.54 270) (layer F.Fab)
+    (fp_text value DMP2045U (at -1.27 2.54 270) (layer F.Fab)
       (effects (font (size 0.9652 0.9652) (thickness 0.08128)) (justify right top))
     )
@@
       (effects (font (size 0.9652 0.9652) (thickness 0.08128)) (justify right top))
     )
-    (fp_text value DMG3415U-7 (at -1.27 2.54 180) (layer F.Fab)
+    (fp_text value DMP2045U (at -1.27 2.54 180) (layer F.Fab)
       (effects (font (size 0.9652 0.9652) (thickness 0.08128)) (justify right top))
     )
