File: electronics/trezor_model_t/kicad/CYM1A113.sch (KiCad schematic (older format))
At the start: 123 parts, among them IC1 MIC803-29D2VC3, IC2 STM32F427VIT6, IC5 TPS61043, IC6 XC6210B332PR, K1 DX07B024XJ1R1300, K3 ATTEND_112J-TDAR-R01, K4 DF37NB-24DS-0.4V, K5 SWD, K6 DF37NB-10DS-0.4V, T1 DMG3415U-7, T2 DMG3415U-7, X1 CTS406 8MHz

Commit message: update mosfet
Parts:
- T1, T2: value DMG3415U-7 -> DMP2045U
Changed lines of the file:
@@
-$EndComp
-$Comp
-L CYM1A113-eagle-import:RAM_A3 #U$41
-U 1 1 F5F54D26
-P 850 10950
-F 0 "#U$41" H 850 10950 50  0001 C CNN
-F 1 "RAM_A3" H 850 10950 50  0001 C CNN
-F 2 "" H 850 10950 50  0001 C CNN
-F 3 "" H 850 10950 50  0001 C CNN
-	1    850  10950
-	1    0    0    -1
-$EndComp
-$Comp
-L CYM1A113-eagle-import:RAM_A3 #U$41
-U 2 1 F5F54D2A
-P 10750 10750
-F 0 "#U$41" H 10750 10750 50  0001 C CNN
-F 1 "RAM_A3" H 10750 10750 50  0001 C CNN
-F 2 "" H 10750 10750 50  0001 C CNN
-F 3 "" H 10750 10750 50  0001 C CNN
-	2    10750 10750
-	1    0    0    -1
 $EndComp
 $Comp
@@
 P 14100 2050
 F 0 "T1" H 14290 2075 42  0000 L BNN
-F 1 "DMG3415U-7" H 14290 1955 42  0000 L BNN
+F 1 "DMP2045U" H 14290 1955 42  0000 L BNN
 F 2 "CYM1A113:SOT23_REFLOW" H 14100 2050 50  0001 C CNN
 F 3 "" H 14100 2050 50  0001 C CNN
@@
 P 3900 5300
 F 0 "T2" H 4090 5325 42  0000 L BNN
-F 1 "DMG3415U-7" H 4090 5205 42  0000 L BNN
+F 1 "DMP2045U" H 4090 5205 42  0000 L BNN
 F 2 "CYM1A113:SOT23_REFLOW" H 3900 5300 50  0001 C CNN
 F 3 "" H 3900 5300 50  0001 C CNN
