File: electronics/trezor_one/kicad/trezor_v1.1.kicad_pcb (KiCad board)
At the start: 16 copper layers, 50 x 26.7 mm, 46 parts, among them IC1 MCP1703T-3302E/CB, K1 USB5_USB_MICRO_MOLEX475890001, K2 SWD, Q2 8MHz, U1 STM32F205RET6, U3 DISPLAY

Commit message: kicad import bug fixes
fixed issues with the usb connector footprint causing kicad to be confused about the correct board edge shape
Routing:
- net GND: track 212.4 -> 208.5 mm
- net Net-(MB5-Pad1): track 17.8 -> 21.3 mm
- net Net-(MB6-Pad1): track 27.9 -> 31.5 mm
- net Net-(C19-Pad2): track 22.9 -> 23.9 mm, vias 0 -> 4

Commit message: add OSHW logo to Trezor One PCB
Parts:
- added REF**: OSHW-Logo_5.7x6mm_SilkScreen, Symbol:OSHW-Logo_5.7x6mm_SilkScreen, F.Cu at (159.5, 98.2)
