File: electronics/trezor_model_t/CYM1A113.brd (EAGLE design)
At the start: 59 x 33.8 mm, 132 parts, among them IC1 MIC803-29D2VC3, IC2 STM32F427VIT6, IC5 TPS61043, IC6 XC6210B332PR, K1 DX07B024XJ1R1300, K3 ATTEND_112J-TDAR-R01, K4 DF37NB-24DS-0.4V, K5 SWD, K6 DF37NB-10DS-0.4V, T1 DMG3415U-7, T2 DMG3415U-7, X1 CTS406 8MHz

Commit message: update mosfet
Parts:
- T1, T2: value DMG3415U-7 -> DMP2045U
Changed lines of the file:
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@@
 <element name="C55" library="vyber_stara_nemenit" package="0402" value="100n" x="47.7" y="4.6" rot="R90"/>
 <element name="C56" library="vyber_stara_nemenit" package="0603_REFLOW" value="1u" x="44.1" y="17.9" rot="R90"/>
-<element name="T1" library="trezor" package="SOT23_REFLOW" value="DMG3415U-7" x="54.65" y="14.1" rot="R270"/>
+<element name="T1" library="trezor" package="SOT23_REFLOW" value="DMP2045U" x="54.65" y="14.1" rot="R270"/>
 <element name="R2" library="vyber_stara_nemenit" package="0402" value="470k" x="54.1" y="11.85" rot="R180"/>
 <element name="C57" library="vyber_stara_nemenit" package="0402" value="220p" x="55.25" y="10.7" rot="R180"/>
 <element name="R3" library="vyber_stara_nemenit" package="0402" value="22k" x="55.95" y="12.25" rot="R270"/>
-<element name="T2" library="trezor" package="SOT23_REFLOW" value="DMG3415U-7" x="61.4" y="30.5" rot="R180"/>
+<element name="T2" library="trezor" package="SOT23_REFLOW" value="DMP2045U" x="61.4" y="30.5" rot="R180"/>
 <element name="R17" library="vyber_stara_nemenit" package="0402" value="470k" x="59" y="27" rot="R270"/>
 <element name="IC1" library="trezor" package="SOT23_MEDIUM_SIZE" value="MIC803-29D2VC3" x="46" y="2.65" rot="R270"/>
