File: electronics/trezor_model_t/CYM1A113.sch (EAGLE design)
At the start: 123 parts, among them IC1 MIC803-29D2VC3, IC2 STM32F427VIT6, IC5 TPS61043, IC6 XC6210B332PR, K1 DX07B024XJ1R1300, K3 ATTEND_112J-TDAR-R01, K4 DF37NB-24DS-0.4V, K5 SWD, K6 DF37NB-10DS-0.4V, T1 DMG3415U-7, T2 DMG3415U-7, X1 CTS406 8MHz

Commit message: update mosfet
Parts:
- T1, T2: value DMG3415U-7 -> DMP2045U
Changed lines of the file:
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@@
 <part name="U$84" library="vyber_stara_nemenit" deviceset="GND" device=""/>
 <part name="C56" library="vyber_stara_nemenit" deviceset="C" device="_0603$REFLOW" value="1u"/>
-<part name="T1" library="trezor" deviceset="PMOS" device="_SOT-23_REF" value="DMG3415U-7"/>
+<part name="T1" library="trezor" deviceset="PMOS" device="_SOT-23_REF" value="DMP2045U"/>
 <part name="R2" library="vyber_stara_nemenit" deviceset="R" device="_0402" value="470k"/>
 <part name="C57" library="vyber_stara_nemenit" deviceset="C" device="_0402" value="220p"/>
@@
 <part name="U$85" library="vyber_stara_nemenit" deviceset="GND" device=""/>
 <part name="U$86" library="vyber_stara_nemenit" deviceset="VCC-2" device="" value="3V3"/>
-<part name="T2" library="trezor" deviceset="PMOS" device="_SOT-23_REF" value="DMG3415U-7"/>
+<part name="T2" library="trezor" deviceset="PMOS" device="_SOT-23_REF" value="DMP2045U"/>
 <part name="R17" library="vyber_stara_nemenit" deviceset="R" device="_0402" value="470k"/>
 <part name="U$51" library="vyber_stara_nemenit" deviceset="VBAT" device="" value="VDD"/>
